File: circuts/motordriver/motordriver.kicad_sch (KiCad schematic)
At the start: 167 parts, among them IC1 PIC16F15243-I_SS, J1 DE9_Plug, J10 Power, J2 OSTTC060162, J4 OSTTC060162, J8 B5B-XH-A_LF__SN_, Q1 IRFS4227, Q13 IRFS4227, Q18 IRFS4227, Q26 IRFS4227, Q27 IRFS4227, Q3 IRFS4227, Q30 IRFS4227, Q31 IRFS4227, Q4 IRFS4227, Q5 IRFS4227, U1 3.3v, U10 IR25602S, U2 UC3843, U3 IR25602S, U4 IR25602S, U5 LM358DT, U6 UC3843, U8 IR25602S

Commit message: compact ic int
Parts:
- removed C36: C, Capacitor_THT:CP_Radial_D8.0mm_P5.00mm, symbol Device:C
- removed C37, C41, C5, C7: C_Polarized, Capacitor_THT:CP_Radial_D8.0mm_P5.00mm, symbol Device:C_Polarized
- removed C40, C42, C6: C, Resistor_SMD:R_0805_2012Metric_Pad1.20x1.40mm_HandSolder, symbol Device:C
- removed D1, D11, D12, D2, D3, D30, D31, D34, D36, D38, D4, D40, D41, D42, D43, D44, D5, D6, D7, D8: 1N4004-T_NRND, Diode_SMD:D_SOD-123, symbol dk_Diodes-Rectifiers-Single:1N4004-T_NRND
- removed Q13, Q18, Q26, Q27, Q3, Q30, Q31, Q4: IRFS4227, Package_TO_SOT_SMD:TO-263-3_TabPin2, symbol Transistor_FET:IRF540N
- removed R1, R22, R25, R26, R28, R35, R36, R4: 10, Resistor_SMD:R_0805_2012Metric_Pad1.20x1.40mm_HandSolder, symbol Device:R_US
- removed U10, U3, U4, U8: IR25602S, Package_SO:SOIC-8_3.9x4.9mm_P1.27mm, symbol Driver_FET:IR25602S
Connections:
- net M2_L: no longer C1.2, C4.1
- net M2_R: no longer C1.1

Commit message: last_touches
Parts:
- removed C10, C9: 1nf, Resistor_SMD:R_0805_2012Metric_Pad1.20x1.40mm_HandSolder, symbol Device:C
- removed C8: 2uf, Resistor_SMD:R_0805_2012Metric_Pad1.20x1.40mm_HandSolder, symbol Device:C
- removed D14, D15, D21: 1N4004-T_NRND, Diode_SMD:D_SOD-123, symbol dk_Diodes-Rectifiers-Single:1N4004-T_NRND
- removed Q5: IRFS4227, Package_TO_SOT_SMD:TO-263-3_TabPin2, symbol Transistor_FET:IRFS4227
- removed U6: UC3843, Package_SO:SOIC-8_3.9x4.9mm_P1.27mm, symbol Regulator_Controller:UC3842_SOIC8
- removed ZD1: 3.3v, Diode_SMD:D_MiniMELF, symbol Diode:BZV55B4V7
- added C5: 2uf, Resistor_SMD:R_0805_2012Metric_Pad1.20x1.40mm_HandSolder, symbol Device:C
- added D1, D2, D3, D4, D5: 1N4004-T_NRND, Diode_SMD:D_SOD-123, symbol dk_Diodes-Rectifiers-Single:1N4004-T_NRND
- added J3: XT60-M, XT60-M:AMASS_XT60-M, symbol XT60-M:XT60-M
- added J5: 640456-3, digikey-footprints:PinHeader_1x3_P2.54_Drill1.1mm, symbol dk_Rectangular-Connectors-Headers-Male-Pins:640456-3
- added Q1, Q10, Q2, Q3, Q4, Q5, Q6, Q9: MMBTA06, Package_TO_SOT_SMD:SOT-23, symbol Transistor_BJT:MMBTA06
- added Q3, Q7, Q8: IRFS4227, Package_TO_SOT_SMD:TO-263-3_TabPin2, symbol Transistor_FET:IRFS4227
- added R1, R63, R64, R73: 10k, Resistor_SMD:R_0805_2012Metric_Pad1.20x1.40mm_HandSolder, symbol Device:R_US
- added R22, R71, R74, R75: 220, Resistor_SMD:R_0805_2012Metric_Pad1.20x1.40mm_HandSolder, symbol Device:R_US
- added R25, R28, R43, R61: 470, Resistor_SMD:R_0805_2012Metric_Pad1.20x1.40mm_HandSolder, symbol Device:R_US
- added R26, R35, R36, R4, R42, R67, R72, R76: 2k, Resistor_SMD:R_0805_2012Metric_Pad1.20x1.40mm_HandSolder, symbol Device:R_US
- added R4, R65, R69: 56k, Resistor_SMD:R_0805_2012Metric_Pad1.20x1.40mm_HandSolder, symbol Device:R_US
- added R62: 0.3, Resistor_THT:R_Axial_DIN0414_L11.9mm_D4.5mm_P25.40mm_Horizontal, symbol Device:R_US
- added R66: 56k, symbol Device:R_US
- added R68: 100k, Resistor_SMD:R_0805_2012Metric_Pad1.20x1.40mm_HandSolder, symbol Device:R_US
- added R70: 5k, symbol Device:R_US
- added U3, U4, U6, U7, U8: BTS7960B, BTS7960B:DPAK127P1490X440-8N, symbol BTS7960B:BTS7960B
- added U9: LM358DT, Package_SO:SOIC-8_3.9x4.9mm_P1.27mm, symbol dk_Linear-Amplifiers-Instrumentation-OP-Amps-Buffer-Amps:LM358DT
- C1, C4: value C -> 2uf
- R16: value 22 -> 2k
- R29, R30, R41: value 10k -> 2k
- R40: value 10k -> 470
- R47: value 56k -> 2k
- R48: value 22 -> 330
- R49: value 100K -> 0.3; footprint Resistor_SMD:R_0805_2012Metric_Pad1.20x1.40mm_HandSolder -> Resistor_THT:R_Axial_DIN0414_L11.9mm_D4.5mm_P25.40mm_Horizontal
- R50: value 300K -> 0.3; footprint Resistor_SMD:R_0805_2012Metric_Pad1.20x1.40mm_HandSolder -> Resistor_THT:R_Axial_DIN0414_L11.9mm_D4.5mm_P25.40mm_Horizontal
Connections:
- net 3.3V: now also R1.1, R73.1
- net 5v+: now also R76.1; no longer R47.2
- net GND: now also C1.2, R30.2, R40.2, R50.2, C5.2, J3.N (NEG), Q1.2 (E), Q10.2 (E), Q2.2 (E), Q4.2 (E), Q9.2 (E), R35.2, R42.2, R61.2, R62.2, R64.2, R65.2, R67.2, R69.2, U9.4 (VCC-)
- net HV: now also R29.1, R47.1, R4.1, R4.1, U3.7 (VS), U4.7 (VS), U6.7 (VS), U7.7 (VS), U8.7 (VS), U9.8 (VCC+)
- net HVblock: now also J3.P (POS)
- net M1_L: now also U8.4 (OUT), U8.8 (OUT)
- net M1_R: now also U6.4 (OUT), U6.8 (OUT)
- net M1_S1: now also R75.1, U8.2 (IN)
- net M1_S2: no longer IC1.15 (RC1)
- net M1_current_sen: now also R70.1
- net M2_L: now also U7.4 (OUT), U7.8 (OUT)
- net M2_R: now also U3.4 (OUT), U3.8 (OUT)
- net M2_S1: now also R32.1, R22.1, U7.2 (IN); no longer R30.1
- net M2_S2: no longer IC1.12 (RB5), R29.1
- net Motor1_OFF: now also R74.1; no longer R41.1
- net Motor2_OFF: now also R71.1; no longer R40.1
- net PGC: now also R26.1; no longer C23.1, R14.1, R15.2, ZD20.1 (K)
- net PGD: now also R25.1, R28.1, R43.1; no longer R49.1, R50.2
- net voltge_sen: now also R48.1; no longer C12.1, R18.1, R19.2, ZD11.1 (K)
- net at Q1.1 (G): now also Q3.3 (C), R4.2; no longer R16.1
- net at R15.1, U2.6 (OUT): no longer R16.2
- net at U2.1 (COMP): now also R76.2; no longer R40.2
- net at C3.1, R3.1: now also J5.1; no longer U2.4 (RC)
- net at R50.1: now also C1.1, R49.1, D4.2 (A), Q5.2 (E), Q8.3 (S), R62.1, R63.1; no longer R48.2
- net at C43.1, D25.2 (A), Q1.3 (S)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: now also Q3.2 (E)
- net error 1: now reaches R41.2
- net error 1: now also R61.1, U6.6 (IS), U8.6 (IS)
- net at D25.1 (K), Q1.2 (D): now also U3.1 (GND), U7.1 (GND)
- net at C4.1: now also R63.2, R65.1, U9.3
- net at C4.2: now also R64.1, R66.2, U9.2
- net at R29.2: now also Q6.3 (C), Q7.1 (G)
- net cs1 renamed CS
- net CS: now also U2.3 (CS), D2.1 (K), D5.1 (K)
- net cs2: no longer names the net of C44.1, R38.1, R39.1
- net cs2: now also D2.2 (A); no longer U2.3 (CS)
- new net: D1.1 (K), Q3.2 (D)
- new net: D1.2 (A), Q3.3 (S)
- new net: J5.2, U2.4 (RC)
- new net: Q3.1 (B), R25.2
- new net: C5.1, D5.2 (A), R68.1, R69.1
- new net: Q10.1 (B), R74.2
- new net: Q9.1 (B), R75.2
- new net: J5.3, R26.2
- new net: R42.1, U6.5 (SR)
- new net: R67.1, U8.5 (SR)
- new net: Q4.1 (B), R71.2
- new net: R66.1, R68.2, R70.2, U9.1
- new net: Q2.1 (B), R22.2
- new net: U4.4 (OUT), U4.8 (OUT)
- new net: D3.1 (K), Q7.2 (D)
- new net: D3.2 (A), Q7.3 (S)
- new net: IC1.12 (RB5), R36.1
- new net: IC1.15 (RC1), R41.1
- new net: C12.1, R18.1, R19.2, R48.2, ZD11.1 (K)
- new net: Q5.1 (B), R43.2
- new net: Q5.3 (C), Q8.1 (G), R47.2
- new net: Q6.1 (B), R28.2
- new net: D4.1 (K), Q8.2 (D), U6.1 (GND), U8.1 (GND)
- new net: Q1.3 (C), Q3.1 (G), R4.2
- new net: R30.1, U3.5 (SR)
- new net: R35.1, U7.5 (SR)
- new net INH1: Q10.3 (C), R72.2, U6.3 (INH), U8.3 (INH)
- new net INH2: Q4.3 (C), R16.2, U3.3 (INH), U7.3 (INH)
- new net M1_D1: Q9.3 (C), R73.2, U6.2 (IN)
- new net M2_D1: Q2.3 (C), R1.2, U3.2 (IN)
- new net PWM: C23.1, R14.1, R15.2, R16.1, R72.1, ZD20.1 (K)
- new net error 2: R36.2, R40.1, U3.6 (IS), U7.6 (IS)
Other:
- moved on the sheet: C11, C2, C23, C24, C3, C30, C32, C43, C44, C45, C46, D10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

Commit message: last
Parts:
- removed C11, C45, C46: 2uf, Resistor_SMD:R_0805_2012Metric_Pad1.20x1.40mm_HandSolder, symbol Device:C
- removed D1, D3: 1N4004-T_NRND, Diode_SMD:D_SOD-123, symbol dk_Diodes-Rectifiers-Single:1N4004-T_NRND
- removed Q1, Q6: MMBTA06, Package_TO_SOT_SMD:SOT-23, symbol Transistor_BJT:MMBTA06
- removed Q3, Q7: IRFS4227, Package_TO_SOT_SMD:TO-263-3_TabPin2, symbol Transistor_FET:IRFS4227
- removed R21, R24, R31, R32, R33, R34, R54, R55: 10k, Resistor_SMD:R_0805_2012Metric_Pad1.20x1.40mm_HandSolder, symbol Device:R_US
- removed R28: 470, Resistor_SMD:R_0805_2012Metric_Pad1.20x1.40mm_HandSolder, symbol Device:R_US
- removed R29: 2k, Resistor_SMD:R_0805_2012Metric_Pad1.20x1.40mm_HandSolder, symbol Device:R_US
- removed R4, R56, R59: 56k, Resistor_SMD:R_0805_2012Metric_Pad1.20x1.40mm_HandSolder, symbol Device:R_US
- removed R51, R52, R53: 0.3, Resistor_THT:R_Axial_DIN0414_L11.9mm_D4.5mm_P25.40mm_Horizontal, symbol Device:R_US
- removed R57: 56k, symbol Device:R_US
- removed R58: 100k, Resistor_SMD:R_0805_2012Metric_Pad1.20x1.40mm_HandSolder, symbol Device:R_US
- removed R60: 5k, symbol Device:R_US
- removed U4: BTS7960B, BTS7960B:DPAK127P1490X440-8N, symbol BTS7960B:BTS7960B
- removed unit 2 of U5
- added R77, R78, R79, R80, R81, R82: 5.1k, Resistor_SMD:R_0805_2012Metric_Pad1.20x1.40mm_HandSolder, symbol Device:R_US
- C23: value 1nf -> 100pf
- R14: value 100K -> 3.3k
- R15: value 300K -> 10k
- R16: value 2k -> 470
- R25: value 470 -> 220
- R46: value 5k -> 2.2k
Connections:
- net GND: now also R77.2, R78.2, R79.2, R80.2, R81.2, R82.2
- net at Q3.1 (B), R25.2: now also R77.1
- net at Q10.1 (B), R74.2: now also R82.1
- net at Q9.1 (B), R75.2: now also R81.1
- net at Q4.1 (B), R71.2: now also R79.1
- net at Q2.1 (B), R22.2: now also R80.1
- net at Q5.1 (B), R43.2: now also R78.1
Other:
- moved on the sheet: C23, C33, C34, C38, C39, C47, C48, D18, D19, F2, Q9, R10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

Commit message: lay out
Parts:
- IC1: footprint SOP65P780X200-20N:SOP65P780X200-20N -> pic16f15243:SSOP20_SS_MCH-M
- J1: footprint Connector_Dsub:DSUB-9_Male_Horizontal_P2.77x2.54mm_EdgePinOffset9.40mm -> DB9:DB9
- J10: footprint (none) -> 282837-2:TE_282837-2
- J2, J4: footprint digikey-footprints:Term_Block_1x6_P5mm -> footprints:CONN_6P-OSTTC_OST
- J5: footprint digikey-footprints:PinHeader_1x3_P2.54_Drill1.1mm -> 640456-3:TE_640456-3
- J8: footprint digikey-footprints:PinHeader_1x5_P2.5mm_Drill1.1mm -> B5B-XH-A_LF__SN_:JST_B5B-XH-A_LF__SN_
- R44: footprint (none) -> Resistor_SMD:R_0402_1005Metric
- R46, R66, R70: footprint (none) -> Resistor_SMD:R_0201_0603Metric
- U1: footprint digikey-footprints:TO-220-3 -> REG1117-3.3:SOT230P700X180-4N
Other:
- moved on the sheet: J2, R7, R8

Commit message: heatsink considered
Parts:
- R44: footprint Resistor_SMD:R_0402_1005Metric -> Resistor_SMD:R_0805_2012Metric_Pad1.20x1.40mm_HandSolder
- R46, R66, R70: footprint Resistor_SMD:R_0201_0603Metric -> Resistor_SMD:R_0805_2012Metric_Pad1.20x1.40mm_HandSolder
Changed lines of the file:
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@@
 			)
 		)
-		(property "Footprint" "Resistor_SMD:R_0201_0603Metric"
+		(property "Footprint" "Resistor_SMD:R_0805_2012Metric_Pad1.20x1.40mm_HandSolder"
 			(at 419.8265 308.6904 90)
 			(effects
@@
 			)
 		)
-		(property "Footprint" "Resistor_SMD:R_0201_0603Metric"
+		(property "Footprint" "Resistor_SMD:R_0805_2012Metric_Pad1.20x1.40mm_HandSolder"
 			(at 274.9446 275.1192 90)
 			(effects
@@
 					(size 1.27 1.27)
 				)
+				(hide yes)
 			)
 		)
@@
 			)
 		)
-		(property "Footprint" "Resistor_SMD:R_0402_1005Metric"
+		(property "Footprint" "Resistor_SMD:R_0805_2012Metric_Pad1.20x1.40mm_HandSolder"
 			(at 246.6738 311.2734 90)
 			(effects
@@
 			)
 		)
-		(property "Footprint" "Resistor_SMD:R_0201_0603Metric"
+		(property "Footprint" "Resistor_SMD:R_0805_2012Metric_Pad1.20x1.40mm_HandSolder"
 			(at 448.0973 272.5362 90)
 			(effects

Commit message: lasy update smd res
Parts:
- R12, R13, R2, R49, R50, R62: footprint Resistor_THT:R_Axial_DIN0414_L11.9mm_D4.5mm_P25.40mm_Horizontal -> Resistor_SMD:R_2512_6332Metric_Pad1.40x3.35mm_HandSolder
Changed lines of the file:
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@@
 			)
 		)
-		(property "Footprint" "Resistor_THT:R_Axial_DIN0414_L11.9mm_D4.5mm_P25.40mm_Horizontal"
+		(property "Footprint" "Resistor_SMD:R_2512_6332Metric_Pad1.40x3.35mm_HandSolder"
 			(at 215.7124 298.0086 90)
 			(effects
@@
 			)
 		)
-		(property "Footprint" "Resistor_THT:R_Axial_DIN0414_L11.9mm_D4.5mm_P25.40mm_Horizontal"
+		(property "Footprint" "Resistor_SMD:R_2512_6332Metric_Pad1.40x3.35mm_HandSolder"
 			(at 373.8085 294.727 90)
 			(effects
@@
 			)
 		)
-		(property "Footprint" "Resistor_THT:R_Axial_DIN0414_L11.9mm_D4.5mm_P25.40mm_Horizontal"
+		(property "Footprint" "Resistor_SMD:R_2512_6332Metric_Pad1.40x3.35mm_HandSolder"
 			(at 381.3965 294.9227 90)
 			(effects
@@
 			)
 		)
-		(property "Footprint" "Resistor_THT:R_Axial_DIN0414_L11.9mm_D4.5mm_P25.40mm_Horizontal"
+		(property "Footprint" "Resistor_SMD:R_2512_6332Metric_Pad1.40x3.35mm_HandSolder"
 			(at 208.2438 297.5057 90)
 			(effects
@@
 			)
 		)
-		(property "Footprint" "Resistor_THT:R_Axial_DIN0414_L11.9mm_D4.5mm_P25.40mm_Horizontal"
+		(property "Footprint" "Resistor_SMD:R_2512_6332Metric_Pad1.40x3.35mm_HandSolder"
 			(at 200.6558 297.31 90)
 			(effects
@@
 			)
 		)
-		(property "Footprint" "Resistor_THT:R_Axial_DIN0414_L11.9mm_D4.5mm_P25.40mm_Horizontal"
+		(property "Footprint" "Resistor_SMD:R_2512_6332Metric_Pad1.40x3.35mm_HandSolder"
 			(at 388.8651 295.4256 90)
 			(effects
