File: circuts/motordriver/motordriver.kicad_pcb (KiCad board)
At the start: 2 copper layers, 142 parts, among them IC1 PIC16F15243-I_SS, J11 RJ45, J4 M2_encoder, J6 M1_ encoder, J8 B5B-XH-A_LF__SN_, J9 regulator_en, Q1 IRFS4227, Q13 IRFS4227, Q18 IRFS4227, Q2 IRFS4227, Q26 IRFS4227, Q27 IRFS4227, Q3 IRFS4227, Q30 IRFS4227, Q31 IRFS4227, Q4 IRFS4227, U1 3.3v, U10 IR25602S, U2 UC3843, U3 IR25602S, U4 IR25602S, U6 LM7805CT_Obsolete, U7 CRE1S0505DC, U8 IR25602S, U9 UC3843B, Y1 XLH536025_000000I

Commit message: lay out
Parts:
- removed C10, C11, C8, C9: 100nf, Resistor_SMD:R_0805_2012Metric_Pad1.20x1.40mm_HandSolder
- removed C36, C40, C42, C6: C, Resistor_SMD:R_0805_2012Metric_Pad1.20x1.40mm_HandSolder
- removed C37, C41, C7: C_Polarized, Capacitor_THT:CP_Radial_D8.0mm_P5.00mm
- removed D1, D11, D12, D21, D26, D27, D3, D30, D31, D34, D36, D37, D38, D39, D40, D41, D42, D43, D44, D6, D7, D8: 1N4004-T_NRND, Diode_SMD:D_SOD-123
- removed D28: 5.6v zener, Diode_SMD:D_SOD-123
- removed F1: 10 A, Diode_SMD:D_SOD-128
- removed J11: RJ45, Connector_RJ:RJ45_OST_PJ012-8P8CX_Vertical
- removed J6: M1_ encoder, digikey-footprints:Term_Block_1x4_P5mm
- removed J9: regulator_en, digikey-footprints:PinHeader_1x2_P2.54mm
- removed Q13, Q18, Q26, Q27, Q30, Q31: IRFS4227, Package_TO_SOT_SMD:TO-263-3_TabPin2
- removed R21: 330, Resistor_SMD:R_0805_2012Metric_Pad1.20x1.40mm_HandSolder
- removed R24: 56k, Resistor_SMD:R_0805_2012Metric_Pad1.20x1.40mm_HandSolder
- removed R28: 10, Resistor_SMD:R_0805_2012Metric_Pad1.20x1.40mm_HandSolder
- removed R29: 22, Resistor_SMD:R_0805_2012Metric_Pad1.20x1.40mm_HandSolder
- removed R31: 300K, Resistor_SMD:R_0805_2012Metric_Pad1.20x1.40mm_HandSolder
- removed R32, R33, R34: 0.3, Resistor_THT:R_Axial_DIN0414_L11.9mm_D4.5mm_P25.40mm_Horizontal
- removed U10, U4: IR25602S, Package_SO:SOIC-8_3.9x4.9mm_P1.27mm
- removed Y1: XLH536025_000000I, digikey-footprints:Oscillator_XLH536025.000000I
- removed ZD35: BZV55B4V7, Diode_SMD:D_MiniMELF
- added C24: 2uf, Resistor_SMD:R_0805_2012Metric_Pad1.20x1.40mm_HandSolder, F.Cu at (80.5, 66.0)
- added C43: 2uf, Resistor_SMD:R_0805_2012Metric_Pad1.20x1.40mm_HandSolder, F.Cu at (125.0, 104.3)
- added C44: 2uf, Resistor_SMD:R_0805_2012Metric_Pad1.20x1.40mm_HandSolder, F.Cu at (107.5, 54.3)
- added C47: 470uf, Capacitor_THT:CP_Radial_D8.0mm_P5.00mm, F.Cu at (87.0, 72.3)
- added C48: 2uf, Resistor_SMD:R_0805_2012Metric_Pad1.20x1.40mm_HandSolder, F.Cu at (92.0, 40.8)
- added J1: DE9_Plug, DB9:DB9, F.Cu at (160.9, 24.4)
- added J10: Power, 282837-2:TE_282837-2, F.Cu at (70.5, 115.8)
- added J2: OSTTC060162, footprints:CONN_6P-OSTTC_OST, F.Cu at (106.5, 26.8)
- added J3: XT60-M, XT60-M:AMASS_XT60-M, F.Cu at (70.0, 69.4)
- added J5: 640456-3, 640456-3:TE_640456-3, F.Cu at (69.5, 100.8)
- added Q10: MMBTA06, Package_TO_SOT_SMD:SOT-23, F.Cu at (148.0, 106.4)
- added Q5: MMBTA06, Package_TO_SOT_SMD:SOT-23, F.Cu at (161.9, 106.6)
- added Q8: IRFS4227, Package_TO_SOT_SMD:TO-263-3_TabPin2, F.Cu at (169.2, 55.2)
- added Q9: MMBTA06, Package_TO_SOT_SMD:SOT-23, F.Cu at (154.9, 106.6)
- added R27: 10k, Resistor_SMD:R_0805_2012Metric_Pad1.20x1.40mm_HandSolder, F.Cu at (183.0, 27.2)
- added R37: 10k, Resistor_SMD:R_0805_2012Metric_Pad1.20x1.40mm_HandSolder, F.Cu at (195.0, 27.4)
- added R38: 100k, Resistor_SMD:R_0805_2012Metric_Pad1.20x1.40mm_HandSolder, F.Cu at (208.5, 31.0)
- added R39: 56k, Resistor_SMD:R_0805_2012Metric_Pad1.20x1.40mm_HandSolder, F.Cu at (208.5, 34.0)
- added R40: 470, Resistor_SMD:R_0805_2012Metric_Pad1.20x1.40mm_HandSolder, F.Cu at (208.5, 36.9)
- added R41: 2k, Resistor_SMD:R_0805_2012Metric_Pad1.20x1.40mm_HandSolder, F.Cu at (208.5, 39.9)
- added R42: 2k, Resistor_SMD:R_0805_2012Metric_Pad1.20x1.40mm_HandSolder, F.Cu at (208.5, 42.8)
- added R43: 470, Resistor_SMD:R_0805_2012Metric_Pad1.20x1.40mm_HandSolder, F.Cu at (208.5, 45.8)
- added R44: 56k, Resistor_SMD:R_0402_1005Metric, F.Cu at (82.5, 116.6)
- added R45: 56k, Resistor_SMD:R_0805_2012Metric_Pad1.20x1.40mm_HandSolder, F.Cu at (188.5, 24.9)
- added R46: 2.2k, Resistor_SMD:R_0201_0603Metric, F.Cu at (79.8, 116.4)
- added R47: 2k, Resistor_SMD:R_0805_2012Metric_Pad1.20x1.40mm_HandSolder, F.Cu at (188.5, 27.8)
- added R48: 330, Resistor_SMD:R_0805_2012Metric_Pad1.20x1.40mm_HandSolder, F.Cu at (188.5, 30.8)
- added R49: 0.3, Resistor_THT:R_Axial_DIN0414_L11.9mm_D4.5mm_P25.40mm_Horizontal, F.Cu at (144.2, 126.8)
- added R50: 0.3, Resistor_THT:R_Axial_DIN0414_L11.9mm_D4.5mm_P25.40mm_Horizontal, F.Cu at (179.2, 125.8)
- added R61: 470, Resistor_SMD:R_0805_2012Metric_Pad1.20x1.40mm_HandSolder, F.Cu at (188.5, 33.7)
- added R62: 0.3, Resistor_THT:R_Axial_DIN0414_L11.9mm_D4.5mm_P25.40mm_Horizontal, F.Cu at (208.2, 126.3)
- added R63: 10k, Resistor_SMD:R_0805_2012Metric_Pad1.20x1.40mm_HandSolder, F.Cu at (188.5, 36.6)
- added R64: 10k, Resistor_SMD:R_0805_2012Metric_Pad1.20x1.40mm_HandSolder, F.Cu at (200.5, 28.0)
- added R65: 56k, Resistor_SMD:R_0805_2012Metric_Pad1.20x1.40mm_HandSolder, F.Cu at (200.5, 30.9)
- added R66: 56k, Resistor_SMD:R_0201_0603Metric, F.Cu at (79.8, 118.2)
- added R67: 2k, Resistor_SMD:R_0805_2012Metric_Pad1.20x1.40mm_HandSolder, F.Cu at (200.5, 33.9)
- added R68: 100k, Resistor_SMD:R_0805_2012Metric_Pad1.20x1.40mm_HandSolder, F.Cu at (200.5, 36.9)
- added R69: 56k, Resistor_SMD:R_0805_2012Metric_Pad1.20x1.40mm_HandSolder, F.Cu at (200.5, 39.8)
- added R70: 5k, Resistor_SMD:R_0201_0603Metric, F.Cu at (86.7, 119.9)
- added R71: 220, Resistor_SMD:R_0805_2012Metric_Pad1.20x1.40mm_HandSolder, F.Cu at (200.5, 42.8)
- added R72: 2k, Resistor_SMD:R_0805_2012Metric_Pad1.20x1.40mm_HandSolder, F.Cu at (200.5, 45.7)
- added R73: 10k, Resistor_SMD:R_0805_2012Metric_Pad1.20x1.40mm_HandSolder, F.Cu at (154.9, 88.5)
- added R74: 220, Resistor_SMD:R_0805_2012Metric_Pad1.20x1.40mm_HandSolder, F.Cu at (152.0, 88.5)
- added R75: 220, Resistor_SMD:R_0805_2012Metric_Pad1.20x1.40mm_HandSolder, F.Cu at (149.1, 88.5)
- added R76: 2k, Resistor_SMD:R_0805_2012Metric_Pad1.20x1.40mm_HandSolder, F.Cu at (146.1, 88.5)
- added R77: 5.1k, Resistor_SMD:R_0805_2012Metric_Pad1.20x1.40mm_HandSolder, F.Cu at (143.2, 88.5)
- added R78: 5.1k, Resistor_SMD:R_0805_2012Metric_Pad1.20x1.40mm_HandSolder, F.Cu at (155.0, 94.5)
- added R79: 5.1k, Resistor_SMD:R_0805_2012Metric_Pad1.20x1.40mm_HandSolder, F.Cu at (152.1, 94.5)
- added R80: 5.1k, Resistor_SMD:R_0805_2012Metric_Pad1.20x1.40mm_HandSolder, F.Cu at (149.1, 94.5)
- added R81: 5.1k, Resistor_SMD:R_0805_2012Metric_Pad1.20x1.40mm_HandSolder, F.Cu at (146.2, 94.5)
- added R82: 5.1k, Resistor_SMD:R_0805_2012Metric_Pad1.20x1.40mm_HandSolder, F.Cu at (143.2, 94.5)
- added U5: LM358DT, Package_SO:SOIC-8_3.9x4.9mm_P1.27mm, F.Cu at (129.0, 92.9)
- added ZD2: BZV55B4V7, Diode_SMD:D_MiniMELF, F.Cu at (136.8, 107.1)
- C1, C4: value C -> 2uf
- C12: footprint Resistor_SMD:R_0805_2012Metric_Pad1.20x1.40mm_HandSolder -> Capacitor_THT:CP_Radial_D8.0mm_P5.00mm
- C23: value 1nf -> 100pf
- C38: value 1nf -> 100nf
- C5: value C_Polarized -> 2uf; footprint Capacitor_THT:CP_Radial_D8.0mm_P5.00mm -> Resistor_SMD:R_0805_2012Metric_Pad1.20x1.40mm_HandSolder
- IC1: footprint SOP65P780X200-20N:SOP65P780X200-20N -> pic16f15243:SSOP20_SS_MCH-M
- J4: value M2_encoder -> OSTTC060162; footprint digikey-footprints:Term_Block_1x4_P5mm -> footprints:CONN_6P-OSTTC_OST
- J8: footprint digikey-footprints:PinHeader_1x5_P2.5mm_Drill1.1mm -> B5B-XH-A_LF__SN_:JST_B5B-XH-A_LF__SN_
- Q2, Q3, Q4: value IRFS4227 -> MMBTA06; footprint Package_TO_SOT_SMD:TO-263-3_TabPin2 -> Package_TO_SOT_SMD:SOT-23
- R1: value 10 -> 10k
- R14: value 100K -> 3.3k
- R15: value 300K -> 10k
- R16: value 22 -> 470
- R19: value 300K -> 100k
- R20: value 330 -> 200; footprint Resistor_SMD:R_0805_2012Metric_Pad1.20x1.40mm_HandSolder -> Resistor_THT:R_Bare_Metal_Element_L16.3mm_W4.8mm_P15.30mm
- R22, R25: value 10 -> 220
- R26, R35, R36, R4: value 10 -> 2k
- R30: value 100K -> 2k
- U1: footprint digikey-footprints:TO-220-3 -> REG1117-3.3:SOT230P700X180-4N
- U3, U8: value IR25602S -> BTS7960B; footprint Package_SO:SOIC-8_3.9x4.9mm_P1.27mm -> BTS7960B:DPAK127P1490X440-8N
- U6: value LM7805CT_Obsolete -> BTS7960B; footprint digikey-footprints:TO-220-3 -> BTS7960B:DPAK127P1490X440-8N
- U7: value CRE1S0505DC -> BTS7960B; footprint Converter_DCDC:Converter_DCDC_Murata_CRE1xxxxxxDC_THT -> BTS7960B:DPAK127P1490X440-8N
- U9: value UC3843B -> LM358DT
- ZD11: footprint Diode_SMD:D_MiniMELF -> Capacitor_THT:CP_Radial_D10.0mm_P5.00mm_P7.50mm
- ZD20: value BZV55B4V7 -> 3.3v
- moved R20 190.7 mm to (221.5, 37.5), turned to 90 degrees
- moved R2 181.0 mm to (221.5, 69.5), turned to 90 degrees
- moved R12 175.2 mm to (221.5, 99.0), turned to 90 degrees
- moved R13 168.8 mm to (220.5, 130.5), turned to 90 degrees
- moved U3 140.3 mm to (188.5, 78.5), turned to 90 degrees
- moved R26 139.3 mm to (183.0, 24.3), turned to 0 degrees
- moved R6 129.7 mm to (126.0, 34.3)
- moved R7 129.4 mm to (121.5, 34.3), turned to 0 degrees
- moved R8 124.9 mm to (117.0, 34.3)
- moved R4 120.8 mm to (166.5, 117.5), turned to 180 degrees
- moved R3 118.9 mm to (137.0, 43.3)
- moved U6 116.5 mm to (210.5, 76.3), turned to 90 degrees
- moved J4 115.9 mm to (70.0, 53.8), turned to 90 degrees
- moved U2 115.2 mm to (161.5, 72.9)
- moved C2 112.1 mm to (130.5, 46.0)
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Connections:
- C1 pad 1: M2_R -> Net-(D4-A)
- C1 pad 2: M2_L -> GND
- C12 pad 1: voltge_sen -> Net-(ZD11-K)
- C19 pad 1: motor_power -> HV
- C2 pad 1: Net-(U2-VREF) -> 5v+
- C20 pad 1: motor_power -> HV
- C21 pad 1: motor_power -> HV
- C22 pad 2: motor_power -> HV
- C23 pad 1: PGC -> PWM
- C27 pad 1: M1_L -> HV
- C27 pad 2: M1_R -> GND
- C3 pad 1: Net-(U2-RC) -> Net-(C3-Pad1)
- C31 pad 1: M2_L -> HV
- C31 pad 2: M2_R -> GND
- C33 pad 2: VDD -> Net-(U1-OUT)
- C34 pad 2: 5v+ -> Net-(U1-IN)
- C35 pad 1: Net-(U9-VREF) -> GND
- C35 pad 2: GND -> HV
- C38 pad 1: Net-(U9-RC) -> 3.3V
- C39 pad 1: PGD -> 3.3V
- C4 pad 1: M2_L -> Net-(C4-Pad1)
- C4 pad 2: Net-(D7-K) -> Net-(C4-Pad2)
- C5 pad 1: Net-(D7-K) -> Net-(D5-A)
- C5 pad 2: M2_L -> GND
- D10 pad 1: 12v -> HV
- D18 pad 2: 5v+ -> 3.3v
- D19 pad 2: motor_power -> HV
- D2 pad 1: motor_power -> CS
- D2 pad 2: M2_L -> Net-(D2-A)
- D25 pad 2: cs2 -> Net-(D25-A)
- D4 pad 1: M2_R -> Net-(D4-K)
- D4 pad 2: Net-(D25-K) -> Net-(D4-A)
- D5 pad 1: Net-(D5-K) -> CS
- D5 pad 2: motor_power -> Net-(D5-A)
- D9 pad 1: 12v -> HV
- F2 pad 1: 5v+ -> Net-(U1-OUT)
- F2 pad 2: 5v block -> 3.3V
- F3 pad 1: 12v -> HV
- F3 pad 2: 12v block -> HVblock
- IC1 pad 1: VDD -> 3.3V
- IC1 pad 12: M2_S2 -> Net-(IC1-RB5)
- IC1 pad 15: M1_S2 -> Net-(IC1-RC1)
- IC1 pad 2: Net-(IC1-RA5) -> B1
- IC1 pad 4: B1 -> Mcler
- J4 pad 2: B2 -> 5v+
- J4 pad 3: A2 -> B1
- J4 pad 4: 5v+ -> A1
- J8 pad 1: B1 -> Mcler
- J8 pad 2: VDD -> 3.3V
- Q1 pad 1: Net-(D21-A) -> Net-(Q1-G)
- Q1 pad 3: cs2 -> Net-(D25-A)
- Q2 pad 1: Net-(D37-A) -> Net-(Q2-B)
- Q2 pad 2: Net-(D38-A) -> GND
- Q2 pad 3: cs1 -> M2_D1
- Q3 pad 1: Net-(D1-A) -> Net-(Q3-B)
- Q3 pad 2: M2_L -> Net-(D25-A)
- Q3 pad 3: Net-(D25-K) -> Net-(Q1-G)
- Q4 pad 1: Net-(D30-A) -> Net-(Q4-B)
- Q4 pad 2: M2_R -> GND
- Q4 pad 3: Net-(D25-K) -> INH2
- R1 pad 1: Net-(D31-A) -> 3.3V
- R1 pad 2: Net-(D31-K) -> M2_D1
- R12 pad 1: cs2 -> Net-(D25-A)
- R13 pad 1: cs2 -> Net-(D25-A)
- R14 pad 1: PGC -> PWM
- R15 pad 1: Net-(D21-K) -> Net-(U2-OUT)
- R15 pad 2: PGC -> PWM
- R16 pad 1: Net-(D21-A) -> PWM
- R16 pad 2: Net-(D21-K) -> INH2
- R17 pad 2: VDD -> 3.3V
- R18 pad 1: voltge_sen -> Net-(ZD11-K)
- R19 pad 1: motor_power -> HV
- R19 pad 2: voltge_sen -> Net-(ZD11-K)
- R2 pad 1: cs2 -> Net-(D25-A)
- R20 pad 1: M2_current_sen -> Net-(U1-IN)
- R20 pad 2: cs2 -> HV
- R22 pad 1: Net-(D11-K) -> M2_S1
- R22 pad 2: Net-(D11-A) -> Net-(Q2-B)
- R25 pad 1: Net-(D30-K) -> PGD
- R25 pad 2: Net-(D30-A) -> Net-(Q3-B)
- R26 pad 1: Net-(D12-K) -> PGC
- R26 pad 2: Net-(D12-A) -> Net-(J5-Pad3)
- R3 pad 1: Net-(U2-RC) -> Net-(C3-Pad1)
- R3 pad 2: Net-(U2-VREF) -> 5v+
- R30 pad 1: PGD -> Net-(U3-SR)
- R35 pad 1: Net-(D42-K) -> Net-(U7-SR)
- R35 pad 2: Net-(D42-A) -> GND
- R36 pad 1: Net-(D43-K) -> Net-(IC1-RB5)
- R36 pad 2: Net-(D43-A) -> error 2
- R4 pad 1: Net-(D1-A) -> HV
- R4 pad 2: Net-(D1-K) -> Net-(Q1-G)
- R5 pad 1: VDD -> 3.3V
- R6 pad 1: VDD -> 3.3V
- R7 pad 1: VDD -> 3.3V
- R8 pad 1: VDD -> 3.3V
- R9 pad 2: VDD -> 3.3V
- U1 pad 1: 5v+ -> Net-(U1-IN)
- U1 pad 3: VDD -> Net-(U1-OUT)
- U2 pad 1: Motor2_OFF -> Net-(U2-COMP)
- U2 pad 3: cs2 -> CS
- U2 pad 6: Net-(D21-K) -> Net-(U2-OUT)
- U2 pad 7: VCC -> HV
- U2 pad 8: Net-(U2-VREF) -> 5v+
- U3 pad 1: VCC -> Net-(D25-K)
- U3 pad 2: M2_S2 -> M2_D1
- U3 pad 3: M2_S1 -> INH2
- U3 pad 4: Net-(D25-K) -> M2_R
- U3 pad 5: Net-(D1-K) -> Net-(U3-SR)
- U3 pad 6: M2_L -> error 2
- U3 pad 7: Net-(D12-A) -> HV
- U3 pad 8: Net-(D7-K) -> M2_R
- U6 pad 1: Net-(U6-IN) -> Net-(D4-K)
- U6 pad 2: GND -> M1_D1
- U6 pad 3: 5v+ -> INH1
- U7 pad 1: GND -> Net-(D25-K)
- U7 pad 4: motor_power -> M2_L
- U7 pad 5: VCC -> Net-(U7-SR)
- U7 pad 7: GND -> HV
- U8 pad 1: VCC -> Net-(D4-K)
- U8 pad 3: M1_S2 -> INH1
- U8 pad 4: Net-(D38-A) -> M1_L
- U8 pad 5: Net-(D31-K) -> Net-(U8-SR)
- U8 pad 6: M1_L -> error 1
- U8 pad 7: Net-(D11-A) -> HV
- U8 pad 8: Net-(D5-K) -> M1_L
- U9 pad 1: Motor1_OFF -> Net-(R66-Pad1)
- U9 pad 2: GND -> Net-(C4-Pad2)
- U9 pad 3: cs1 -> Net-(C4-Pad1)
- U9 pad 4: Net-(U9-RC) -> GND
- U9 pad 5: GND -> (no net)
- U9 pad 6: Net-(D37-K) -> (no net)
- U9 pad 7: VCC -> (no net)
- U9 pad 8: Net-(U9-VREF) -> HV
- ZD11 pad 1: voltge_sen -> Net-(ZD11-K)
- ZD20 pad 1: PGC -> PWM
Routing:
- net GND: track 0.00 -> 1054.2 mm, vias 0 -> 13
- net HV: track 0.00 -> 528.9 mm, vias 0 -> 10
- net 3.3V: track 0.00 -> 365.4 mm, vias 0 -> 8
- net M2_R: track 0.00 -> 355.3 mm, vias 0 -> 5
- net Net-(D25-A): track 0.00 -> 317.9 mm, vias 0 -> 6
- net 5v+: track 0.00 -> 309.7 mm, vias 0 -> 6
- net Net-(D4-A): track 0.00 -> 254.4 mm, vias 0 -> 7
- net Net-(C24-Pad2): track 0.00 -> 243.9 mm, vias 0 -> 7
- net Net-(C4-Pad2): track 0.00 -> 242.9 mm, vias 0 -> 5
- net M1_L: track 0.00 -> 242.3 mm, vias 0 -> 3
- net Net-(R38-Pad2): track 0.00 -> 221.2 mm, vias 0 -> 6
- net HVblock: track 0.00 -> 215.2 mm, vias 0 -> 1
- net Net-(R66-Pad1): track 0.00 -> 208.6 mm, vias 0 -> 3
- net PWM: track 0.00 -> 208.1 mm, vias 0 -> 3
- net Net-(U1-IN): track 0.00 -> 207.8 mm, vias 0 -> 7
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
Commit message: edited lay out
Parts:
- moved U9 13.8 mm to (197.0, 58.0), turned to -90 degrees
Routing:
- net M2_R: track 355.3 -> 129.6 mm, vias 5 -> 1
- net HV: track 528.9 -> 491.2 mm, vias 10 -> 15
- net M2_S1: track 138.7 -> 172.1 mm, vias 4 -> 3
- net Net-(Q2-B): track 46.6 -> 76.9 mm
- net Net-(C4-Pad2): track 242.9 -> 217.3 mm, vias 5 -> 4
- net Net-(D25-A): track 317.9 -> 292.5 mm, vias 6 -> 4
- net SCL: track 164.0 -> 139.1 mm, vias 4 -> 2
- net M2_L: track 190.8 -> 166.1 mm, vias 9 -> 5
- net Net-(D18-K): track 90.3 -> 66.1 mm
- net M1_R: track 191.3 -> 213.8 mm, vias 5 -> 1
- net PGC: track 195.9 -> 175.5 mm
- net 3.3V: track 365.4 -> 345.3 mm, vias 8 -> 9
- net M1_L: track 242.3 -> 224.3 mm, vias 3 -> 4
- net Net-(U1-IN): track 207.8 -> 190.8 mm, vias 7 -> 3
- net Net-(Q5-C): track 96.2 -> 112.8 mm, vias 3 -> 4
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
Commit message: heatsink considered
Parts:
- added REF1: MountingHole_3.2mm_M3, MountingHole:MountingHole_3.2mm_M3, F.Cu at (208.0, 90.5)
- added REF2: MountingHole_3.2mm_M3, MountingHole:MountingHole_3.2mm_M3, F.Cu at (158.5, 114.5)
- R44: footprint Resistor_SMD:R_0402_1005Metric -> Resistor_SMD:R_0805_2012Metric_Pad1.20x1.40mm_HandSolder
- R46, R66, R70: footprint Resistor_SMD:R_0201_0603Metric -> Resistor_SMD:R_0805_2012Metric_Pad1.20x1.40mm_HandSolder
- moved R26 107.0 mm to (90.5, 78.0)
- moved R27 107.0 mm to (90.5, 81.0)
- moved R30 107.0 mm to (90.5, 84.0)
- moved R35 107.0 mm to (90.5, 86.9)
- moved R36 107.0 mm to (90.5, 89.8)
- moved R37 101.7 mm to (127.5, 103.5), turned to 90 degrees
- moved R45 95.8 mm to (108.5, 77.5)
- moved R47 95.8 mm to (108.5, 80.5)
- moved R48 95.8 mm to (108.5, 83.4)
- moved R63 95.8 mm to (108.5, 89.3)
- moved R61 95.8 mm to (108.5, 86.3)
- moved Q4 34.2 mm to (135.5, 115.5)
- moved U2 27.7 mm to (138.0, 87.6), turned to 180 degrees
- moved D10 25.8 mm to (150.2, 96.0)
- moved D17 25.8 mm to (150.2, 99.4)
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Routing:
- net Net-(C24-Pad2): track 257.3 -> 108.8 mm, vias 7 -> 3
- net Net-(J5-Pad3): track 201.9 -> 73.6 mm
- net Net-(C24-Pad1): track 198.3 -> 73.4 mm, vias 3 -> 2
- net Net-(IC1-RB5): track 142.7 -> 21.9 mm
- net PGC: track 175.5 -> 62.4 mm
- net voltge_sen: track 151.7 -> 47.7 mm
- net error 1: track 104.8 -> 200.0 mm, vias 4 -> 6
- net error 2: track 111.7 -> 181.1 mm, vias 5 -> 4
- net Net-(ZD11-K): track 172.9 -> 113.8 mm, vias 2 -> 4
- net Net-(U3-SR): track 72.4 -> 125.4 mm, vias 2 -> 4
- net M2_S1: track 172.1 -> 122.5 mm
- net Net-(U1-IN): track 190.8 -> 236.3 mm
- net 5v+: track 305.9 -> 264.7 mm, vias 6 -> 5
- net Net-(D25-A): track 292.5 -> 328.4 mm, vias 4 -> 7
- net Net-(U7-SR): track 83.3 -> 118.0 mm
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Other:
- board outline added: 178 x 116.5 mm
- board text added: "ENG / Ahmed siddiq"
- board text added: "ENG / Mohamed aldesoky"
- board text added: "If you can read this, you have voided your warranty"

Commit message: lasy update smd res
Parts:
- R12, R13, R2, R49, R50, R62: footprint Resistor_THT:R_Axial_DIN0414_L11.9mm_D4.5mm_P25.40mm_Horizontal -> Resistor_SMD:R_2512_6332Metric_Pad1.40x3.35mm_HandSolder
- moved R1 100.6 mm to (173.0, 133.0), turned to -90 degrees
- moved R44 92.0 mm to (169.5, 133.0), turned to -90 degrees
- moved R66 86.3 mm to (166.2, 133.2), turned to -90 degrees
- moved R70 81.3 mm to (163.7, 133.2), turned to -90 degrees
- moved R46 76.3 mm to (161.2, 133.2), turned to -90 degrees
- moved R45 74.4 mm to (158.0, 133.0), turned to 90 degrees
- moved C4 65.1 mm to (186.5, 63.5), turned to 90 degrees
- moved C28 56.4 mm to (93.5, 131.0), turned to -90 degrees
- moved C29 54.9 mm to (90.5, 131.0), turned to -90 degrees
- moved C30 53.7 mm to (87.6, 131.0), turned to -90 degrees
- moved U5 53.1 mm to (165.5, 123.5), turned to 180 degrees
- moved C43 51.4 mm to (87.5, 76.0), turned to 180 degrees
- moved C33 49.9 mm to (85.4, 131.0), turned to -90 degrees
- moved C26 49.5 mm to (67.5, 60.0), turned to 180 degrees
- moved C34 49.4 mm to (82.5, 131.0), turned to -90 degrees
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Routing:
- net GND: track 1021.8 -> 0.00 mm, vias 7 -> 0
- net HV: track 502.4 -> 0.00 mm, vias 10 -> 0
- net 3.3V: track 341.6 -> 0.00 mm, vias 8 -> 0
- net Net-(D25-A): track 328.4 -> 0.00 mm, vias 7 -> 0
- net 5v+: track 264.7 -> 0.00 mm, vias 5 -> 0
- net Net-(D4-A): track 262.3 -> 0.00 mm, vias 6 -> 0
- net Net-(U1-IN): track 236.3 -> 0.00 mm, vias 3 -> 0
- net M1_L: track 218.0 -> 0.00 mm, vias 3 -> 0
- net HVblock: track 213.9 -> 0.00 mm, vias 1 -> 0
- net M1_R: track 212.9 -> 0.00 mm, vias 7 -> 0
- net PWM: track 209.2 -> 0.00 mm, vias 3 -> 0
- net Net-(R38-Pad2): track 208.6 -> 0.00 mm, vias 3 -> 0
- net Net-(C4-Pad2): track 206.0 -> 0.00 mm, vias 4 -> 0
- net Net-(R66-Pad1): track 204.6 -> 0.00 mm, vias 4 -> 0
- net error 1: track 200.0 -> 0.00 mm, vias 6 -> 0
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Other:
- board outline removed
- board text removed: "ENG / Ahmed siddiq"
- board text removed: "ENG / Mohamed aldesoky"
- board text removed: "If you can read this, you have voided your warranty"

Commit message: layout
Parts:
- moved R2 137.7 mm to (88.5, 132.5), turned to 180 degrees
- moved R13 130.4 mm to (88.5, 120.5), turned to 180 degrees
- moved R12 129.6 mm to (88.5, 126.5), turned to 180 degrees
- moved R62 121.4 mm to (78.0, 132.5)
- moved R50 93.2 mm to (78.0, 126.5)
- moved R64 84.0 mm to (126.5, 95.8)
- moved R65 84.0 mm to (126.5, 98.7)
- moved R67 84.0 mm to (126.5, 101.7)
- moved R68 84.0 mm to (126.5, 104.6)
- moved R69 84.0 mm to (126.5, 107.5)
- moved R71 84.0 mm to (126.5, 110.5)
- moved R72 84.0 mm to (126.5, 113.5)
- moved R20 65.0 mm to (152.5, 52.8)
- moved R49 60.8 mm to (78.0, 120.5)
- moved R35 59.8 mm to (131.5, 114.0)
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Other:
- board outline added: 130 x 111 mm
