File: circuts/SBC/SBC.kicad_sch (KiCad schematic)
At the start: 139 parts, among them IC1 PIC16F15243-I_SS, J1 DE9_Plug, J10 Power, J2 OSTTC060162, J3 XT60-M, J4 OSTTC060162, J5 640456-3, J8 B5B-XH-A_LF__SN_, Q1 IRFS4227, Q10 MMBTA06, Q2 MMBTA06, Q3 MMBTA06, Q4 MMBTA06, Q5 MMBTA06, Q8 IRFS4227, Q9 MMBTA06, U1 3.3v, U2 UC3843, U3 BTS7960B, U5 LM358DT, U6 BTS7960B, U7 BTS7960B, U8 BTS7960B, U9 LM358DT

Commit message: start
Parts:
- added C6, C7, C8: 2uf, Resistor_SMD:R_0805_2012Metric_Pad1.20x1.40mm_HandSolder, symbol Device:C
Connections:
- net M1_L: now also C6.2
- net M1_R: now also C6.1
- net M2_L: now also C7.2, C8.2
- net M2_R: now also C7.1, C8.1
Other:
- moved on the sheet: C31

Commit message: 29-6 siddyq
Parts:
- removed U1: 3.3v, REG1117-3.3:SOT230P700X180-4N, symbol dk_PMIC-Voltage-Regulators-Linear:LM7805CT_Obsolete
- added C10, C41, C42, C45, C56, C57: 2uf, Capacitor_SMD:C_0805_2012Metric_Pad1.18x1.45mm_HandSolder, symbol Device:C
- added C10, C11, C9: 1nf, Capacitor_SMD:C_0805_2012Metric_Pad1.18x1.45mm_HandSolder, symbol Device:C
- added C11, C36, C37, C40, C58, C59, C71, C72, C73, C74: 100nf, Capacitor_SMD:C_0805_2012Metric_Pad1.18x1.45mm_HandSolder, symbol Device:C
- added C46, C49, C50: 100uf, Capacitor_SMD:CP_Elec_4x4.5, symbol Device:C_Polarized
- added C51, C52, C53: 470uf, Capacitor_SMD:CP_Elec_4x4.5, symbol Device:C_Polarized
- added C54, C55, C9: 1000uf, Capacitor_SMD:CP_Elec_4x4.5, symbol Device:C_Polarized
- added C60, C61, C65, C66: 100nf, Resistor_SMD:R_0805_2012Metric_Pad1.20x1.40mm_HandSolder, symbol Device:C
- added C62, C63, C64: C, Capacitor_SMD:C_0805_2012Metric_Pad1.18x1.45mm_HandSolder, symbol Device:C
- added C67, C68, C69, C70: 1nf, Resistor_SMD:R_0805_2012Metric_Pad1.20x1.40mm_HandSolder, symbol Device:C
- added D1: 20v zener, Diode_SMD:D_MiniMELF, symbol Diode:BZV55B5V6
- added D1, D11, D3, D6: LED, Capacitor_SMD:C_0603_1608Metric_Pad1.08x0.95mm_HandSolder, symbol Device:LED
- added D13, D14, D15, D16: SMAJ6.5A, Diode_SMD:D_SMF, symbol Diode:SMAJ6.5A
- added D3: 5.6v zener, Diode_SMD:D_MiniMELF, symbol Diode:BZV55B5V6
- added D6, D8: BZV55B3V3, Diode_SMD:D_MiniMELF, symbol Diode:BZV55B3V3
- added D7 (x2), D8: 1N4004-T_NRND, digikey-footprints:DO-41, symbol dk_Diodes-Rectifiers-Single:1N4004-T_NRND
- added F1, F4: 1A, Capacitor_SMD:C_0805_2012Metric_Pad1.18x1.45mm_HandSolder, symbol Device:Fuse
- added F1: 1A, Capacitor_SMD:C_0603_1608Metric_Pad1.08x0.95mm_HandSolder, symbol Device:Fuse
- added F5, F6: 1A, Diode_SMD:D_SOD-128, symbol Device:Fuse
- added J11: metal detect, TerminalBlock:TerminalBlock_bornier-3_P5.08mm, symbol Connector:Screw_Terminal_01x03
- added J12: 12v Power, symbol Connector:Screw_Terminal_01x02
- added J13: 5v Power, symbol Connector:Screw_Terminal_01x02
- added J6: Conn_02x04_Odd_Even, Connector_PinHeader_2.54mm:PinHeader_2x04_P2.54mm_Vertical, symbol Connector_Generic:Conn_02x04_Odd_Even
- added J6: grip_con, Connector_Dsub:DSUB-9_Male_Horizontal_P2.77x2.54mm_EdgePinOffset9.40mm, symbol Connector:DE9_Plug
- added J7: motor_con, Connector_Dsub:DSUB-9_Male_Horizontal_P2.77x2.54mm_EdgePinOffset9.40mm, symbol Connector:DE9_Plug
- added J9: buzzer, symbol Connector:Screw_Terminal_01x02
- added Q6: FDS4559, Package_SO:SOIC-8_3.9x4.9mm_P1.27mm, symbol Transistor_FET:FDS4559
- added Q7: BC817, Package_TO_SOT_SMD:SOT-23, symbol Transistor_BJT:BC817
- added R21, R28, R29: 1k, Capacitor_SMD:C_0805_2012Metric_Pad1.18x1.45mm_HandSolder, symbol Device:R
- added R24: 5k, Capacitor_SMD:C_0805_2012Metric_Pad1.18x1.45mm_HandSolder, symbol Device:R
- added R31: 220, Capacitor_SMD:C_0805_2012Metric_Pad1.18x1.45mm_HandSolder, symbol Device:R
- added R32: 330, Capacitor_SMD:C_0805_2012Metric_Pad1.18x1.45mm_HandSolder, symbol Device:R
- added R33, R34: 10k, Resistor_SMD:R_1206_3216Metric_Pad1.30x1.75mm_HandSolder, symbol Device:R
- added R51, R56: 200, Resistor_THT:R_Bare_Metal_Element_L16.3mm_W4.8mm_P15.30mm, symbol Device:R_US
- added R52, R53, R54, R55: 10k, Resistor_SMD:R_0805_2012Metric_Pad1.20x1.40mm_HandSolder, symbol Device:R
- added R57, R58, R59, R60: 5.1k, Resistor_SMD:R_0805_2012Metric_Pad1.20x1.40mm_HandSolder, symbol Device:R_US
- added R83, R84, R85, R87, R89: 10k, Resistor_SMD:R_0805_2012Metric_Pad1.20x1.40mm_HandSolder, symbol Device:R_US
- added R86, R88, R90: 1k, Resistor_SMD:R_0805_2012Metric_Pad1.20x1.40mm_HandSolder, symbol Device:R_US
- added SW1, SW2, SW3, SW4: SW_Push, symbol Switch:SW_Push
- added U1, U12: AMS1117-3.3, Package_TO_SOT_SMD:SOT-223-3_TabPin2, symbol Regulator_Linear:AMS1117-3.3
- added U10: ESP32-DEVKIT-V1, ESP32-DEVKIT-V1:MODULE_ESP32_DEVKIT_V1, symbol ESP32-DEVKIT-V1:ESP32-DEVKIT-V1
- added U11: AMS1117-5.0, Package_TO_SOT_SMD:SOT-223-3_TabPin2, symbol Regulator_Linear:AMS1117-5.0
- added U4: ~, Connector_PinHeader_2.54mm:PinHeader_1x08_P2.54mm_Vertical, symbol New_Library_0:IMU_10DOF_
- added ZD1, ZD3: BZV55B4V7, Diode_SMD:D_MiniMELF, symbol Diode:BZV55B4V7
- R6: value 10k -> 1k
Connections:
- net HVblock is gone; now on net HV: F3.2, J1.1, J1.6, J10.1 (Pin_1), J3.P (POS)
- net 3.3V: now also R5.2, C10.1, C11.1, C11.1, C40.1, C45.1, C50.1, C53.1, C9.1, D14.1 (A1), F6.2, J6.2 (Pin_2), J6.4, J7.4, R31.2, R33.1, R34.2, R52.2, R53.2, R54.2, R55.2, R83.1, R84.1, R85.2, R87.2, R89.2, U10.1 (3V3), U4. (VCC), ZD3.1 (K); no longer R5.1, R6.1
- net 5v+: now also C10.1, C37.1, C42.1, C49.1, C52.1, C55.1, C57.1, C59.1, C63.1, D13.1 (A1), D16.1 (A1), D3.1 (K), D8.1 (K), F4.1, F5.2, J6.3, J7.3, R32.2, U10.30 (VIN), U4. (VCC), ZD1.1 (K)
- net A1: now also R60.1; no longer J4.4, R6.2
- net A2: now also R58.1; no longer J2.4, R8.2
- net B1: now also R59.2; no longer J4.3, R5.2
- net B2: now also R57.2; no longer J2.3, R7.2
- net CS: now also J6.3 (Pin_3)
- net GND: now also C10.2, C10.2, C11.2, C11.2, C36.2, C37.2, C40.2, C41.2, C42.2, C45.2, C46.2, C49.2, C50.2, C51.2, C52.2, C53.2, C54.2, C55.2, C56.2, C57.2, C58.2, C59.2, C60.1, C61.1, C62.2, C63.2, C65.1, C66.1, C67.2, C68.2, C69.2, C70.2, C71.2, C72.2, C73.2, C74.2, C9.2, C9.2, D1.2 (A), D11.1 (K), D13.2 (A2), D14.2 (A2), D15.2 (A2), D16.2 (A2), D3.1 (K), D3.2 (A), D6.1 (K), D6.2 (A), D7.2 (A), D8.2 (A), D8.2 (A), J11.3 (Pin_3), J12.2 (Pin_2), J13.2 (Pin_2), J6.1 (Pin_1), J6.2, J6.7, J7.2, J7.7, Q6.7 (D), Q6.8 (D), Q7.2 (E), SW1.2, SW2.2, SW3.2, SW4.2, U1.1 (GND), U10.2 (GND), U10.29 (GND), U11.1 (GND), U12.1 (GND), U4. (VCC), ZD1.2 (A), ZD3.2 (A)
- net HV: now also C36.1, C41.1, C46.1, C51.1, C54.1, C56.1, C58.1, C62.1, C9.1, D1.1 (K), D15.1 (A1), D7.1 (K), F1.1, J11.1 (Pin_1), J6.1, J6.6, J7.1, J7.6, R29.2, R51.2, R56.2
- net SCL: now also J6.5, J7.5, R52.1, R53.1, U4. (VCC)
- net SDA: now also J6.9, J7.9, R33.2, R54.1, R55.1, U10.11 (D21), U4. (VCC)
- net at C33.2, F2.1: now also U12.2 (VO)
- net at C34.2, R20.1: now also U12.3 (VI)
- new net: F1.2, J12.1 (Pin_1)
- new net: Q6.2 (G), Q7.3 (C), R24.2
- new net: C69.1, J4.4, R60.2, R84.2
- new net: R90.1, SW4.1
- new net: Q7.1 (B), R28.2
- new net: C65.2, R56.1, U1.3 (VI)
- new net: R86.1, SW2.1
- new net: F1.2, J9.1 (Pin_1)
- new net: C61.2, F5.1, U11.2 (VO)
- new net: C60.2, R51.1, U11.3 (VI)
- new net: D6.2 (A), R31.1
- new net: C70.1, J4.3, R59.1, R83.2
- new net: D3.2 (A), R29.1
- new net: R6.1, SW1.1
- new net: D1.2 (A), R21.2
- new net: C67.1, J2.4, R58.2, R8.2
- new net: R88.1, SW3.1
- new net: C66.2, F6.1, U1.2 (VO)
- new net: C68.1, J2.3, R57.1, R7.2
- new net: D11.2 (A), R32.1
- new net 12v: C64.1, D7.1 (K), F1.1, R21.1, R24.1
- new net 5v block: F4.2, J13.1 (Pin_1)
- new net CSN: J6.4 (Pin_4)
- new net Data_ready: U10.15 (D23), U4. (VCC)
- new net FSYC: U10.24 (D26), U4. (VCC)
- new net IRQ: J6.8 (Pin_8), U10.25 (D27)
- new net MISO: J6.7 (Pin_7)
- new net MOSI: J6.6 (Pin_6)
- new net RST: J6.8, J7.8
- new net SCK: J6.5 (Pin_5)
- new net SDL: R34.1, U10.14 (D22)
- new net SW1: C72.1, R85.1, R86.2, U10.21 (D32)
- new net SW2: C73.1, R87.1, R88.2, U10.22 (D33)
- new net SW3: C74.1, R89.1, R90.2, U10.20 (D35)
- new net SW4: C71.1, R5.1, R6.2, U10.19 (D34)
- new net buzz: D6.1 (K), R28.1, U10.5 (D4)
- new net buzzing_gnd: C64.2, D1.1 (K), D7.2 (A), J9.2 (Pin_2), Q6.1 (S)
- new net care: U10.12 (RX0), U10.13 (TX0), U10.27 (D12), U10.3 (D15), U10.4 (D2)
- new net detect: D8.1 (K), J11.2 (Pin_2), U10.8 (D5)
- new net int_a: U10.23 (D25), U4. (VCC)
Other:
- moved on the sheet: C15, C16, C17, C18, C19, C20, C21, C22, C25, C26, C27, C28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
