File: circuts/SBC/SBC.kicad_sch (KiCad schematic)
At the start: 246 parts, among them IC1 PIC16F15243-I_SS, J1 640456-3, J10 motor_con, J11 buzzer, J12 metal detect, J13 12v Power, J14 5v Power, J2 B5B-XH-A_LF__SN_, J3 Power, J4 DE9_Plug, J5 OSTTC060162, J6 XT60-M, J7 OSTTC060162, J8 grip_con, J9 Conn_02x04_Odd_Even, Q1 MMBTA06, Q10 BC817, Q2 MMBTA06, Q3 MMBTA06, Q4 IRFS4227, Q5 MMBTA06, Q6 MMBTA06, Q7 MMBTA06, Q8 IRFS4227, Q9 FDS4559, SW1 SW_Push, SW2 SW_Push, SW3 SW_Push, SW4 SW_Push, U1 UC3843, U10 ESP32-DEVKIT-V1, U12 AMS1117-5.0, U2 BTS7960B, U3 BTS7960B, U4 LM358DT, U5 AMS1117-3.3, U6 AMS1117-3.3, U7 BTS7960B, U8 BTS7960B, U9 LM358DT

Commit message: siddyq 7-5 finshing befor ly mod
Parts:
- removed F2: 1A, Diode_SMD:D_SOD-128, symbol Device:Fuse
- removed U12: AMS1117-5.0, Package_TO_SOT_SMD:SOT-223-3_TabPin2, symbol Regulator_Linear:AMS1117-5.0
- added C78: 1nf, Capacitor_SMD:C_0805_2012Metric_Pad1.18x1.45mm_HandSolder, symbol Device:C
- added C79, C83: 100nf, Capacitor_SMD:C_0805_2012Metric_Pad1.18x1.45mm_HandSolder, symbol Device:C
- added C80: 2uf, Capacitor_SMD:C_0805_2012Metric_Pad1.18x1.45mm_HandSolder, symbol Device:C
- added C81: 470uf, Capacitor_SMD:CP_Elec_4x4.5, symbol Device:C_Polarized
- added C82, C89: 2uf, Resistor_SMD:R_0805_2012Metric_Pad1.20x1.40mm_HandSolder, symbol Device:C
- added C84, C85, C86: 100nf, Resistor_SMD:R_0805_2012Metric_Pad1.20x1.40mm_HandSolder, symbol Device:C
- added C87: 1nf, Resistor_SMD:R_0805_2012Metric_Pad1.20x1.40mm_HandSolder, symbol Device:C
- added C88: 470uf, Capacitor_THT:CP_Radial_D8.0mm_P5.00mm, symbol Device:C_Polarized
- added D25, D26, D27, D28: 1N4004-T_NRND, Diode_SMD:D_SOD-123, symbol dk_Diodes-Rectifiers-Single:1N4004-T_NRND
- added J15: Barrel_Jack_MountingPin, Connector_BarrelJack:BarrelJack_GCT_DCJ200-10-A_Horizontal, symbol Connector:Barrel_Jack_MountingPin
- added R100, R106: 200, Resistor_THT:R_Bare_Metal_Element_L16.3mm_W4.8mm_P15.30mm, symbol Device:R_US
- added R101, R103, R91, R92, R93, R94, R95, R96, R97, R98: 10k, Resistor_SMD:R_0805_2012Metric_Pad1.20x1.40mm_HandSolder, symbol Device:R_US
- added R102: 1k, Resistor_SMD:R_0805_2012Metric_Pad1.20x1.40mm_HandSolder, symbol Device:R_US
- added R104: 1ohm, Resistor_SMD:R_0805_2012Metric_Pad1.20x1.40mm_HandSolder, symbol Device:R_US
- added R99: 2k, Resistor_SMD:R_0805_2012Metric_Pad1.20x1.40mm_HandSolder, symbol Device:R_US
- added SW5: SW_Push, BUTT-2:SW_BUTT-2, symbol Switch:SW_Push
- added U12, U13: L7805, Package_TO_SOT_SMD:TO-252-2, symbol Regulator_Linear:L7805
- added ZD10, ZD8: 3.3v, Diode_SMD:D_MiniMELF, symbol Diode:BZV55B4V7
- added ZD11: BZV55B4V7, Diode_SMD:D_MiniMELF, symbol Diode:BZV55B4V7
- added ZD9: 20v, Diode_SMD:D_MiniMELF, symbol Diode:BZV55B4V7
- R42: value 200 -> 10
- U6: value AMS1117-3.3 -> step down moudl
Connections:
- net 3.3V: now also R101.2; no longer D16.1 (A1), R39.1, R8.1, U10.1 (3V3), ZD6.1 (K)
- net 5v+: now also R39.1, R40.2, R8.1, R104.2, ZD11.1 (K); no longer C1.1, R4.2, R9.1, U1.8 (VREF)
- net GND: now also C78.2, C79.2, C80.2, C81.2, C82.1, C83.2, C84.1, C85.2, C86.1, C87.2, C88.2, C89.1, J15.2, J15.MP (MountPin), SW5.2, U12.2 (GND), U13.2 (GND), ZD11.2 (A), ZD9.2 (A)
- net HV: now also D26.1 (K), D28.2 (A), R100.2, R103.2, ZD10.1 (K), ZD8.1 (K); no longer F3.1, R15.1, R40.2, R42.2, R47.1, U1.7 (VCC), U4.8 (VCC+), U9.8 (VCC+)
- net INH1: now also R95.2, R97.1; no longer U7.3 (INH), U8.3 (INH)
- net INH2: now also R91.1, R93.2; no longer U2.3 (INH), U3.3 (INH)
- net M1_D1: now also R98.1; no longer U7.2 (IN)
- net M1_S1: now also R96.2; no longer U8.2 (IN)
- net M2_D1: now also R92.1; no longer U2.2 (IN)
- net M2_S1: now also R94.2; no longer U3.2 (IN)
- net SW4: now also C83.1, R101.1, R102.2
- net at F6.2, J13.1 (Pin_1): now also J15.1
- net at C31.2, R42.1, U6.3 (VI): now also ZD9.1 (K)
- net at C74.2, F4.1: now also U13.3 (OUT)
- net at C73.2, R88.1: now also U13.1 (IN)
- net at C33.2, U6.2 (VO): now also C82.2, D25.2 (A)
- net 12v renamed buzzing_vcc
- new net: C78.1, C79.1, C80.1, C81.1, D16.1 (A1), U10.1 (3V3)
- new net: R103.1, U1.7 (VCC), ZD10.2 (A)
- new net: D27.1 (K), R106.2
- new net: D27.2 (A), D28.1 (K)
- new net: R100.1, R42.2, ZD8.2 (A)
- new net: R96.1, U8.2 (IN)
- new net: R93.1, U3.3 (INH)
- new net: C84.2, R106.1, U12.1 (IN)
- new net: R98.2, U7.2 (IN)
- new net: R97.2, U7.3 (INH)
- new net: D26.2 (A), F3.1
- new net: R95.1, U8.3 (INH)
- new net: R94.1, U3.2 (IN)
- new net: R92.2, U2.2 (IN)
- new net: R91.2, U2.3 (INH)
- new net: C86.2, R104.1, U12.3 (OUT)
- new net: D25.1 (K), R99.1
- new net: R102.1, SW5.1
- new net 9v+: C85.1, C87.1, C88.1, C89.2, R15.1, R47.1, R99.2, U4.8 (VCC+), U9.8 (VCC+), ZD6.1 (K)
- new net s5v+: C1.1, R4.2, R9.1, U1.8 (VREF)
Other:
- moved on the sheet: C30, C31, C32, C33, C69, C70, C71, C72, C73, C74, D10, D11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

Commit message: Signed-off-by: ahmedsiddyq <morganalpop@gmail.com>
Parts:
- removed C6, C7: 2uf, Resistor_SMD:R_0805_2012Metric_Pad1.20x1.40mm_HandSolder, symbol Device:C
- removed C83: 100nf, Capacitor_SMD:C_0805_2012Metric_Pad1.18x1.45mm_HandSolder, symbol Device:C
- removed F1: 1A, Diode_SMD:D_SOD-128, symbol Device:Fuse
- added C90: 100nf, Capacitor_SMD:C_0805_2012Metric_Pad1.18x1.45mm_HandSolder, symbol Device:C
- added C91: 33uf, Capacitor_THT:CP_Radial_D4.0mm_P1.50mm, symbol Device:C
- added D29, D30, D31, D32, D37, D38, D39, D40, D41, D42: 1N5822, Diode_THT:D_DO-201AD_P15.24mm_Horizontal, symbol Diode:1N5822
- added D33, D34, D35, D36: SMAJ26A, Diode_THT:D_DO-201AE_P15.24mm_Horizontal, symbol Diode:SMAJ6.5A
- added D43, D44: LED, Diode_SMD:D_SOD-123, symbol Device:LED
- added R105: 1ohm, Resistor_SMD:R_0805_2012Metric_Pad1.20x1.40mm_HandSolder, symbol Device:R_US
- added R107: 10k, Resistor_SMD:R_0805_2012Metric_Pad1.20x1.40mm_HandSolder, symbol Device:R_US
- added R108, R109, R110: 1k, Resistor_SMD:R_0805_2012Metric_Pad1.20x1.40mm_HandSolder, symbol Device:R_US
- added R111: 1.5k, Resistor_SMD:R_0805_2012Metric_Pad1.20x1.40mm_HandSolder, symbol Device:R_US
- added R112: 330, Resistor_SMD:R_0805_2012Metric_Pad1.20x1.40mm_HandSolder, symbol Device:R_US
- added SW6: rst, BUTT-2:SW_BUTT-2, symbol Switch:SW_Push
- added SW7: SW_Push, BUTT-2:SW_BUTT-2, symbol Switch:SW_Push
- added ZD12: BZV55B4V7, Capacitor_THT:CP_Radial_D10.0mm_P5.00mm_P7.50mm, symbol Diode:BZV55B4V7
- added ZD13, ZD14, ZD15, ZD16, ZD17, ZD18, ZD19, ZD20, ZD21, ZD22: 3.3v, Diode_SMD:D_MiniMELF, symbol Diode:BZV55B4V7
- C12: value 2uf -> 33uf; footprint Resistor_SMD:R_0805_2012Metric_Pad1.20x1.40mm_HandSolder -> Capacitor_THT:CP_Radial_D4.0mm_P1.50mm
- R10: value 10k -> 2.2k
- R101: value 10k -> 1ohm op*
- R102: value 1k -> 1ohm
- R11: value 3.3k -> 470
- R99: value 2k -> 1ohm
Connections:
- net RST is gone; now on net Mcler: J10.8, J8.8
- net buzzing_vcc is gone; now on net HV: C77.1, D23.1 (K), F5.1, R72.1, R73.1
- net 3.3V: now also R101.1, R105.2, R107.2; no longer R101.2, U11. (VCC)
- net 5v+: now also R102.1, D44.2 (A), R109.2, R110.2; no longer U11. (VCC)
- net 9v+: now also D28.2 (A), D43.2 (A)
- net A1: now also ZD20.1 (K)
- net A2: now also ZD22.1 (K)
- net B1: now also ZD19.1 (K)
- net B2: now also ZD21.1 (K)
- net GND: now also Q9.1 (S), C90.2, D30.2 (A), D31.2 (A), D37.2 (A), D39.2 (A), R111.2, R112.2, SW6.2, ZD13.2 (A), ZD14.2 (A), ZD15.2 (A), ZD16.2 (A), ZD17.2 (A), ZD18.2 (A), ZD19.2 (A), ZD20.2 (A), ZD21.2 (A), ZD22.2 (A); no longer Q9.7 (D), Q9.8 (D), SW5.2
- net HV: now also D29.1 (K), D32.1 (K), D38.1 (K), D40.1 (K), ZD12.1 (K); no longer D28.2 (A)
- net M1_L: now also D31.1 (K), D32.2 (A), D33.2 (A2)
- net M1_R: now also D29.2 (A), D30.1 (K), D34.2 (A2)
- net M1_S1: now also ZD15.1 (K)
- net M2_L: now also C91.2, D35.2 (A2), D39.1 (K), D40.2 (A)
- net M2_R: now also C91.1, D36.2 (A2), D37.1 (K), D38.2 (A)
- net M2_S1: now also ZD14.1 (K)
- net Mcler: now also J4.8, U10.26 (D14), C90.1, R107.1, R108.2
- net Motor1_OFF: now also ZD16.1 (K)
- net Motor2_OFF: now also ZD13.1 (K)
- net SCL: now also ZD18.1 (K); no longer J10.5, R89.1, U11. (VCC)
- net SDA: now also ZD17.1 (K); no longer J10.9, R90.1, U11. (VCC)
- net SW4: no longer R101.1, R102.2
- net buzzing_gnd: now also Q9.7 (D), Q9.8 (D); no longer Q9.1 (S)
- net at C32.2, U5.2 (VO): now also R105.1
- net at C14.1, D2.2 (A), Q3.2 (E)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: now also D42.2 (A)
- net SDL2: now reaches U10.10 (D19)
- net SDL2: now also U10.9 (D18)
- net at C34.1, D6.2 (A), Q7.2 (E)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: now also D41.2 (A)
- net at D2.1 (K), Q4.2 (D), U2.1 (GND)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: now also D42.1 (K)
- net at D6.1 (K), Q8.2 (D), U7.1 (GND)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: now also D41.1 (K)
- net at C73.2, R88.1, U13.1 (IN): now also ZD12.2 (A)
- net tst1: now reaches R97.2, U7.3 (INH)
- net tst1: now also SW5.1
- net tst2: now reaches R91.2, U2.3 (INH)
- net tst2: now also SW7.1
- new net: D44.1 (K), R112.1
- new net: R108.1, SW6.1
- new net: D43.1 (K), R111.1
- new net: R110.1, SW5.2
- new net: D33.1 (A1), D34.1 (A1)
- new net: D35.1 (A1), D36.1 (A1)
- new net: R101.2, U11. (VCC)
- new net: R102.2, U11. (VCC)
- new net: R109.1, SW7.2
- new net SCL2: J10.5, R89.1, U11. (VCC)
- new net SDA2: J10.9, R90.1, U11. (VCC)
Other:
- moved on the sheet: C11, C12, C13, C16, C17, C18, C19, C20, C23, C24, C25, C26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

Commit message: LAST EDIT AT 7-6
Changed lines of the file:
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@@
 	(wire
 		(pts
-			(xy 937.5532 144.3674) (xy 937.5532 141.3588)
+			(xy 937.5532 144.3674) (xy 937.5532 141.9604)
 		)
 		(stroke
@@
 	(wire
 		(pts
-			(xy 937.5532 141.3588) (xy 940.2575 141.3588)
+			(xy 937.5532 141.9604) (xy 940.6688 141.9604)
 		)
 		(stroke
@@
 	(global_label "3.3V"
 		(shape input)
-		(at 940.2575 141.3588 0)
+		(at 940.6688 141.9604 0)
 		(fields_autoplaced yes)
 		(effects
@@
 		)
 		(property "Intersheetrefs" "${INTERSHEET_REFS}"
-			(at 947.3551 141.3588 0)
+			(at 947.7664 141.9604 0)
 			(effects
 				(font

Commit message: sidyq 7-8 using curren amp design
Parts:
- removed J12: metal detect, TerminalBlock:TerminalBlock_bornier-3_P5.08mm, symbol Connector:Screw_Terminal_01x03
- removed R22, R51: 0.3, Resistor_SMD:R_2512_6332Metric_Pad1.40x3.35mm_HandSolder, symbol Device:R_US
- added C6: 470uf, Capacitor_THT:CP_Radial_D8.0mm_P5.00mm, symbol Device:C_Polarized
- added D45: 1N4004-T_NRND, Diode_SMD:D_SOD-123, symbol dk_Diodes-Rectifiers-Single:1N4004-T_NRND
- added D50, D52: L_LED, Diode_SMD:D_SOD-123, symbol Device:LED
- added D51, D53: R_LED, Diode_SMD:D_SOD-123, symbol Device:LED
- added J12: Screw_Terminal_01x04, symbol Connector:Screw_Terminal_01x04
- added R113: 1ohm op*, Resistor_SMD:R_0805_2012Metric_Pad1.20x1.40mm_HandSolder, symbol Device:R_US
- added R114: 220, Capacitor_SMD:C_0805_2012Metric_Pad1.18x1.45mm_HandSolder, symbol Device:R
- added R115, R116: 1.5k, Resistor_SMD:R_0805_2012Metric_Pad1.20x1.40mm_HandSolder, symbol Device:R_US
- added R117: 220, Resistor_SMD:R_0805_2012Metric_Pad1.20x1.40mm_HandSolder, symbol Device:R_US
- added ZD23, ZD24, ZD25, ZD26, ZD27, ZD28, ZD29, ZD30: 3.3v, Diode_SMD:D_MiniMELF, symbol Diode:BZV55B4V7
- R44: value 470 -> 220
Connections:
- net 3.3V: now also R113.1
- net 5v+: now also D45.2 (A)
- net GND: now also C6.2, J12.4 (Pin_4), ZD23.2 (A), ZD24.2 (A), ZD25.2 (A), ZD26.2 (A), ZD27.2 (A), ZD28.2 (A), ZD29.2 (A), ZD30.2 (A)
- net HV: now also C6.1, R114.1, R117.1
- net M1_L: now also D50.2 (A), D51.1 (K)
- net M1_R: now also R115.2
- net M2_L: now also D52.2 (A), D53.1 (K)
- net M2_R: now also R116.2
- net SDA2: now also U10.10 (D19)
- net SDL2: no longer U10.10 (D19)
- net detect: now also J12.3 (Pin_3)
- net tst1: now also R95.1, U8.3 (INH), ZD27.1 (K), ZD30.1 (K)
- net tst2: now also R93.1, U3.3 (INH), ZD23.1 (K), ZD26.1 (K)
- net at C78.1, C79.1, C80.1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: now also R113.2
- net FRQ: now reaches U10.28 (D13)
- net FRQ: now also J12.2 (Pin_2)
- net at R96.1, U8.2 (IN): now also ZD29.1 (K)
- net at R98.2, U7.2 (IN): now also ZD28.1 (K)
- net at R94.1, U3.2 (IN): now also ZD25.1 (K)
- net at R92.2, U2.2 (IN): now also ZD24.1 (K)
- new net: D45.1 (K), R114.2
- new net: J12.1 (Pin_1), R117.2
- new net: D52.1 (K), D53.2 (A), R116.1
- new net: D50.1 (K), D51.2 (A), R115.1
Other:
- moved on the sheet: C37, C76, C77, D17, D20, D22, D23, D24, F5, F7, J10, J11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

Commit message: 7-8 start layouting
Parts:
- removed R44: 220, Resistor_SMD:R_0805_2012Metric_Pad1.20x1.40mm_HandSolder, symbol Device:R_US
- removed R45: 5.1k, Resistor_SMD:R_0805_2012Metric_Pad1.20x1.40mm_HandSolder, symbol Device:R_US
- added C7, C83, C92, C93: 100nf, Resistor_SMD:R_0805_2012Metric_Pad1.20x1.40mm_HandSolder, symbol Device:C
- added D46, D47, D48, D49, D54, D55, D56: 1N4004-T_NRND, Diode_SMD:D_SOD-123, symbol dk_Diodes-Rectifiers-Single:1N4004-T_NRND
- added R118, R22: 2.2k, Resistor_SMD:R_0805_2012Metric_Pad1.20x1.40mm_HandSolder, symbol Device:R_US
- added R119: 220, Resistor_SMD:R_0805_2012Metric_Pad1.20x1.40mm_HandSolder, symbol Device:R_US
- added R120: 5.1k, Resistor_SMD:R_0805_2012Metric_Pad1.20x1.40mm_HandSolder, symbol Device:R_US
- added R51: 470, Resistor_SMD:R_0805_2012Metric_Pad1.20x1.40mm_HandSolder, symbol Device:R_US
- added RV1, RV2: R_Potentiometer, Potentiometer_SMD:Potentiometer_Vishay_TS53YJ_Vertical, symbol Device:R_Potentiometer
- added U14, U15: LM358DT, Package_SO:SOIC-8_3.9x4.9mm_P1.27mm, symbol dk_Linear-Amplifiers-Instrumentation-OP-Amps-Buffer-Amps:LM358DT
- C8: value 100pf -> 2pf
Connections:
- net 5v+: now also RV1.3, RV2.3
- net 9v+: now also U14.8 (VCC+), U15.8 (VCC+)
- net GND: now also C7.2, C83.2, C92.2, C93.2, R120.2, RV1.1, RV2.1, U14.4 (VCC-), U15.4 (VCC-)
- net M2_S1: now also D56.2 (A); no longer R3.1, ZD14.1 (K)
- net Motor2_OFF: now also D54.2 (A); no longer R2.1, ZD13.1 (K)
- net PGD: now also D46.2 (A), D48.2 (A); no longer R13.1
- net at Q3.1 (B), R13.2, R14.1: now also D47.1 (K)
- net at R29.1, R31.2, R33.2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: now also R22.2
- net at Q7.1 (B): now also D49.1 (K), R119.2, R120.1
- new net: C93.1, RV1.2, U14.2
- new net: D46.1 (K), R13.1
- new net: R118.2, U15.1
- new net: D56.1 (K), R3.1, ZD14.1 (K)
- new net: D54.1 (K), R2.1, ZD13.1 (K)
- new net: R51.2, U14.1
- new net: C92.1, RV2.2, U15.2
- new net: D48.1 (K), R119.1
- new net Current_limt1: C83.1, U15.3
- new net Current_limt2: C7.1, R22.1, U14.3
- new net kill1: D49.2 (A), R118.1
- new net kill2: D47.2 (A), R51.1
Other:
- moved on the sheet: C11, C12, C13, C3, C4, C5, C9, C91, D29, D30, D31, D32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

Commit message: 7-8 AT 2 PM LAYOUT EDITING
Parts:
- removed R89, R90: 10k, Resistor_SMD:R_0805_2012Metric_Pad1.20x1.40mm_HandSolder, symbol Device:R
- removed U6: step down moudl, Package_TO_SOT_SMD:SOT-223-3_TabPin2, symbol Regulator_Linear:AMS1117-3.3
- added R44, R45: 10k, Resistor_SMD:R_0805_2012Metric_Pad1.20x1.40mm_HandSolder, symbol Device:R
- added U14: L7809, Package_TO_SOT_THT:TO-220-3_Vertical, symbol Regulator_Linear:L7805
- added ZD31, ZD32, ZD33, ZD34: 3.3v, Diode_SMD:D_MiniMELF, symbol Diode:BZV55B4V7
- C1, C10, C11, C13, C14, C15, C16, C17, C18, C2, C3, C4, C5, C7, C8, C9: footprint Resistor_SMD:R_0805_2012Metric_Pad1.20x1.40mm_HandSolder -> Capacitor_SMD:C_0805_2012Metric_Pad1.18x1.45mm_HandSolder
- C12: footprint Capacitor_THT:CP_Radial_D4.0mm_P1.50mm -> Capacitor_THT:CP_Radial_D8.0mm_P5.00mm
- D1, D2, D21, D22, D23, D25, D26, D27, D28, D3, D4, D43, D44, D45, D46, D47, D48, D49, D5, D50, D51, D52, D53, D54, D55, D56, D6, D7, D9: footprint Diode_SMD:D_SOD-123 -> Diode_SMD:D_MiniMELF
- D10, D12, D13, D14: footprint Capacitor_SMD:C_0603_1608Metric_Pad1.08x0.95mm_HandSolder -> Diode_SMD:D_MiniMELF
- D15, D16, D17, D18: footprint Diode_SMD:D_SMF -> Diode_SMD:D_MiniMELF
- D29, D30, D31, D32, D37, D38, D39, D40, D41, D42: footprint Diode_THT:D_DO-201AD_P15.24mm_Horizontal -> Diode_SMD:D_MiniMELF
- D33, D34, D35, D36: footprint Diode_THT:D_DO-201AE_P15.24mm_Horizontal -> Diode_SMD:D_MiniMELF
- J10: value motor_con -> DE9_Plug
- J12: footprint (none) -> TerminalBlock:TerminalBlock_MaiXu_MX126-5.0-04P_1x04_P5.00mm
- J8: value grip_con -> DE9_Plug
- R100, R106, R40, R42, R88: footprint Resistor_THT:R_Bare_Metal_Element_L16.3mm_W4.8mm_P15.30mm -> Resistor_SMD:R_0805_2012Metric_Pad1.20x1.40mm_HandSolder
- R114, R72, R73, R74, R75, R76, R77: footprint Capacitor_SMD:C_0805_2012Metric_Pad1.18x1.45mm_HandSolder -> Resistor_SMD:R_0805_2012Metric_Pad1.20x1.40mm_HandSolder
- R78, R79: footprint Resistor_SMD:R_1206_3216Metric_Pad1.30x1.75mm_HandSolder -> Resistor_SMD:R_0805_2012Metric_Pad1.20x1.40mm_HandSolder
- SW1, SW2, SW3, SW4, SW5, SW6, SW7: footprint BUTT-2:SW_BUTT-2 -> Button_Switch_SMD:SW_DIP_SPSTx01_Slide_6.7x4.1mm_W6.73mm_P2.54mm_LowProfile_JPin
- ZD12, ZD4: footprint Capacitor_THT:CP_Radial_D10.0mm_P5.00mm_P7.50mm -> Diode_SMD:D_MiniMELF
- renumbered U14 to U4, U15 to U9
Connections:
- net 3.3V: now also R44.2, R45.2
- net Current_limt1: now also U9.5; no longer U9.3
- net Current_limt2: now also U4.5; no longer U4.3
- net Data_ready: now also U11.8 (DRDY); no longer U11. (VCC)
- net FSYC: now also U11.6 (FSSYNC); no longer U11. (VCC)
- net GND: now also J10.1, J10.5, J10.G1, J10.G2, J4.1, J4.5, J4.G1, J4.G2, J8.1, J8.5, J8.G1, J8.G2, U11.3 (GND), U14.2 (GND), ZD31.2 (A), ZD32.2 (A), ZD33.2 (A), ZD34.2 (A); no longer J10.2, J10.7, J4.2, J4.7, J8.2, J8.7, U11. (VCC)
- net HV: now also J10.2, J4.2, J8.2; no longer J10.1, J4.1, J8.1
- net Mcler: now also J10.7, J4.7, J8.7; no longer J10.8, J4.8, J8.8
- net SCL: now also J10.8, J4.8, J8.8, R44.1, ZD31.1 (K), ZD33.1 (K); no longer J4.5, J8.5
- net SCL2: now also U11.4 (SCL); no longer J10.5, U11. (VCC)
- net SDA: now also J10.9, R45.1, ZD32.1 (K), ZD34.1 (K)
- net SDA2: now also U11.5 (SDA); no longer J10.9, U11. (VCC)
- net int_a: now also U11.7 (INTA); no longer U11. (VCC)
- net at C93.1, RV1.2: now also U4.6; no longer U4.2
- net at R118.2: now also U9.7; no longer U9.1
- net at C31.2, R42.1, ZD9.1 (K): now also U14.1 (IN)
- net at R51.2: now also U4.7; no longer U4.1
- net at C92.1, RV2.2: now also U9.6; no longer U9.2
- net at C33.2, C82.2, D25.2 (A): now also U14.3 (OUT)
- net at R101.2: now also U11.2 (3.3V); no longer U11. (VCC)
- net at R102.2: now also U11.1 (VCC); no longer U11. (VCC)

Commit message: lay-out frist low side
Parts:
- added R89: 2.2k, Resistor_SMD:R_0805_2012Metric_Pad1.20x1.40mm_HandSolder, symbol Device:R_US
Connections:
- net at C92.1, U9.6: now also R89.1; no longer RV2.2
- new net: R89.2, RV2.2
Other:
- moved on the sheet: C1, C2, C8, J1, R1, R10, R103, R11, R4, R9, RV2, U1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

Commit message: 7-9 siddyq mid layout
Parts:
- removed D2, D6: 1N4004-T_NRND, Diode_SMD:D_MiniMELF, symbol dk_Diodes-Rectifiers-Single:1N4004-T_NRND
- removed R103: 10k, Resistor_SMD:R_0805_2012Metric_Pad1.20x1.40mm_HandSolder, symbol Device:R_US
- removed ZD10: 3.3v, Diode_SMD:D_MiniMELF, symbol Diode:BZV55B4V7
- added D57, D58, D59, D60, D61, D62, D63, D64, D65, D66, D67, D68: 1N4004-T_NRND, Diode_SMD:D_0603_1608Metric_Pad1.05x0.95mm_HandSolder, symbol dk_Diodes-Rectifiers-Single:1N4004-T_NRND
- added R121, R122, R123, R124, R125, R126, R127, R90: 10k, Resistor_SMD:R_0805_2012Metric_Pad1.20x1.40mm_HandSolder, symbol Device:R_US
- D3, D46, D47, D48, D49, D54, D55, D56, D7: footprint Diode_SMD:D_MiniMELF -> Diode_SMD:D_0603_1608Metric_Pad1.05x0.95mm_HandSolder
- R11: value 470 -> 220
- RV1, RV2: footprint Potentiometer_SMD:Potentiometer_Vishay_TS53YJ_Vertical -> Potentiometer_SMD:Potentiometer_Bourns_3214W_Vertical
- ZD13, ZD14, ZD15, ZD16, ZD17, ZD18, ZD19, ZD20, ZD21, ZD22, ZD23, ZD24, ZD25, ZD26, ZD27, ZD28, ZD29, ZD30, ZD31, ZD32, ZD33, ZD34: footprint Diode_SMD:D_MiniMELF -> Diode_SMD:D_SOD-123
Connections:
- net GND: now also R121.1, R122.2, R123.2, R124.2, R125.1, R126.1, R127.2, R90.1
- net HV: now also D66.2 (A), D67.2 (A), D68.2 (A); no longer R100.2, R27.1, ZD8.1 (K)
- net INH1: now also D61.2 (A), D63.2 (A); no longer R97.1
- net INH2: now also D59.2 (A), D65.2 (A); no longer R91.1, R93.2
- net M1_D1: now also D62.2 (A); no longer R98.1
- net M1_S1: now also D55.2 (A), D60.2 (A); no longer R34.1, R96.2, ZD15.1 (K)
- net M2_D1: now also D58.2 (A); no longer R92.1
- net M2_S1: now also D64.2 (A); no longer R94.2
- net Motor1_OFF: now also D57.2 (A); no longer R35.1, ZD16.1 (K)
- net tst1: now also R125.2, R126.2
- net tst2: now also R122.1, R90.2
- net at U1.7 (VCC): now also D68.1 (K)
- net at R94.1, U3.2 (IN), ZD25.1 (K): now also R123.1
- net at R96.1, U8.2 (IN), ZD29.1 (K): now also R127.1
- net at R92.2, U2.2 (IN), ZD24.1 (K): now also R121.2
- net at R98.2, U7.2 (IN), ZD28.1 (K): now also R124.1
- net at D55.1 (K): now also R34.1, ZD15.1 (K)
- new net: D60.1 (K), R96.2
- new net: D57.1 (K), R35.1, ZD16.1 (K)
- new net: D66.1 (K), R27.1
- new net: D65.1 (K), R93.2
- new net: D58.1 (K), R92.1
- new net: D62.1 (K), R98.1
- new net: D64.1 (K), R94.2
- new net: D67.1 (K), R100.2, ZD8.1 (K)
- new net: D63.1 (K), R97.1
- new net: D59.1 (K), R91.1
Other:
- moved on the sheet: D41, D42
