File: circuts/SBC/SBC.kicad_sch (KiCad schematic)
At the start: 371 parts, among them IC1 PIC16F15243-I_SS, J1 640456-3, J10 DE9_Plug, J11 buzzer, J12 Screw_Terminal_01x04, J13 12v Power, J14 5v Power, J15 Barrel_Jack_MountingPin, J2 B5B-XH-A_LF__SN_, J3 Power, J4 DE9_Plug, J5 OSTTC060162, J6 XT60-M, J7 OSTTC060162, J8 DE9_Plug, J9 Conn_02x04_Odd_Even, Q1 MMBTA06, Q10 BC817, Q2 MMBTA06, Q3 MMBTA06, Q4 IRFS4227, Q5 MMBTA06, Q6 MMBTA06, Q7 MMBTA06, Q8 IRFS4227, Q9 FDS4559, SW1 SW_Push, SW2 SW_Push, SW3 SW_Push, SW4 SW_Push, SW5 SW_Push, SW6 rst, SW7 SW_Push, U1 UC3843, U10 ESP32-DEVKIT-V1, U12 L7805, U13 L7805, U14 L7809, U2 BTS7960B, U3 BTS7960B, U4 LM358DT, U5 AMS1117-3.3, U7 BTS7960B, U8 BTS7960B, U9 LM358DT

Commit message: Signed-off-by: ahmedsiddyq <morganalpop@gmail.com>
Parts:
- removed R44, R45: 10k, Resistor_SMD:R_0805_2012Metric_Pad1.20x1.40mm_HandSolder, symbol Device:R
- added D6: 1N4004-T_NRND, Diode_SMD:D_0603_1608Metric_Pad1.05x0.95mm_HandSolder, symbol dk_Diodes-Rectifiers-Single:1N4004-T_NRND
Connections:
- net 3.3V: now also D6.1 (K); no longer J2.2
- net 9v+: now also C82.2
- net INH1: no longer R95.2
- net at D61.1 (K): now also R95.2
- net at C33.2, D25.2 (A), U14.3 (OUT): no longer C82.2
- new net: D6.2 (A), J2.2
Other:
- moved on the sheet: C82, D61

Commit message: almost ready
Parts:
- removed D19: 20v zener, Diode_SMD:D_MiniMELF, symbol Diode:BZV55B5V6
- removed D20: 5.6v zener, Diode_SMD:D_MiniMELF, symbol Diode:BZV55B5V6
- removed D21, D22, D23, D27, D28: 1N4004-T_NRND, Diode_SMD:D_MiniMELF, symbol dk_Diodes-Rectifiers-Single:1N4004-T_NRND
- removed F6: 1A, Capacitor_SMD:C_0603_1608Metric_Pad1.08x0.95mm_HandSolder, symbol Device:Fuse
- removed J12: Screw_Terminal_01x04, TerminalBlock:TerminalBlock_MaiXu_MX126-5.0-04P_1x04_P5.00mm, symbol Connector:Screw_Terminal_01x04
- removed J13: 12v Power, 282837-2:TE_282837-2, symbol Connector:Screw_Terminal_01x02
- removed Q9: FDS4559, Package_SO:SOIC-8_3.9x4.9mm_P1.27mm, symbol Transistor_FET:FDS4559
- removed R81, R82, R83: 10k, Resistor_SMD:R_0805_2012Metric_Pad1.20x1.40mm_HandSolder, symbol Device:R_US
- removed ZD32: 3.3v, Diode_SMD:D_SOD-123, symbol Diode:BZV55B4V7
- added C94: C, Capacitor_SMD:C_0805_2012Metric_Pad1.18x1.45mm_HandSolder, symbol Device:C
- added D19: SMAJ6.5A, Diode_SMD:D_MiniMELF, symbol Diode:SMAJ6.5A
- added D2: 1N4004-T_NRND, Diode_SMD:D_0603_1608Metric_Pad1.05x0.95mm_HandSolder, symbol dk_Diodes-Rectifiers-Single:1N4004-T_NRND
- added D20: 1N4004-T_NRND, Diode_SMD:D_MiniMELF, symbol dk_Diodes-Rectifiers-Single:1N4004-T_NRND
- added J13: Conn_01x04_Pin, Connector_PinSocket_2.54mm:PinSocket_1x04_P2.54mm_Vertical, symbol Connector:Conn_01x04_Pin
- added Q11: AO3400A, Package_TO_SOT_SMD:SOT-23_Handsoldering, symbol Transistor_FET:AO3400A
- added ZD10, ZD35, ZD36: BZV55B4V7, Diode_SMD:D_MiniMELF, symbol Diode:BZV55B4V7
- C11, C18, C2, C4, C45, C46, C47, C78: footprint Capacitor_SMD:C_0805_2012Metric_Pad1.18x1.45mm_HandSolder -> Capacitor_SMD:C_0201_0603Metric_Pad0.64x0.40mm_HandSolder
- C12: footprint Capacitor_THT:CP_Radial_D8.0mm_P5.00mm -> Capacitor_THT:CP_Radial_D4.0mm_P1.50mm
- C22: value 2uf -> 1nf; footprint Capacitor_THT:CP_Radial_D8.0mm_P5.00mm -> Capacitor_SMD:C_0201_0603Metric_Pad0.64x0.40mm_HandSolder
- C26, C36, C41, C42, C43, C44, C87: footprint Resistor_SMD:R_0805_2012Metric_Pad1.20x1.40mm_HandSolder -> Capacitor_SMD:C_0201_0603Metric_Pad0.64x0.40mm_HandSolder
- ZD31: value 3.3v -> BZV55B4V7; footprint Diode_SMD:D_SOD-123 -> Diode_SMD:D_MiniMELF
Connections:
- net SDL is gone; now on net SCL: R79.1, U10.14 (D22)
- net 5v+: now also ZD10.1 (K)
- net 9v+: now also D2.2 (A)
- net FRQ: now also J13.3 (Pin_3)
- net GND: now also J13.1 (Pin_1), Q11.2 (S), ZD10.2 (A), ZD35.2 (A), ZD36.2 (A)
- net HV: now also J15.1, D20.2 (A), ZD35.1 (K); no longer C77.1, F5.1, R114.1, R72.1, R73.1
- net SCL: now also ZD36.1 (K); no longer ZD31.1 (K)
- net SDA: now also ZD31.1 (K)
- net buzzing_gnd: now also C94.2, D19.2 (A2), Q11.3 (D)
- net detect: now also J13.2 (Pin_2)
- net at Q10.3 (C), R73.2: now also Q11.1 (G)
- net at R106.2: now also D2.1 (K)
- net at R117.2: now also J13.4 (Pin_4)
- new net buzzing_vcc: C77.1, C94.1, D19.1 (A1), D20.1 (K), F5.1, R114.1, R72.1, R73.1
Other:
- moved on the sheet: C70, C75, C76, D17, D18, R117, R85, SW2

Commit message: bom has been deplated
Parts:
- removed D8: 20v zener, Diode_SMD:D_MiniMELF, symbol Diode:BZV55B5V6
- removed D9: 1N4004-T_NRND, Diode_SMD:D_MiniMELF, symbol dk_Diodes-Rectifiers-Single:1N4004-T_NRND
- removed R78, R79: 10k, Resistor_SMD:R_0805_2012Metric_Pad1.20x1.40mm_HandSolder, symbol Device:R
- added C100, C102, C103, C99: 2uf, Resistor_SMD:R_0805_2012Metric_Pad1.20x1.40mm_HandSolder, symbol Device:C
- added C101, C104, C105, C98: 100nf, Capacitor_SMD:C_0805_2012Metric_Pad1.18x1.45mm_HandSolder, symbol Device:C
- added C95: 2uf, Capacitor_SMD:C_0805_2012Metric_Pad1.18x1.45mm_HandSolder, symbol Device:C
- added C96, C97: 470uf, Capacitor_THT:CP_Radial_D8.0mm_P5.00mm, symbol Device:C_Polarized
- added D21: BZV55B3V3, Diode_SMD:D_MiniMELF, symbol Diode:BZV55B3V3
- added D8: SMAJ6.5A, Diode_SMD:D_MiniMELF, symbol Diode:SMAJ6.5A
- C54: value 100uf -> 470uf; footprint Capacitor_SMD:CP_Elec_4x4.5 -> Capacitor_THT:CP_Radial_D8.0mm_P5.00mm
- C57: footprint Capacitor_SMD:CP_Elec_4x4.5 -> Capacitor_THT:CP_Radial_D8.0mm_P5.00mm
- C60: value 1000uf -> 470uf; footprint Capacitor_SMD:CP_Elec_4x4.5 -> Capacitor_THT:CP_Radial_D8.0mm_P5.00mm
Connections:
- net 3.3V: no longer C65.1
- net FRQ: now also D21.1 (K)
- net GND: now also C65.1, C95.1, D21.2 (A), D8.2 (A2); no longer C65.2
- net HV: now also C100.2, C101.1, C102.2, C103.2, C104.1, C105.1, C96.1, C97.1, C98.1, C99.2, D8.1 (A1)
- net at D42.1 (K), Q4.2 (D), U2.1 (GND)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: now also C100.1, C101.2, C102.1, C104.2, C96.2
- net at D41.1 (K), Q8.2 (D), U7.1 (GND)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: now also C103.1, C105.2, C97.2, C98.2, C99.1
- net at R101.2, U11.2 (3.3V): now also C65.2
- net at R102.2, U11.1 (VCC): now also C95.2
Other:
- moved on the sheet: C19, C23, C31, C33, C6, C65, D26, F3

Commit message: siddyq at fanaly
Parts:
- removed C24: 470uf, Capacitor_THT:CP_Radial_D8.0mm_P5.00mm, symbol Device:C_Polarized
- removed C55, C56: 100uf, Capacitor_SMD:CP_Elec_4x4.5, symbol Device:C_Polarized
- removed C58, C59: 470uf, Capacitor_SMD:CP_Elec_4x4.5, symbol Device:C_Polarized
- removed C61, C62: 1000uf, Capacitor_SMD:CP_Elec_4x4.5, symbol Device:C_Polarized
- added C24: 100nf, Resistor_SMD:R_0805_2012Metric_Pad1.20x1.40mm_HandSolder, symbol Device:C
Connections:
- net 3.3v: now also C35.1, C36.1, C37.1, C38.2, C47.1, C50.1, C53.1, C68.1, D6.1 (K), IC1.1 (VDD), J10.4, J4.4, J8.4, J9.2 (Pin_2), R101.1, R105.2, R107.2, R113.1, R64.1, R65.2, R67.1, R69.2, R70.2, R71.2, R76.2, R80.2, ZD5.1 (K), C24.1
- net GND: now also C24.2
- removed net 3.3V: C35.1, C36.1, C37.1, C38.2, C47.1, C50.1, C53.1, C68.1, D6.1 (K), IC1.1 (VDD), J10.4, J4.4, J8.4, J9.2 (Pin_2), R101.1, R105.2, R107.2, R113.1, R64.1, R65.2, R66.1, R67.1, R68.1, R69.2, R70.2, R71.2, R76.2, R80.2, ZD5.1 (K)
- new net: R66.1, R68.1
Other:
- moved on the sheet: D5

Commit message: siddyq has done almost done 7-25
Parts:
- removed C46: 1nf, Capacitor_SMD:C_0201_0603Metric_Pad0.64x0.40mm_HandSolder, symbol Device:C
- removed R108: 1k, Resistor_SMD:R_0805_2012Metric_Pad1.20x1.40mm_HandSolder, symbol Device:R_US
Connections:
- net SDL2 is gone; now on net FSYC: U10.9 (D18)
- net CS: no longer J9.3 (Pin_3)
- net FSYC: no longer U10.24 (D26)
- net IRQ: no longer J9.8 (Pin_8)
- net Mcler: now also SW6.1
- net SCL2: now also U10.6 (RX2)
- net SDA2: now also U10.7 (TX2); no longer U10.10 (D19)
- net int_a: now also U10.10 (D19); no longer U10.23 (D25)
- removed net care: U10.12 (RX0), U10.13 (TX0), U10.27 (D12), U10.3 (D15), U10.4 (D2)
- new net CSp: J9.3 (Pin_3)
- new net IRQo: J9.8 (Pin_8)
- new net care0: U10.12 (RX0), U10.13 (TX0)
- new net carei: U10.4 (D2)
- new net carett: U10.3 (D15)
- new net careuu: U10.27 (D12)
Other:
- moved on the sheet: J9

Commit message: siddyq test plane
Parts:
- added C46, C55, C56, C58: 2uf, Capacitor_SMD:C_0805_2012Metric_Pad1.18x1.45mm_HandSolder, symbol Device:C
Connections:
- net M1_L: now also C46.2, C55.2
- net M1_R: now also C46.1, C55.1
- net M2_L: now also C56.2, C58.2
- net M2_R: now also C56.1, C58.1
Other:
- moved on the sheet: C3, C4, C5, C91

Commit message: sidd	[[
Changed lines of the file:
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@@
 	)
 	(junction
-		(at 256.5363 294.7837)
-		(diameter 0)
-		(color 0 0 0 0)
-	)
-	(junction
 		(at 265.5612 360.5651)
 		(diameter 0)
@@
 	)
 	(junction
+		(at 256.5363 294.7837)
+		(diameter 0)
+		(color 0 0 0 0)
+	)
+	(junction
 		(at 1140.4687 167.8988)
 		(diameter 0)
@@
 	)
 	(junction
-		(at 256.5363 294.7856)
-		(diameter 0)
-		(color 0 0 0 0)
-	)
-	(junction
 		(at 199.2365 216.1011)
 		(diameter 0)
@@
 	(wire
 		(pts
-			(xy 256.5363 294.7837) (xy 256.5363 294.7856)
-		)
-		(stroke
-			(width 0)
-			(type default)
-		)
-	)
-	(wire
-		(pts
 			(xy 827.9226 301.6867) (xy 827.9226 305.849)
 		)
@@
 	(wire
 		(pts
-			(xy 1126.1723 64.1594) (xy 1126.1723 64.2093)
-		)
-		(stroke
-			(width 0)
-			(type default)
-		)
-	)
-	(wire
-		(pts
 			(xy 1020.5293 158.2207) (xy 1020.5293 158.2602)
 		)
@@
 	(wire
 		(pts
+			(xy 136.7317 65.4673) (xy 142.9349 65.4673)
+		)
+		(stroke
+			(width 0)
+			(type default)
+		)
+	)
+	(wire
+		(pts
 			(xy 431.8794 194.7861) (xy 423.5106 194.7861)
 		)
@@
 	(wire
 		(pts
-			(xy 1124.9023 64.1594) (xy 1126.1723 64.1594)
-		)
-		(stroke
-			(width 0)
-			(type default)
-		)
-	)
-	(wire
-		(pts
 			(xy 719.501 149.8547) (xy 719.501 150.9788)
 		)
@@
 	(wire
 		(pts
+			(xy 255.4448 294.7837) (xy 255.4448 294.7856)
+		)
+		(stroke
+			(width 0)
+			(type default)
+		)
+	)
+	(wire
+		(pts
 			(xy 232.1244 372.5313) (xy 239.4183 372.5313)
 		)
@@
 	(wire
 		(pts
-			(xy 255.4448 294.7856) (xy 256.5363 294.7856)
-		)
-		(stroke
-			(width 0)
-			(type default)
-		)
-	)
-	(wire
-		(pts
 			(xy 551.5075 257.521) (xy 544.0156 257.521)
 		)
@@
 	(wire
 		(pts
+			(xy 256.5363 294.7837) (xy 255.4448 294.7837)
+		)
+		(stroke
+			(width 0)
+			(type default)
+		)
+	)
+	(wire
+		(pts
 			(xy 1004.3842 45.2268) (xy 1004.3842 45.1919)
 		)
@@
 	(wire
 		(pts
-			(xy 541.3333 149.6842) (xy 544.9759 149.6842)
+			(xy 529.3545 150.6164) (xy 544.9759 150.6164)
 		)
 		(stroke
@@
 	(wire
 		(pts
-			(xy 256.5363 294.7856) (xy 256.5363 310.2574)
+			(xy 256.5363 294.7837) (xy 256.5363 310.2574)
 		)
 		(stroke
@@
 	(wire
 		(pts
-			(xy 255.8282 294.7837) (xy 256.5363 294.7837)
-		)
-		(stroke
-			(width 0)
-			(type default)
-		)
-	)
-	(wire
-		(pts
 			(xy 1138.3513 242.9176) (xy 1138.3513 251.299)
 		)
@@
 	(wire
 		(pts
-			(xy 544.9759 151.4654) (xy 544.9759 149.6842)
+			(xy 544.9759 151.4654) (xy 544.9759 150.6164)
 		)
 		(stroke
@@
 	)
 	(global_label "M2_S1"
-		(shape input)
+		(shape output)
 		(at 191.1949 62.9273 0)
 		(fields_autoplaced yes)
@@
 	)
 	(global_label "error 1"
-		(shape output)
+		(shape input)
 		(at 206.5896 57.8451 0)
 		(fields_autoplaced yes)
@@
 	)
 	(global_label "error 2"
-		(shape output)
+		(shape input)
 		(at 206.556 65.4652 0)
 		(fields_autoplaced yes)
@@
 	)
 	(global_label "SCL"
-		(shape input)
+		(shape bidirectional)
 		(at 142.9349 68.0073 180)
 		(fields_autoplaced yes)
@@
 		)
 		(property "Intersheetrefs" "${INTERSHEET_REFS}"
-			(at 136.4421 68.0073 0)
+			(at 135.3308 68.0073 0)
 			(effects
 				(font
@@
 	)
 	(global_label "M1_S1"
-		(shape input)
+		(shape output)
 		(at 191.1949 55.3073 0)
 		(fields_autoplaced yes)
@@
 	(global_label "FRQ"
 		(shape input)
-		(at 1124.9023 64.1594 180)
+		(at 1126.1723 64.2093 180)
 		(fields_autoplaced yes)
 		(effects
@@
 		)
 		(property "Intersheetrefs" "${INTERSHEET_REFS}"
-			(at 1118.228 64.1594 0)
+			(at 1119.498 64.2093 0)
 			(effects
 				(font
@@
 	)
 	(global_label "Motor2_OFF"
-		(shape input)
+		(shape output)
 		(at 191.1949 68.0073 0)
 		(fields_autoplaced yes)
@@
 	(global_label "SDA"
 		(shape output)
-		(at 541.3333 149.6842 180)
+		(at 529.3545 150.6164 180)
 		(fields_autoplaced yes)
 		(effects
@@
 		)
 		(property "Intersheetrefs" "${INTERSHEET_REFS}"
-			(at 534.78 149.6842 0)
+			(at 522.8012 150.6164 0)
 			(effects
 				(font
@@
 	)
 	(global_label " SDA"
-		(shape input)
-		(at 142.9349 65.4673 180)
+		(shape bidirectional)
+		(at 136.7317 65.4673 180)
 		(fields_autoplaced yes)
 		(effects
@@
 		)
 		(property "Intersheetrefs" "${INTERSHEET_REFS}"
-			(at 135.414 65.4673 0)
+			(at 128.0995 65.4673 0)
 			(effects
 				(font
@@
 		(fields_autoplaced yes)
 		(property "Reference" "D31"
-			(at 127.3967 450.3183 90)
+			(at 127 450.3183 90)
 			(effects
 				(font
@@
 		)
 		(property "Value" "1N5822"
-			(at 127.3967 452.8583 90)
+			(at 127 452.8583 90)
 			(effects
 				(font
@@
 		(on_board yes)
 		(dnp no)
-		(fields_autoplaced yes)
 		(property "Reference" "U7"
-			(at 343.4335 187.9212 0)
+			(at 343.3994 188.3097 0)
 			(effects
 				(font
