File: circuts/SBC/SBC.kicad_pcb (KiCad board)
At the start: 2 copper layers, 141 parts, among them IC1 PIC16F15243-I_SS, J1 DE9_Plug, J10 Power, J2 OSTTC060162, J3 XT60-M, J4 OSTTC060162, J5 640456-3, J8 B5B-XH-A_LF__SN_, Q1 IRFS4227, Q10 MMBTA06, Q2 MMBTA06, Q3 MMBTA06, Q4 MMBTA06, Q5 MMBTA06, Q8 IRFS4227, Q9 MMBTA06, U1 3.3v, U2 UC3843, U3 BTS7960B, U5 LM358DT, U6 BTS7960B, U7 BTS7960B, U8 BTS7960B, U9 LM358DT

Commit message: layout
Parts:
- removed D25: 1N4004-T_NRND, Diode_SMD:D_SOD-123
- removed REF1, REF2: MountingHole_3.2mm_M3, MountingHole:MountingHole_3.2mm_M3
- removed ZD11: BZV55B4V7, Capacitor_THT:CP_Radial_D10.0mm_P5.00mm_P7.50mm
- removed ZD12, ZD13: BZV55B4V7, Diode_SMD:D_MiniMELF
- removed ZD20: 3.3v, Diode_SMD:D_MiniMELF
- added C10: 2uf, Resistor_SMD:R_0805_2012Metric_Pad1.20x1.40mm_HandSolder, F.Cu at (149.0, 77.0)
- added C11: 1nf, Resistor_SMD:R_0805_2012Metric_Pad1.20x1.40mm_HandSolder, F.Cu at (149.5, 70.5)
- added C36: 1nf, Resistor_SMD:R_0805_2012Metric_Pad1.20x1.40mm_HandSolder, F.Cu at (51.5, 72.5)
- added C37: 470uf, Capacitor_THT:CP_Radial_D8.0mm_P5.00mm, F.Cu at (98.2, 63.0)
- added C40: 2uf, Resistor_SMD:R_0805_2012Metric_Pad1.20x1.40mm_HandSolder, F.Cu at (71.0, 74.5)
- added C41: 1nf, Resistor_SMD:R_0805_2012Metric_Pad1.20x1.40mm_HandSolder, F.Cu at (72.5, 180.1)
- added C42: 1nf, Resistor_SMD:R_0805_2012Metric_Pad1.20x1.40mm_HandSolder, F.Cu at (72.5, 183.1)
- added C45: 1nf, Capacitor_SMD:C_0805_2012Metric_Pad1.18x1.45mm_HandSolder, F.Cu at (72.6, 147.3)
- added C46: 1nf, Capacitor_SMD:C_0805_2012Metric_Pad1.18x1.45mm_HandSolder, F.Cu at (72.6, 150.3)
- added C49: 100nf, Capacitor_SMD:C_0805_2012Metric_Pad1.18x1.45mm_HandSolder, F.Cu at (72.6, 159.4)
- added C50: 100nf, Capacitor_SMD:C_0805_2012Metric_Pad1.18x1.45mm_HandSolder, F.Cu at (72.6, 162.4)
- added C51: 2uf, Capacitor_SMD:C_0805_2012Metric_Pad1.18x1.45mm_HandSolder, F.Cu at (51.6, 147.5)
- added C52: 2uf, Capacitor_SMD:C_0805_2012Metric_Pad1.18x1.45mm_HandSolder, F.Cu at (51.6, 150.5)
- added C53: 2uf, Capacitor_SMD:C_0805_2012Metric_Pad1.18x1.45mm_HandSolder, F.Cu at (51.6, 153.5)
- added C54: 100uf, Capacitor_SMD:CP_Elec_4x4.5, F.Cu at (116.6, 195.2)
- added C55: 100uf, Capacitor_SMD:CP_Elec_4x4.5, F.Cu at (116.6, 189.3)
- added C56: 100uf, Capacitor_SMD:CP_Elec_4x4.5, F.Cu at (116.6, 183.5)
- added C57: 470uf, Capacitor_SMD:CP_Elec_4x4.5, F.Cu at (124.4, 180.2)
- added C58: 470uf, Capacitor_SMD:CP_Elec_4x4.5, F.Cu at (124.4, 174.3)
- added C59: 470uf, Capacitor_SMD:CP_Elec_4x4.5, F.Cu at (124.4, 168.5)
- added C6: 2uf, Resistor_SMD:R_0805_2012Metric_Pad1.20x1.40mm_HandSolder, F.Cu at (72.5, 165.4)
- added C60: 1000uf, Capacitor_SMD:CP_Elec_4x4.5, F.Cu at (124.6, 195.0)
- added C61: 1000uf, Capacitor_SMD:CP_Elec_4x4.5, F.Cu at (71.3, 195.5)
- added C62: 1000uf, Capacitor_SMD:CP_Elec_4x4.5, F.Cu at (124.4, 187.5)
- added C63: 2uf, Capacitor_SMD:C_0805_2012Metric_Pad1.18x1.45mm_HandSolder, F.Cu at (51.6, 156.5)
- added C64: 2uf, Capacitor_SMD:C_0805_2012Metric_Pad1.18x1.45mm_HandSolder, F.Cu at (51.6, 159.5)
- added C65: 2uf, Capacitor_SMD:C_0805_2012Metric_Pad1.18x1.45mm_HandSolder, F.Cu at (51.6, 162.5)
- added C66: 100nf, Capacitor_SMD:C_0805_2012Metric_Pad1.18x1.45mm_HandSolder, F.Cu at (57.1, 147.5)
- added C67: 100nf, Capacitor_SMD:C_0805_2012Metric_Pad1.18x1.45mm_HandSolder, F.Cu at (57.1, 150.5)
- added C68: 100nf, Capacitor_SMD:C_0805_2012Metric_Pad1.18x1.45mm_HandSolder, F.Cu at (57.1, 153.5)
- added C69: 100nf, Capacitor_SMD:C_0805_2012Metric_Pad1.18x1.45mm_HandSolder, F.Cu at (57.1, 156.5)
- added C7: 2uf, Resistor_SMD:R_0805_2012Metric_Pad1.20x1.40mm_HandSolder, F.Cu at (72.5, 168.3)
- added C70: 100nf, Capacitor_SMD:C_0805_2012Metric_Pad1.18x1.45mm_HandSolder, F.Cu at (57.1, 159.5)
- added C71: 100nf, Capacitor_SMD:C_0805_2012Metric_Pad1.18x1.45mm_HandSolder, F.Cu at (57.1, 162.6)
- added C72: 100nf, Capacitor_SMD:C_0805_2012Metric_Pad1.18x1.45mm_HandSolder, F.Cu at (117.6, 143.5)
- added C73: 100nf, Resistor_SMD:R_0805_2012Metric_Pad1.20x1.40mm_HandSolder, F.Cu at (51.5, 168.5)
- added C74: 100nf, Resistor_SMD:R_0805_2012Metric_Pad1.20x1.40mm_HandSolder, F.Cu at (51.5, 171.4)
- added C75: C, Capacitor_SMD:C_0805_2012Metric_Pad1.18x1.45mm_HandSolder, F.Cu at (120.6, 143.5)
- added C76: C, Capacitor_SMD:C_0805_2012Metric_Pad1.18x1.45mm_HandSolder, F.Cu at (123.1, 143.5)
- added C77: C, Capacitor_SMD:C_0805_2012Metric_Pad1.18x1.45mm_HandSolder, F.Cu at (64.6, 137.5)
- added C8: 100pf, Resistor_SMD:R_0805_2012Metric_Pad1.20x1.40mm_HandSolder, F.Cu at (157.0, 45.0)
- added C9: 100nf, Resistor_SMD:R_0805_2012Metric_Pad1.20x1.40mm_HandSolder, F.Cu at (149.0, 74.0)
- added D1: LED, Diode_SMD:D_SOD-123, F.Cu at (62.5, 80.7)
- added D11: BZV55B3V3, Diode_SMD:D_MiniMELF, F.Cu at (97.6, 139.8)
- added D12: LED, Capacitor_SMD:C_0603_1608Metric_Pad1.08x0.95mm_HandSolder, F.Cu at (67.6, 179.0)
- added D13: LED, Capacitor_SMD:C_0603_1608Metric_Pad1.08x0.95mm_HandSolder, F.Cu at (67.6, 181.5)
- added D14: LED, Capacitor_SMD:C_0603_1608Metric_Pad1.08x0.95mm_HandSolder, F.Cu at (67.6, 184.0)
- added D15: SMAJ6.5A, Diode_SMD:D_SMF, F.Cu at (115.6, 156.4)
- added D16: SMAJ6.5A, Diode_SMD:D_SMF, F.Cu at (115.6, 159.8)
- added D20: 5.6v zener, Diode_SMD:D_MiniMELF, F.Cu at (90.9, 139.8)
- added D21: 1N4004-T_NRND, Diode_SMD:D_SOD-123, F.Cu at (115.6, 169.8)
- added D22: 1N4004-T_NRND, Diode_SMD:D_SOD-123, F.Cu at (115.6, 173.2)
- added D23: 1N4004-T_NRND, Diode_SMD:D_SOD-123, F.Cu at (115.6, 176.5)
- added D24: BZV55B3V3, Diode_SMD:D_MiniMELF, F.Cu at (87.6, 139.8)
- added D3: 1N4004-T_NRND, Diode_SMD:D_SOD-123, F.Cu at (65.2, 68.2)
- added D6: 1N4004-T_NRND, Diode_SMD:D_SOD-123, F.Cu at (125.5, 34.1)
- added D7: 1N4004-T_NRND, Diode_SMD:D_SOD-123, F.Cu at (78.7, 68.2)
- added D8: 20v zener, Diode_SMD:D_MiniMELF, F.Cu at (46.5, 59.0)
- added F1: 1A, Diode_SMD:D_SOD-128, F.Cu at (107.0, 77.3)
- added F4: 1A, Diode_SMD:D_SOD-128, F.Cu at (45.1, 161.2)
- added F5: 1A, Capacitor_SMD:C_0805_2012Metric_Pad1.18x1.45mm_HandSolder, F.Cu at (63.3, 147.0)
- added F6: 1A, Capacitor_SMD:C_0603_1608Metric_Pad1.08x0.95mm_HandSolder, F.Cu at (67.6, 186.5)
- added F7: 1A, Capacitor_SMD:C_0805_2012Metric_Pad1.18x1.45mm_HandSolder, F.Cu at (63.3, 150.0)
- added J11: buzzer, 282837-2:TE_282837-2, F.Cu at (135.6, 172.9)
- added J12: metal detect, TerminalBlock:TerminalBlock_bornier-3_P5.08mm, F.Cu at (135.6, 192.6)
- added J13: 12v Power, 282837-2:TE_282837-2, F.Cu at (135.6, 161.4)
- added J14: 5v Power, 282837-2:TE_282837-2, F.Cu at (135.6, 149.0)
- added J6: XT60-M, XT60-M:AMASS_XT60-M, F.Cu at (28.5, 89.9)
- added J7: OSTTC060162, footprints:CONN_6P-OSTTC_OST, F.Cu at (85.0, 26.0)
- added J9: Conn_02x04_Odd_Even, Connector_PinHeader_2.54mm:PinHeader_2x04_P2.54mm_Vertical, F.Cu at (37.3, 187.1)
- added Q6: MMBTA06, Package_TO_SOT_SMD:SOT-23, F.Cu at (45.9, 87.0)
- added Q7: MMBTA06, Package_TO_SOT_SMD:SOT-23, F.Cu at (58.1, 42.5)
- added R21: 470, Resistor_SMD:R_0805_2012Metric_Pad1.20x1.40mm_HandSolder, F.Cu at (45.0, 92.5)
- added R24: 10k, Resistor_SMD:R_0805_2012Metric_Pad1.20x1.40mm_HandSolder, F.Cu at (97.4, 73.0)
- added R28: 56k, Resistor_SMD:R_0805_2012Metric_Pad1.20x1.40mm_HandSolder, F.Cu at (101.0, 73.0)
- added R29: 56k, Resistor_SMD:R_0805_2012Metric_Pad1.20x1.40mm_HandSolder, F.Cu at (91.0, 68.5)
- added R31: 100k, Resistor_SMD:R_0805_2012Metric_Pad1.20x1.40mm_HandSolder, F.Cu at (94.5, 68.5)
- added R32: 56k, Resistor_SMD:R_0805_2012Metric_Pad1.20x1.40mm_HandSolder, F.Cu at (102.5, 68.5)
- added R33: 2.2k, Resistor_SMD:R_0805_2012Metric_Pad1.20x1.40mm_HandSolder, F.Cu at (149.0, 80.0)
- added R34: 220, Resistor_SMD:R_0805_2012Metric_Pad1.20x1.40mm_HandSolder, F.Cu at (117.0, 39.0)
- added R51: 0.3, Resistor_SMD:R_2512_6332Metric_Pad1.40x3.35mm_HandSolder, F.Cu at (28.0, 55.0)
- added R52: 10k, Resistor_SMD:R_0805_2012Metric_Pad1.20x1.40mm_HandSolder, F.Cu at (166.0, 51.0)
- added R53: 10k, Resistor_SMD:R_0805_2012Metric_Pad1.20x1.40mm_HandSolder, F.Cu at (166.0, 48.0)
- added R54: 56k, Resistor_SMD:R_0805_2012Metric_Pad1.20x1.40mm_HandSolder, F.Cu at (166.0, 45.1)
- added R55: 56k, Resistor_SMD:R_0805_2012Metric_Pad1.20x1.40mm_HandSolder, F.Cu at (162.5, 63.0)
- added R56: 2k, Resistor_SMD:R_0805_2012Metric_Pad1.20x1.40mm_HandSolder, F.Cu at (134.0, 33.5)
- added R57: 100k, Resistor_SMD:R_0805_2012Metric_Pad1.20x1.40mm_HandSolder, F.Cu at (75.5, 74.5)
- added R58: 56k, Resistor_SMD:R_0805_2012Metric_Pad1.20x1.40mm_HandSolder, F.Cu at (67.0, 74.5)
- added R60: 5.1k, Resistor_SMD:R_0805_2012Metric_Pad1.20x1.40mm_HandSolder, F.Cu at (51.5, 174.4)
- added R83: 10k, Resistor_SMD:R_0805_2012Metric_Pad1.20x1.40mm_HandSolder, F.Cu at (56.9, 183.2)
- added R84: 1k, Resistor_SMD:R_0805_2012Metric_Pad1.20x1.40mm_HandSolder, F.Cu at (56.9, 186.2)
- added R85: 1k, Resistor_SMD:R_0805_2012Metric_Pad1.20x1.40mm_HandSolder, F.Cu at (63.1, 153.0)
- added R86: 1k, Resistor_SMD:R_0805_2012Metric_Pad1.20x1.40mm_HandSolder, F.Cu at (63.1, 155.9)
- added R87: 1k, Resistor_SMD:R_0805_2012Metric_Pad1.20x1.40mm_HandSolder, F.Cu at (63.1, 158.9)
- added R88: 200, Resistor_THT:R_Bare_Metal_Element_L16.3mm_W4.8mm_P15.30mm, F.Cu at (47.5, 198.0)
- added R89: 10k, Resistor_SMD:R_0805_2012Metric_Pad1.20x1.40mm_HandSolder, F.Cu at (63.1, 161.8)
- added R90: 10k, Resistor_SMD:R_0805_2012Metric_Pad1.20x1.40mm_HandSolder, F.Cu at (63.1, 167.0)
- added SW1: SW_Push, BUTT-2:SW_BUTT-2, F.Cu at (35.0, 139.0)
- added SW2: SW_Push, BUTT-2:SW_BUTT-2, F.Cu at (42.5, 139.0)
- added SW3: SW_Push, BUTT-2:SW_BUTT-2, F.Cu at (50.0, 139.0)
- added SW4: SW_Push, BUTT-2:SW_BUTT-2, F.Cu at (57.6, 139.0)
- added U10: ESP32-DEVKIT-V1, ESP32-DEVKIT-V1:MODULE_ESP32_DEVKIT_V1, F.Cu at (93.3, 172.8)
- added U11: ~, Connector_PinHeader_2.54mm:PinHeader_1x08_P2.54mm_Vertical, F.Cu at (24.0, 177.0)
- added U12: AMS1117-5.0, Package_TO_SOT_SMD:SOT-223-3_TabPin2, F.Cu at (36.2, 150.5)
- added U4: LM358DT, Package_SO:SOIC-8_3.9x4.9mm_P1.27mm, F.Cu at (57.6, 59.5)
- added ZD1: 3.3v, Diode_SMD:D_MiniMELF, F.Cu at (43.2, 59.0)
- added ZD3: BZV55B4V7, Diode_SMD:D_MiniMELF, F.Cu at (57.5, 80.8)
- added ZD4: BZV55B4V7, Capacitor_THT:CP_Radial_D10.0mm_P5.00mm_P7.50mm, F.Cu at (72.5, 39.0)
- added ZD5: BZV55B4V7, Diode_SMD:D_MiniMELF, F.Cu at (57.5, 74.2)
- added ZD6: BZV55B4V7, Diode_SMD:D_MiniMELF, F.Cu at (84.2, 139.8)
- added ZD7: BZV55B4V7, Diode_SMD:D_MiniMELF, F.Cu at (80.9, 139.8)
- C12: footprint Capacitor_THT:CP_Radial_D8.0mm_P5.00mm -> Resistor_SMD:R_0805_2012Metric_Pad1.20x1.40mm_HandSolder
- C15, C29, C34, C38: value 100nf -> 2uf
- C16, C20, C39: value 1nf -> 2uf
- C17, C31: value 470uf -> 100nf; footprint Capacitor_THT:CP_Radial_D8.0mm_P5.00mm -> Resistor_SMD:R_0805_2012Metric_Pad1.20x1.40mm_HandSolder
- C18, C2, C4, C43, C44: value 2uf -> 1nf
- C19: value 100nf -> 470uf; footprint Resistor_SMD:R_0805_2012Metric_Pad1.20x1.40mm_HandSolder -> Capacitor_THT:CP_Radial_D8.0mm_P5.00mm
- C21: value 470uf -> 2uf; footprint Capacitor_THT:CP_Radial_D8.0mm_P5.00mm -> Resistor_SMD:R_0805_2012Metric_Pad1.20x1.40mm_HandSolder
- C22: footprint Resistor_SMD:R_0805_2012Metric_Pad1.20x1.40mm_HandSolder -> Capacitor_THT:CP_Radial_D8.0mm_P5.00mm
- C23: value 100pf -> 470uf; footprint Resistor_SMD:R_0805_2012Metric_Pad1.20x1.40mm_HandSolder -> Capacitor_THT:CP_Radial_D8.0mm_P5.00mm
- C24: value 2uf -> 470uf; footprint Resistor_SMD:R_0805_2012Metric_Pad1.20x1.40mm_HandSolder -> Capacitor_THT:CP_Radial_D8.0mm_P5.00mm
- C3, C30: value 1nf -> 100nf
- C32, C35: value 2uf -> 100nf
- C47: value 470uf -> 1nf; footprint Capacitor_THT:CP_Radial_D8.0mm_P5.00mm -> Capacitor_SMD:C_0805_2012Metric_Pad1.18x1.45mm_HandSolder
- C48: value 2uf -> 100nf; footprint Resistor_SMD:R_0805_2012Metric_Pad1.20x1.40mm_HandSolder -> Capacitor_SMD:C_0805_2012Metric_Pad1.18x1.45mm_HandSolder
- D10: value 1N4004-T_NRND -> LED; footprint Diode_SMD:D_SOD-123 -> Capacitor_SMD:C_0603_1608Metric_Pad1.08x0.95mm_HandSolder
- D17, D18: value LED -> SMAJ6.5A; footprint Diode_SMD:D_SOD-123 -> Diode_SMD:D_SMF
- D19: value LED -> 20v zener; footprint Diode_SMD:D_SOD-123 -> Diode_SMD:D_MiniMELF
- D4, D5: value 1N4004-T_NRND -> LED
- D9: value 20v zener -> 1N4004-T_NRND; footprint Diode_SMD:D_MiniMELF -> Diode_SMD:D_SOD-123
- J1: value DE9_Plug -> 640456-3; footprint DB9:DB9 -> 640456-3:TE_640456-3
- J10: value Power -> motor_con; footprint 282837-2:TE_282837-2 -> DB9:DB9
- J2: value OSTTC060162 -> B5B-XH-A_LF__SN_; footprint footprints:CONN_6P-OSTTC_OST -> B5B-XH-A_LF__SN_:JST_B5B-XH-A_LF__SN_
- J3: value XT60-M -> Power; footprint XT60-M:AMASS_XT60-M -> 282837-2:TE_282837-2
- J4: value OSTTC060162 -> DE9_Plug; footprint footprints:CONN_6P-OSTTC_OST -> DB9:DB9
- J5: value 640456-3 -> OSTTC060162; footprint 640456-3:TE_640456-3 -> footprints:CONN_6P-OSTTC_OST
- J8: value B5B-XH-A_LF__SN_ -> grip_con; footprint B5B-XH-A_LF__SN_:JST_B5B-XH-A_LF__SN_ -> DB9:DB9
- Q1: value IRFS4227 -> MMBTA06; footprint Package_TO_SOT_SMD:TO-263-3_TabPin2 -> Package_TO_SOT_SMD:SOT-23
- Q10: value MMBTA06 -> BC817
- Q4: value MMBTA06 -> IRFS4227; footprint Package_TO_SOT_SMD:SOT-23 -> Package_TO_SOT_SMD:TO-263-3_TabPin2
- Q9: value MMBTA06 -> FDS4559; footprint Package_TO_SOT_SMD:SOT-23 -> Package_SO:SOIC-8_3.9x4.9mm_P1.27mm
- R1, R15, R17, R9: value 10k -> 2k
- R10: value 330 -> 10k
- R11: value 1.5k -> 3.3k
- R12: value 0.3 -> 2k; footprint Resistor_SMD:R_2512_6332Metric_Pad1.40x3.35mm_HandSolder -> Resistor_SMD:R_0805_2012Metric_Pad1.20x1.40mm_HandSolder
- R13, R2: value 0.3 -> 220; footprint Resistor_SMD:R_2512_6332Metric_Pad1.40x3.35mm_HandSolder -> Resistor_SMD:R_0805_2012Metric_Pad1.20x1.40mm_HandSolder
- R14: value 3.3k -> 5.1k
- R16, R43: value 470 -> 2k
- R18: value 26k -> 0.3; footprint Resistor_SMD:R_0805_2012Metric_Pad1.20x1.40mm_HandSolder -> Resistor_SMD:R_2512_6332Metric_Pad1.40x3.35mm_HandSolder
- R19: value 100k -> 330
- R20: value 200 -> 0.3; footprint Resistor_THT:R_Bare_Metal_Element_L16.3mm_W4.8mm_P15.30mm -> Resistor_SMD:R_2512_6332Metric_Pad1.40x3.35mm_HandSolder
- R22: value 220 -> 0.3; footprint Resistor_SMD:R_0805_2012Metric_Pad1.20x1.40mm_HandSolder -> Resistor_SMD:R_2512_6332Metric_Pad1.40x3.35mm_HandSolder
- R25, R71: value 220 -> 10k
- R26: value 2k -> 26k
- R27: value 10k -> 100k
- R3: value 56k -> 220
- R35: value 2k -> 220
- R36: value 2k -> 5.1k
- R37, R5, R6, R63: value 10k -> 5.1k
- R38: value 100k -> 2k
- R39, R65, R66, R69: value 56k -> 10k
- R4: value 2k -> 56k
- R40: value 470 -> 200; footprint Resistor_SMD:R_0805_2012Metric_Pad1.20x1.40mm_HandSolder -> Resistor_THT:R_Bare_Metal_Element_L16.3mm_W4.8mm_P15.30mm
- R41: value 2k -> 1.5k
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Connections:
- C1 pad 1: Net-(D4-A) -> 5v+
- C12 pad 1: Net-(ZD11-K) -> M1_R
- C12 pad 2: GND -> M1_L
- C13 pad 1: M1_current_sen -> M1_R
- C13 pad 2: GND -> M1_L
- C14 pad 1: M2_current_sen -> Net-(D2-A)
- C15 pad 1: 5v+ -> M1_current_sen
- C16 pad 1: 5v+ -> GND
- C16 pad 2: GND -> HV
- C17 pad 1: 5v+ -> HV
- C18 pad 1: GND -> HV
- C18 pad 2: 5v+ -> GND
- C2 pad 1: 5v+ -> Net-(C2-Pad1)
- C20 pad 1: HV -> GND
- C20 pad 2: GND -> HV
- C21 pad 1: HV -> Net-(C21-Pad1)
- C21 pad 2: GND -> Net-(C21-Pad2)
- C22 pad 1: GND -> Net-(ZD4-K)
- C22 pad 2: HV -> GND
- C23 pad 1: PWM -> HV
- C24 pad 1: Net-(C24-Pad1) -> HV
- C24 pad 2: Net-(C24-Pad2) -> GND
- C25 pad 1: M1_L -> 5v+
- C25 pad 2: M1_R -> GND
- C26 pad 1: M1_L -> 5v+
- C26 pad 2: M1_R -> GND
- C27 pad 1: HV -> 5v+
- C28 pad 1: M1_R -> Net-(D3-A)
- C28 pad 2: M1_L -> GND
- C29 pad 1: M2_L -> GND
- C29 pad 2: M2_R -> 5v+
- C3 pad 1: Net-(C3-Pad1) -> M2_L
- C3 pad 2: GND -> M2_R
- C30 pad 1: M2_L -> GND
- C30 pad 2: M2_R -> Net-(U5-VI)
- C31 pad 1: HV -> GND
- C31 pad 2: GND -> Net-(U6-VI)
- C32 pad 1: M2_R -> GND
- C32 pad 2: M2_L -> Net-(U5-VO)
- C33 pad 2: Net-(U1-OUT) -> Net-(U6-VO)
- C34 pad 1: GND -> Net-(D6-A)
- C34 pad 2: Net-(U1-IN) -> GND
- C35 pad 1: GND -> 3.3V
- C35 pad 2: HV -> GND
- C38 pad 1: 3.3V -> GND
- C38 pad 2: GND -> 3.3V
- C39 pad 1: 3.3V -> Net-(C39-Pad1)
- C39 pad 2: GND -> Net-(C39-Pad2)
- C4 pad 1: Net-(C4-Pad1) -> M2_L
- C4 pad 2: Net-(C4-Pad2) -> M2_R
- C43 pad 1: Net-(D25-A) -> Net-(C43-Pad1)
- C44 pad 1: Net-(D2-A) -> Net-(C44-Pad1)
- C48 pad 1: GND -> HV
- C48 pad 2: 3.3V -> GND
- C5 pad 1: Net-(D5-A) -> M2_R
- C5 pad 2: GND -> M2_L
- D10 pad 1: HV -> buzzing_gnd
- D10 pad 2: GND -> Net-(D10-A)
- D17 pad 1: Net-(D17-K) -> 5v+
- D17 pad 2: Motor2_OFF -> GND
- D18 pad 1: Net-(D18-K) -> HV
- D18 pad 2: 3.3v -> GND
- D19 pad 1: Net-(D19-K) -> HV
- D19 pad 2: HV -> GND
- D2 pad 1: CS -> Net-(D2-K)
- D4 pad 2: Net-(D4-A) -> HV
- D5 pad 1: CS -> Net-(D5-K)
- D5 pad 2: Net-(D5-A) -> 3.3v
- F2 pad 1: Net-(U1-OUT) -> Net-(U6-VO)
- F3 pad 2: HVblock -> HV
- J1 pad 1: HVblock -> Net-(C2-Pad1)
- J1 pad 2: GND -> Net-(U1-RC)
- J1 pad 3: 5v+ -> Net-(J1-Pad3)
- J10 pad 1: HVblock -> HV
- J2 pad 1: GND -> Mcler
- J2 pad 2: 5v+ -> 3.3V
- J2 pad 3: B2 -> GND
- J2 pad 4: A2 -> PGD
- J2 pad 5: M2_L -> PGC
- J4 pad 1: GND -> HV
- J4 pad 2: 5v+ -> GND
- J4 pad 3: B1 -> 5v+
- J4 pad 4: A1 -> 3.3V
- J4 pad 5: M1_L -> SCL
- J4 pad 6: M1_R -> HV
- J5 pad 1: Net-(C3-Pad1) -> GND
- J5 pad 2: Net-(U2-RC) -> 5v+
- J5 pad 3: Net-(J5-Pad3) -> Net-(C41-Pad1)
- J8 pad 1: Mcler -> HV
- J8 pad 2: 3.3V -> GND
- J8 pad 3: GND -> 5v+
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Routing:
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Other:
- board outline added: 170 x 194.5 mm

Commit message: 7-8 AT 2 PM LAYOUT EDITING
Parts:
- removed F1, F2: 1A, Diode_SMD:D_SOD-128
- removed R89, R90: 10k, Resistor_SMD:R_0805_2012Metric_Pad1.20x1.40mm_HandSolder
- removed SW3: SW_Push, BUTT-2:SW_BUTT-2
- removed U6: AMS1117-3.3, Package_TO_SOT_SMD:SOT-223-3_TabPin2
- added C78: 1nf, Capacitor_SMD:C_0805_2012Metric_Pad1.18x1.45mm_HandSolder, F.Cu at (-95.4, 35.1)
- added C79: 100nf, Capacitor_SMD:C_0805_2012Metric_Pad1.18x1.45mm_HandSolder, F.Cu at (-95.4, 38.1)
- added C80: 2uf, Capacitor_SMD:C_0805_2012Metric_Pad1.18x1.45mm_HandSolder, F.Cu at (-95.4, 41.1)
- added C81: 470uf, Capacitor_SMD:CP_Elec_4x4.5, F.Cu at (-102.4, 49.7)
- added C82: 2uf, Resistor_SMD:R_0805_2012Metric_Pad1.20x1.40mm_HandSolder, F.Cu at (-145.6, 33.3)
- added C83: 100nf, Resistor_SMD:R_0805_2012Metric_Pad1.20x1.40mm_HandSolder, F.Cu at (-145.6, 36.2)
- added C84: 100nf, Resistor_SMD:R_0805_2012Metric_Pad1.20x1.40mm_HandSolder, F.Cu at (-145.6, 39.2)
- added C85: 100nf, Resistor_SMD:R_0805_2012Metric_Pad1.20x1.40mm_HandSolder, F.Cu at (-145.6, 42.1)
- added C86: 100nf, Resistor_SMD:R_0805_2012Metric_Pad1.20x1.40mm_HandSolder, F.Cu at (-145.6, 45.1)
- added C87: 1nf, Resistor_SMD:R_0805_2012Metric_Pad1.20x1.40mm_HandSolder, F.Cu at (-145.6, 48.0)
- added C88: 470uf, Capacitor_THT:CP_Radial_D8.0mm_P5.00mm, F.Cu at (-113.5, 47.9)
- added C89: 2uf, Resistor_SMD:R_0805_2012Metric_Pad1.20x1.40mm_HandSolder, F.Cu at (-145.6, 51.0)
- added C90: 100nf, Capacitor_SMD:C_0805_2012Metric_Pad1.18x1.45mm_HandSolder, F.Cu at (-95.4, 44.1)
- added C91: 33uf, Capacitor_THT:CP_Radial_D4.0mm_P1.50mm, F.Cu at (-122.2, 44.7)
- added C92: 100nf, Resistor_SMD:R_0805_2012Metric_Pad1.20x1.40mm_HandSolder, F.Cu at (-140.9, 30.3)
- added C93: 100nf, Resistor_SMD:R_0805_2012Metric_Pad1.20x1.40mm_HandSolder, F.Cu at (-140.9, 33.3)
- added D25: 1N4004-T_NRND, Diode_SMD:D_MiniMELF, F.Cu at (-144.8, -6.21)
- added D26: 1N4004-T_NRND, Diode_SMD:D_MiniMELF, F.Cu at (-144.8, -2.87)
- added D27: 1N4004-T_NRND, Diode_SMD:D_MiniMELF, F.Cu at (-144.8, 0.47)
- added D28: 1N4004-T_NRND, Diode_SMD:D_MiniMELF, F.Cu at (-144.8, 3.81)
- added D29: 1N5822, Diode_SMD:D_MiniMELF, F.Cu at (-144.8, 7.15)
- added D30: 1N5822, Diode_SMD:D_MiniMELF, F.Cu at (-144.8, 10.5)
- added D31: 1N5822, Diode_SMD:D_MiniMELF, F.Cu at (-144.8, 13.8)
- added D32: 1N5822, Diode_SMD:D_MiniMELF, F.Cu at (-144.8, 17.2)
- added D33: SMAJ26A, Diode_SMD:D_MiniMELF, F.Cu at (-144.8, 20.5)
- added D34: SMAJ26A, Diode_SMD:D_MiniMELF, F.Cu at (-144.8, 23.9)
- added D35: SMAJ26A, Diode_SMD:D_MiniMELF, F.Cu at (-144.8, 27.2)
- added D36: SMAJ26A, Diode_SMD:D_MiniMELF, F.Cu at (-138.4, -6.21)
- added D37: 1N5822, Diode_SMD:D_MiniMELF, F.Cu at (-138.4, -2.87)
- added D38: 1N5822, Diode_SMD:D_MiniMELF, F.Cu at (-138.4, 0.47)
- added D39: 1N5822, Diode_SMD:D_MiniMELF, F.Cu at (-138.4, 3.81)
- added D40: 1N5822, Diode_SMD:D_MiniMELF, F.Cu at (-138.4, 7.15)
- added D41: 1N5822, Diode_SMD:D_MiniMELF, F.Cu at (-138.4, 10.5)
- added D42: 1N5822, Diode_SMD:D_MiniMELF, F.Cu at (-138.4, 13.8)
- added D43: LED, Diode_SMD:D_MiniMELF, F.Cu at (-138.4, 17.2)
- added D44: LED, Diode_SMD:D_MiniMELF, F.Cu at (-138.4, 20.5)
- added D45: 1N4004-T_NRND, Diode_SMD:D_MiniMELF, F.Cu at (-138.4, 23.9)
- added D46: 1N4004-T_NRND, Diode_SMD:D_MiniMELF, F.Cu at (-138.4, 27.2)
- added D47: 1N4004-T_NRND, Diode_SMD:D_MiniMELF, F.Cu at (-132.0, -6.21)
- added D48: 1N4004-T_NRND, Diode_SMD:D_MiniMELF, F.Cu at (-132.0, -2.87)
- added D49: 1N4004-T_NRND, Diode_SMD:D_MiniMELF, F.Cu at (-132.0, 0.47)
- added D50: L_LED, Diode_SMD:D_MiniMELF, F.Cu at (-132.0, 3.81)
- added D51: R_LED, Diode_SMD:D_MiniMELF, F.Cu at (-132.0, 7.15)
- added D52: L_LED, Diode_SMD:D_MiniMELF, F.Cu at (-132.0, 10.5)
- added D53: R_LED, Diode_SMD:D_MiniMELF, F.Cu at (-132.0, 13.8)
- added D54: 1N4004-T_NRND, Diode_SMD:D_MiniMELF, F.Cu at (-132.0, 17.2)
- added D55: 1N4004-T_NRND, Diode_SMD:D_MiniMELF, F.Cu at (-132.0, 20.5)
- added D56: 1N4004-T_NRND, Diode_SMD:D_MiniMELF, F.Cu at (-132.0, 23.9)
- added J15: Barrel_Jack_MountingPin, Connector_BarrelJack:BarrelJack_GCT_DCJ200-10-A_Horizontal, F.Cu at (7.85, 196.2)
- added R100: 200, Resistor_SMD:R_0805_2012Metric_Pad1.20x1.40mm_HandSolder, F.Cu at (-113.7, -4.70)
- added R101: 1ohm op*, Resistor_SMD:R_0805_2012Metric_Pad1.20x1.40mm_HandSolder, F.Cu at (-136.1, 48.0)
- added R102: 1ohm, Resistor_SMD:R_0805_2012Metric_Pad1.20x1.40mm_HandSolder, F.Cu at (-136.1, 51.0)
- added R103: 10k, Resistor_SMD:R_0805_2012Metric_Pad1.20x1.40mm_HandSolder, F.Cu at (-131.4, 30.3)
- added R104: 1ohm, Resistor_SMD:R_0805_2012Metric_Pad1.20x1.40mm_HandSolder, F.Cu at (-131.4, 33.3)
- added R105: 1ohm, Resistor_SMD:R_0805_2012Metric_Pad1.20x1.40mm_HandSolder, F.Cu at (-131.4, 36.2)
- added R106: 200, Resistor_SMD:R_0805_2012Metric_Pad1.20x1.40mm_HandSolder, F.Cu at (-113.7, 1.65)
- added R107: 10k, Resistor_SMD:R_0805_2012Metric_Pad1.20x1.40mm_HandSolder, F.Cu at (-131.4, 39.2)
- added R108: 1k, Resistor_SMD:R_0805_2012Metric_Pad1.20x1.40mm_HandSolder, F.Cu at (-131.4, 42.1)
- added R109: 1k, Resistor_SMD:R_0805_2012Metric_Pad1.20x1.40mm_HandSolder, F.Cu at (-131.4, 45.1)
- added R110: 1k, Resistor_SMD:R_0805_2012Metric_Pad1.20x1.40mm_HandSolder, F.Cu at (-131.4, 48.0)
- added R111: 1.5k, Resistor_SMD:R_0805_2012Metric_Pad1.20x1.40mm_HandSolder, F.Cu at (-131.4, 51.0)
- added R112: 330, Resistor_SMD:R_0805_2012Metric_Pad1.20x1.40mm_HandSolder, F.Cu at (-126.6, 30.3)
- added R113: 1ohm op*, Resistor_SMD:R_0805_2012Metric_Pad1.20x1.40mm_HandSolder, F.Cu at (-126.6, 33.3)
- added R114: 220, Resistor_SMD:R_0805_2012Metric_Pad1.20x1.40mm_HandSolder, F.Cu at (-95.4, 47.1)
- added R115: 1.5k, Resistor_SMD:R_0805_2012Metric_Pad1.20x1.40mm_HandSolder, F.Cu at (-126.6, 36.2)
- added R116: 1.5k, Resistor_SMD:R_0805_2012Metric_Pad1.20x1.40mm_HandSolder, F.Cu at (-126.6, 39.2)
- added R117: 220, Resistor_SMD:R_0805_2012Metric_Pad1.20x1.40mm_HandSolder, F.Cu at (-126.6, 42.1)
- added R118: 2.2k, Resistor_SMD:R_0805_2012Metric_Pad1.20x1.40mm_HandSolder, F.Cu at (-126.6, 45.1)
- added R119: 220, Resistor_SMD:R_0805_2012Metric_Pad1.20x1.40mm_HandSolder, F.Cu at (-126.6, 48.0)
- added R120: 5.1k, Resistor_SMD:R_0805_2012Metric_Pad1.20x1.40mm_HandSolder, F.Cu at (-126.6, 51.0)
- added R59: 5k, Resistor_SMD:R_0805_2012Metric_Pad1.20x1.40mm_HandSolder, F.Cu at (-140.9, 42.1)
- added R91: 10k, Resistor_SMD:R_0805_2012Metric_Pad1.20x1.40mm_HandSolder, F.Cu at (-140.9, 45.1)
- added R92: 10k, Resistor_SMD:R_0805_2012Metric_Pad1.20x1.40mm_HandSolder, F.Cu at (-140.9, 48.0)
- added R93: 10k, Resistor_SMD:R_0805_2012Metric_Pad1.20x1.40mm_HandSolder, F.Cu at (-140.9, 51.0)
- added R94: 10k, Resistor_SMD:R_0805_2012Metric_Pad1.20x1.40mm_HandSolder, F.Cu at (-136.1, 30.3)
- added R95: 10k, Resistor_SMD:R_0805_2012Metric_Pad1.20x1.40mm_HandSolder, F.Cu at (-136.1, 33.3)
- added R96: 10k, Resistor_SMD:R_0805_2012Metric_Pad1.20x1.40mm_HandSolder, F.Cu at (-136.1, 36.2)
- added R97: 10k, Resistor_SMD:R_0805_2012Metric_Pad1.20x1.40mm_HandSolder, F.Cu at (-136.1, 39.2)
- added R98: 10k, Resistor_SMD:R_0805_2012Metric_Pad1.20x1.40mm_HandSolder, F.Cu at (-136.1, 42.1)
- added R99: 1ohm, Resistor_SMD:R_0805_2012Metric_Pad1.20x1.40mm_HandSolder, F.Cu at (-136.1, 45.1)
- added RV1: R_Potentiometer, Potentiometer_SMD:Potentiometer_Vishay_TS53YJ_Vertical, F.Cu at (-120.5, 32.1)
- added RV2: R_Potentiometer, Potentiometer_SMD:Potentiometer_Vishay_TS53YJ_Vertical, F.Cu at (-120.5, 38.7)
- added SW5: SW_Push, Button_Switch_SMD:SW_DIP_SPSTx01_Slide_6.7x4.1mm_W6.73mm_P2.54mm_LowProfile_JPin, F.Cu at (-133.6, 164.9)
- added SW6: rst, Button_Switch_SMD:SW_DIP_SPSTx01_Slide_6.7x4.1mm_W6.73mm_P2.54mm_LowProfile_JPin, F.Cu at (-133.6, 170.7)
- added SW7: SW_Push, Button_Switch_SMD:SW_DIP_SPSTx01_Slide_6.7x4.1mm_W6.73mm_P2.54mm_LowProfile_JPin, F.Cu at (-133.6, 176.5)
- added U13: L7805, Package_TO_SOT_SMD:TO-252-2, F.Cu at (-40.6, 172.0)
- added U14: L7809, Package_TO_SOT_THT:TO-220-3_Vertical, F.Cu at (2.73, 3.42)
- added ZD10: 3.3v, Diode_SMD:D_MiniMELF, F.Cu at (-125.6, -2.87)
- added ZD11: BZV55B4V7, Diode_SMD:D_MiniMELF, F.Cu at (-125.6, 0.47)
- added ZD12: BZV55B4V7, Diode_SMD:D_MiniMELF, F.Cu at (3.04, 5.50)
- added ZD13: 3.3v, Diode_SMD:D_MiniMELF, F.Cu at (-125.6, 3.81)
- added ZD14: 3.3v, Diode_SMD:D_MiniMELF, F.Cu at (-125.6, 7.15)
- added ZD15: 3.3v, Diode_SMD:D_MiniMELF, F.Cu at (-125.6, 10.5)
- added ZD16: 3.3v, Diode_SMD:D_MiniMELF, F.Cu at (-125.6, 13.8)
- added ZD17: 3.3v, Diode_SMD:D_MiniMELF, F.Cu at (-125.6, 17.2)
- added ZD18: 3.3v, Diode_SMD:D_MiniMELF, F.Cu at (-125.6, 20.5)
- added ZD19: 3.3v, Diode_SMD:D_MiniMELF, F.Cu at (-125.6, 23.9)
- added ZD20: 3.3v, Diode_SMD:D_MiniMELF, F.Cu at (-125.6, 27.2)
- added ZD21: 3.3v, Diode_SMD:D_MiniMELF, F.Cu at (-119.2, -6.21)
- added ZD22: 3.3v, Diode_SMD:D_MiniMELF, F.Cu at (-119.2, -2.87)
- added ZD23: 3.3v, Diode_SMD:D_MiniMELF, F.Cu at (-119.2, 0.47)
- added ZD24: 3.3v, Diode_SMD:D_MiniMELF, F.Cu at (-119.2, 3.81)
- added ZD25: 3.3v, Diode_SMD:D_MiniMELF, F.Cu at (-119.2, 7.15)
- added ZD26: 3.3v, Diode_SMD:D_MiniMELF, F.Cu at (-119.2, 10.5)
- added ZD27: 3.3v, Diode_SMD:D_MiniMELF, F.Cu at (-119.2, 13.8)
- added ZD28: 3.3v, Diode_SMD:D_MiniMELF, F.Cu at (-119.2, 17.2)
- added ZD29: 3.3v, Diode_SMD:D_MiniMELF, F.Cu at (-119.2, 20.5)
- added ZD30: 3.3v, Diode_SMD:D_MiniMELF, F.Cu at (-119.2, 23.9)
- added ZD31: 3.3v, Diode_SMD:D_MiniMELF, F.Cu at (2.72, 1.17)
- added ZD32: 3.3v, Diode_SMD:D_MiniMELF, F.Cu at (2.72, 4.51)
- added ZD33: 3.3v, Diode_SMD:D_MiniMELF, F.Cu at (2.72, 7.85)
- added ZD34: 3.3v, Diode_SMD:D_MiniMELF, F.Cu at (2.72, 11.2)
- added ZD8: 3.3v, Diode_SMD:D_MiniMELF, F.Cu at (-132.0, 27.2)
- added ZD9: 20v, Diode_SMD:D_MiniMELF, F.Cu at (-125.6, -6.21)
- C1, C10, C11, C13, C14, C15, C16, C17, C18, C2, C3, C4, C5, C9: footprint Resistor_SMD:R_0805_2012Metric_Pad1.20x1.40mm_HandSolder -> Capacitor_SMD:C_0805_2012Metric_Pad1.18x1.45mm_HandSolder
- C12: value 2uf -> 33uf; footprint Resistor_SMD:R_0805_2012Metric_Pad1.20x1.40mm_HandSolder -> Capacitor_THT:CP_Radial_D8.0mm_P5.00mm
- C6: value 2uf -> 470uf; footprint Resistor_SMD:R_0805_2012Metric_Pad1.20x1.40mm_HandSolder -> Capacitor_THT:CP_Radial_D8.0mm_P5.00mm
- C7: value 2uf -> 100nf; footprint Resistor_SMD:R_0805_2012Metric_Pad1.20x1.40mm_HandSolder -> Capacitor_SMD:C_0805_2012Metric_Pad1.18x1.45mm_HandSolder
- C8: value 100pf -> 2pf; footprint Resistor_SMD:R_0805_2012Metric_Pad1.20x1.40mm_HandSolder -> Capacitor_SMD:C_0805_2012Metric_Pad1.18x1.45mm_HandSolder
- D1, D2, D21, D22, D23, D3, D4, D5, D6, D7, D9: footprint Diode_SMD:D_SOD-123 -> Diode_SMD:D_MiniMELF
- D10, D12, D13, D14: footprint Capacitor_SMD:C_0603_1608Metric_Pad1.08x0.95mm_HandSolder -> Diode_SMD:D_MiniMELF
- D15, D16, D17, D18: footprint Diode_SMD:D_SMF -> Diode_SMD:D_MiniMELF
- J10: value motor_con -> DE9_Plug
- J12: value metal detect -> Screw_Terminal_01x04; footprint TerminalBlock:TerminalBlock_bornier-3_P5.08mm -> TerminalBlock:TerminalBlock_MaiXu_MX126-5.0-04P_1x04_P5.00mm
- J8: value grip_con -> DE9_Plug
- R10: value 10k -> 2.2k
- R11: value 3.3k -> 470
- R22: value 0.3 -> 2.2k; footprint Resistor_SMD:R_2512_6332Metric_Pad1.40x3.35mm_HandSolder -> Resistor_SMD:R_0805_2012Metric_Pad1.20x1.40mm_HandSolder
- R40, R88: footprint Resistor_THT:R_Bare_Metal_Element_L16.3mm_W4.8mm_P15.30mm -> Resistor_SMD:R_0805_2012Metric_Pad1.20x1.40mm_HandSolder
- R42: value 200 -> 10; footprint Resistor_THT:R_Bare_Metal_Element_L16.3mm_W4.8mm_P15.30mm -> Resistor_SMD:R_0805_2012Metric_Pad1.20x1.40mm_HandSolder
- R44: value 470 -> 10k
- R45: value 5.1k -> 10k
- R51: value 0.3 -> 470; footprint Resistor_SMD:R_2512_6332Metric_Pad1.40x3.35mm_HandSolder -> Resistor_SMD:R_0805_2012Metric_Pad1.20x1.40mm_HandSolder
- R72, R73, R74, R75, R76, R77: footprint Capacitor_SMD:C_0805_2012Metric_Pad1.18x1.45mm_HandSolder -> Resistor_SMD:R_0805_2012Metric_Pad1.20x1.40mm_HandSolder
- R78, R79: footprint Resistor_SMD:R_1206_3216Metric_Pad1.30x1.75mm_HandSolder -> Resistor_SMD:R_0805_2012Metric_Pad1.20x1.40mm_HandSolder
- SW1, SW2, SW4: footprint BUTT-2:SW_BUTT-2 -> Button_Switch_SMD:SW_DIP_SPSTx01_Slide_6.7x4.1mm_W6.73mm_P2.54mm_LowProfile_JPin
- U12: value AMS1117-5.0 -> L7805; footprint Package_TO_SOT_SMD:SOT-223-3_TabPin2 -> Package_TO_SOT_SMD:TO-252-2
- ZD4: footprint Capacitor_THT:CP_Radial_D10.0mm_P5.00mm_P7.50mm -> Diode_SMD:D_MiniMELF
- moved C7 258.1 mm to (-145.6, 30.3)
- moved J12 229.8 mm to (3.52, 4.53), turned to 0 degrees
- moved Q4 180.2 mm to (216.5, 66.0), turned to -90 degrees
- moved Q8 172.7 mm to (215.8, 91.9)
- moved J2 169.9 mm to (-46.0, 13.0), turned to 180 degrees
- moved R51 169.6 mm to (-140.9, 39.2)
- moved R22 169.3 mm to (-140.9, 36.2)
- moved C13 153.4 mm to (-80.2, 185.5)
- moved C31 153.4 mm to (-80.2, 188.5)
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Connections:
- C1 pad 1: 5v+ -> s5v+
- C34 pad 1: Net-(D6-A) -> Net-(D41-A)
- C6 pad 1: M2_R -> HV
- C6 pad 2: M2_L -> GND
- C7 pad 1: M2_R -> Current_limt2
- C7 pad 2: M2_L -> GND
- C73 pad 2: Net-(U12-VI) -> Net-(U13-IN)
- C74 pad 2: Net-(U12-VO) -> Net-(U13-OUT)
- C77 pad 1: 12v -> HV
- D16 pad 1: 3.3V -> Net-(D16-A1)
- D23 pad 1: 12v -> HV
- D6 pad 2: Net-(D6-A) -> Net-(D41-A)
- F3 pad 1: HV -> Net-(D26-A)
- F4 pad 1: Net-(U12-VO) -> Net-(U13-OUT)
- F5 pad 1: 12v -> HV
- J10 pad 1: HV -> GND
- J10 pad 2: GND -> HV
- J10 pad 5: SCL -> GND
- J10 pad 7: GND -> Mcler
- J10 pad 8: RST -> SCL
- J10 pad G1: (no net) -> GND
- J10 pad G2: (no net) -> GND
- J12 pad 1: HV -> Net-(J12-Pin_1)
- J12 pad 2: detect -> FRQ
- J12 pad 3: GND -> detect
- J4 pad 1: HV -> GND
- J4 pad 2: GND -> HV
- J4 pad 5: SCL -> GND
- J4 pad 7: GND -> Mcler
- J4 pad 8: unconnected-(J4-Pad8) -> SCL
- J4 pad G1: (no net) -> GND
- J4 pad G2: (no net) -> GND
- J8 pad 1: HV -> GND
- J8 pad 2: GND -> HV
- J8 pad 5: SCL -> GND
- J8 pad 7: GND -> Mcler
- J8 pad 8: RST -> SCL
- J8 pad G1: (no net) -> GND
- J8 pad G2: (no net) -> GND
- Q7 pad 1: Net-(Q7-B) -> Net-(D49-K)
- Q7 pad 2: Net-(D6-A) -> Net-(D41-A)
- Q8 pad 3: Net-(D6-A) -> Net-(D41-A)
- Q9 pad 1: buzzing_gnd -> GND
- Q9 pad 7: GND -> buzzing_gnd
- Q9 pad 8: GND -> buzzing_gnd
- R13 pad 1: PGD -> Net-(D46-K)
- R15 pad 1: HV -> 9v+
- R2 pad 1: Motor2_OFF -> Net-(D54-K)
- R22 pad 1: Net-(D2-A) -> Current_limt2
- R22 pad 2: GND -> Net-(R22-Pad2)
- R29 pad 1: Net-(R29-Pad1) -> Net-(R22-Pad2)
- R3 pad 1: M2_S1 -> Net-(D56-K)
- R31 pad 2: Net-(R29-Pad1) -> Net-(R22-Pad2)
- R33 pad 2: Net-(R29-Pad1) -> Net-(R22-Pad2)
- R39 pad 1: 3.3V -> 5v+
- R4 pad 2: 5v+ -> s5v+
- R40 pad 2: HV -> 5v+
- R42 pad 2: HV -> Net-(ZD8-A)
- R44 pad 1: PGD -> SCL
- R44 pad 2: Net-(Q7-B) -> 3.3V
- R45 pad 1: Net-(Q7-B) -> SDA
- R45 pad 2: GND -> 3.3V
- R47 pad 1: HV -> 9v+
- R48 pad 1: Net-(D6-A) -> Net-(D41-A)
- R49 pad 1: Net-(D6-A) -> Net-(D41-A)
- R51 pad 1: Net-(D6-A) -> kill2
- R51 pad 2: GND -> Net-(R51-Pad2)
- R52 pad 1: Net-(D6-A) -> Net-(D41-A)
- R72 pad 1: 12v -> HV
- R73 pad 1: 12v -> HV
- R8 pad 1: 3.3V -> 5v+
- R88 pad 1: Net-(U12-VI) -> Net-(U13-IN)
- R9 pad 1: 5v+ -> s5v+
- U1 pad 7: HV -> Net-(U1-VCC)
- U1 pad 8: 5v+ -> s5v+
- U10 pad 1: 3.3V -> Net-(D16-A1)
- U10 pad 10: unconnected-(U10-D19-Pad10) -> SDA2
- U10 pad 26: unconnected-(U10-D14-Pad26) -> Mcler
- U10 pad 28: unconnected-(U10-D13-Pad28) -> FRQ
- U10 pad 9: unconnected-(U10-D18-Pad9) -> SDL2
- U11 pad 1: (no net) -> Net-(U11-VCC)
- U11 pad 2: (no net) -> Net-(U11-3.3V)
- U11 pad 3: (no net) -> GND
- U11 pad 4: (no net) -> SCL2
- U11 pad 5: (no net) -> SDA2
- U11 pad 6: (no net) -> FSYC
- U11 pad 7: (no net) -> int_a
- U11 pad 8: (no net) -> Data_ready
- U12 pad 1: GND -> Net-(U12-IN)
- U12 pad 2: Net-(U12-VO) -> GND
- U12 pad 3: Net-(U12-VI) -> Net-(U12-OUT)
- U2 pad 2: M2_D1 -> Net-(U2-IN)
- U2 pad 3: INH2 -> tst2
- U3 pad 2: M2_S1 -> Net-(U3-IN)
- U3 pad 3: INH2 -> tst2
- U4 pad 1: Net-(R29-Pad1) -> Net-(R22-Pad2)
- U4 pad 5: (no net) -> Current_limt2
- U4 pad 6: (no net) -> Net-(C93-Pad1)
- U4 pad 7: (no net) -> Net-(R51-Pad2)
- U4 pad 8: HV -> 9v+
- U7 pad 2: M1_D1 -> Net-(U7-IN)
- U7 pad 3: INH1 -> tst1
- U8 pad 2: M1_S1 -> Net-(U8-IN)
- U8 pad 3: INH1 -> tst1
- U9 pad 5: (no net) -> Current_limt1
- U9 pad 6: (no net) -> Net-(C92-Pad1)
- U9 pad 7: (no net) -> Net-(R118-Pad2)
- U9 pad 8: HV -> 9v+
- ZD6 pad 1: 3.3V -> 9v+
Routing:
- net GND: track 1423.4 -> 46.9 mm, vias 8 -> 14
- net HV: track 951.2 -> 0.00 mm, vias 17 -> 20
- net 3.3V: track 716.9 -> 0.00 mm, vias 20 -> 19
- net 5v+: track 639.7 -> 0.00 mm, vias 16 -> 13
- net SDA: track 353.2 -> 0.00 mm
- net SCL: track 346.6 -> 0.00 mm, vias 6 -> 4
- net M1_L: track 302.9 -> 0.00 mm
- net Net-(C41-Pad1): track 289.4 -> 0.00 mm, vias 6 -> 5
- net M1_R: track 255.6 -> 0.00 mm
- net M2_L: track 244.0 -> 0.00 mm
- net Net-(D2-A): track 239.8 -> 0.00 mm, vias 8 -> 7
- net M2_R: track 228.1 -> 0.00 mm
- net Net-(C44-Pad1): track 227.7 -> 0.00 mm, vias 6 -> 5
- net CS: track 204.8 -> 0.00 mm, vias 3 -> 2
- net Net-(D2-K): track 198.8 -> 0.00 mm, vias 5 -> 4
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Other:
- board outline removed

Commit message: Signed-off-by: ahmedsiddyq <morganalpop@gmail.com>
Parts:
- added SW3: SW_Push, Button_Switch_SMD:SW_DIP_SPSTx01_Slide_6.7x4.1mm_W6.73mm_P2.54mm_LowProfile_JPin, F.Cu at (-69.1, 166.5)
- moved U5 153.4 mm to (-25.4, 62.0)
- moved C81 22.2 mm to (-104.0, 27.5)
- moved Q4 7.00 mm to (216.5, 73.0)
- moved U9 5.83 mm to (242.0, 94.0)
- moved Q8 5.02 mm to (216.2, 86.9)
- moved IC1 2.15 mm to (183.2, 49.8), turned to 90 degrees
- moved J10 1.50 mm to (177.5, 156.0)
- moved J8 0.59 mm to (177.5, 123.0)
Routing:
- net GND: track 46.9 -> 77.3 mm

Commit message: lay-out frist low side
Parts:
- added R89: 2.2k, Resistor_SMD:R_0805_2012Metric_Pad1.20x1.40mm_HandSolder, B.Cu at (229.5, 107.0)
- C39, C40, C83, C92, D49, D7, IC1, R118, R52, R53, R54, R55, R57, R58, R59, U4, U9: moved to B.Cu
- RV1, RV2: footprint Potentiometer_SMD:Potentiometer_Vishay_TS53YJ_Vertical -> Potentiometer_THT:Potentiometer_ACP_CA9-H5_Horizontal
- moved D41 414.1 mm to (266.5, 97.5)
- moved C83 386.4 mm to (234.0, 108.5)
- moved C92 381.5 mm to (233.0, 106.5)
- moved R59 377.7 mm to (232.5, 99.0)
- moved RV2 372.7 mm to (245.5, 109.0), turned to 180 degrees
- moved D49 366.4 mm to (220.2, 101.5)
- moved D48 361.8 mm to (212.8, 107.0), turned to 180 degrees
- moved R118 358.7 mm to (228.0, 99.0)
- moved R48 347.4 mm to (222.0, 103.0), turned to -90 degrees
- moved R119 345.6 mm to (214.5, 103.5), turned to 90 degrees
- moved R49 344.1 mm to (219.0, 103.0), turned to -90 degrees
- moved R120 342.2 mm to (211.5, 103.5), turned to -90 degrees
- moved R58 322.3 mm to (240.0, 101.0)
- moved C40 320.3 mm to (242.0, 101.0)
- moved R57 310.6 mm to (237.0, 99.0), turned to 180 degrees
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Connections:
- RV2 pad 2: Net-(C92-Pad1) -> Net-(R89-Pad2)
Routing:
- net Net-(Q3-C): vias 3 -> 2
- net M2_L: vias 6 -> 5
- net GND: vias 14 -> 15
- net 5v+: vias 13 -> 14

Commit message: 7-9 siddyq mid layout
Parts:
- removed D2, D6: 1N4004-T_NRND, Diode_SMD:D_MiniMELF
- removed R103: 10k, Resistor_SMD:R_0805_2012Metric_Pad1.20x1.40mm_HandSolder
- removed ZD10: 3.3v, Diode_SMD:D_MiniMELF
- added D57: 1N4004-T_NRND, Diode_SMD:D_0603_1608Metric_Pad1.05x0.95mm_HandSolder, F.Cu at (46.1, -105.5)
- added D58: 1N4004-T_NRND, Diode_SMD:D_0603_1608Metric_Pad1.05x0.95mm_HandSolder, F.Cu at (197.0, 100.4)
- added D59: 1N4004-T_NRND, Diode_SMD:D_0603_1608Metric_Pad1.05x0.95mm_HandSolder, F.Cu at (207.4, 101.5)
- added D60: 1N4004-T_NRND, Diode_SMD:D_0603_1608Metric_Pad1.05x0.95mm_HandSolder, F.Cu at (198.9, -10.5)
- added D61: 1N4004-T_NRND, Diode_SMD:D_0603_1608Metric_Pad1.05x0.95mm_HandSolder, F.Cu at (203.3, -18.3)
- added D62: 1N4004-T_NRND, Diode_SMD:D_0603_1608Metric_Pad1.05x0.95mm_HandSolder, F.Cu at (-79.0, -15.2)
- added D63: 1N4004-T_NRND, Diode_SMD:D_0603_1608Metric_Pad1.05x0.95mm_HandSolder, F.Cu at (-79.0, -12.7)
- added D64: 1N4004-T_NRND, Diode_SMD:D_0603_1608Metric_Pad1.05x0.95mm_HandSolder, F.Cu at (207.0, 57.6)
- added D65: 1N4004-T_NRND, Diode_SMD:D_0603_1608Metric_Pad1.05x0.95mm_HandSolder, F.Cu at (196.5, 63.9)
- added D66: 1N4004-T_NRND, Diode_SMD:D_0603_1608Metric_Pad1.05x0.95mm_HandSolder, F.Cu at (-74.6, -15.2)
- added D67: 1N4004-T_NRND, Diode_SMD:D_0603_1608Metric_Pad1.05x0.95mm_HandSolder, F.Cu at (-74.6, -12.7)
- added D68: 1N4004-T_NRND, Diode_SMD:D_0603_1608Metric_Pad1.05x0.95mm_HandSolder, F.Cu at (-74.6, -10.1)
- added R121: 10k, Resistor_SMD:R_0805_2012Metric_Pad1.20x1.40mm_HandSolder, F.Cu at (196.0, 105.5)
- added R122: 10k, Resistor_SMD:R_0805_2012Metric_Pad1.20x1.40mm_HandSolder, F.Cu at (208.0, 52.5)
- added R123: 10k, Resistor_SMD:R_0805_2012Metric_Pad1.20x1.40mm_HandSolder, F.Cu at (200.0, 58.0)
- added R124: 10k, Resistor_SMD:R_0805_2012Metric_Pad1.20x1.40mm_HandSolder, F.Cu at (-88.0, -5.85)
- added R125: 10k, Resistor_SMD:R_0805_2012Metric_Pad1.20x1.40mm_HandSolder, F.Cu at (-88.0, -2.90)
- added R126: 10k, Resistor_SMD:R_0805_2012Metric_Pad1.20x1.40mm_HandSolder, F.Cu at (185.0, -14.4)
- added R127: 10k, Resistor_SMD:R_0805_2012Metric_Pad1.20x1.40mm_HandSolder, F.Cu at (185.0, -11.5)
- added R90: 10k, Resistor_SMD:R_0805_2012Metric_Pad1.20x1.40mm_HandSolder, F.Cu at (207.5, 105.0)
- C21, C28, C7, C93, R21, R22, R24, R25, R28, R29, R30, R31, R32, R33, R51: moved to B.Cu
- D3: footprint Diode_SMD:D_MiniMELF -> Diode_SMD:D_0603_1608Metric_Pad1.05x0.95mm_HandSolder; moved to B.Cu
- D46, D47, D48, D49, D54, D55, D56, D7: footprint Diode_SMD:D_MiniMELF -> Diode_SMD:D_0603_1608Metric_Pad1.05x0.95mm_HandSolder
- R11: value 470 -> 220
- RV1, RV2: footprint Potentiometer_THT:Potentiometer_ACP_CA9-H5_Horizontal -> Potentiometer_SMD:Potentiometer_Bourns_3214W_Vertical
- ZD13, ZD14, ZD15, ZD16, ZD17, ZD18, ZD19, ZD20, ZD21, ZD22, ZD23, ZD24, ZD25, ZD26, ZD27, ZD28, ZD29, ZD30, ZD31, ZD32, ZD33, ZD34: footprint Diode_SMD:D_MiniMELF -> Diode_SMD:D_SOD-123
- moved D47 358.3 mm to (221.0, 55.5), turned to -90 degrees
- moved D46 358.2 mm to (219.0, 51.6), turned to 90 degrees
- moved D42 357.8 mm to (216.5, 59.8), turned to 90 degrees
- moved R91 348.8 mm to (203.5, 100.5), turned to -90 degrees
- moved R92 344.9 mm to (200.0, 100.5), turned to 90 degrees
- moved R94 343.0 mm to (205.5, 61.5)
- moved R93 342.5 mm to (201.5, 61.5), turned to 180 degrees
- moved R22 339.9 mm to (198.5, 56.0)
- moved ZD23 339.8 mm to (204.0, 105.3), turned to -90 degrees
- moved C7 337.7 mm to (191.5, 51.0), turned to 90 degrees
- moved C93 334.2 mm to (193.0, 48.0), turned to 180 degrees
- moved ZD24 333.6 mm to (198.5, 105.7), turned to -90 degrees
- moved R20 333.5 mm to (213.0, 58.0), turned to 90 degrees
- moved R51 333.3 mm to (192.0, 55.5), turned to 90 degrees
- moved R18 330.9 mm to (209.9, 58.0), turned to 90 degrees
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Connections:
- D55 pad 1: unconnected-(D55-K-Pad1) -> Net-(D55-K)
- D55 pad 2: unconnected-(D55-A-Pad2) -> M1_S1
- R100 pad 2: HV -> Net-(D67-K)
- R27 pad 1: HV -> Net-(D66-K)
- R34 pad 1: M1_S1 -> Net-(D55-K)
- R35 pad 1: Motor1_OFF -> Net-(D57-K)
- R91 pad 1: INH2 -> Net-(D59-K)
- R92 pad 1: M2_D1 -> Net-(D58-K)
- R93 pad 2: INH2 -> Net-(D65-K)
- R94 pad 2: M2_S1 -> Net-(D64-K)
- R96 pad 2: M1_S1 -> Net-(D60-K)
- R97 pad 1: INH1 -> Net-(D63-K)
- R98 pad 1: M1_D1 -> Net-(D62-K)
- ZD15 pad 1: M1_S1 -> Net-(D55-K)
- ZD16 pad 1: Motor1_OFF -> Net-(D57-K)
- ZD8 pad 1: HV -> Net-(D67-K)
Routing:
- net voltge_sen: vias 2 -> 0
- net s5v+: vias 1 -> 0
- net kill2: vias 4 -> 0
- net error 2: vias 3 -> 0
- net error 1: vias 4 -> 0
- net detect: vias 2 -> 0
- net buzzing_gnd: vias 3 -> 0
- net buzz: vias 4 -> 0
- net SW4: vias 5 -> 0
- net SW3: vias 3 -> 0
- net SW2: vias 5 -> 0
- net SW1: vias 2 -> 0
- net SDA: vias 3 -> 0
- net SCL: vias 4 -> 0
- net PWM: vias 3 -> 0
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