File: circuts/SBC/SBC.kicad_pcb (KiCad board)
At the start: 2 copper layers, 371 parts, among them IC1 PIC16F15243-I_SS, J1 640456-3, J10 DE9_Plug, J11 buzzer, J12 Screw_Terminal_01x04, J13 12v Power, J14 5v Power, J15 Barrel_Jack_MountingPin, J2 B5B-XH-A_LF__SN_, J3 Power, J4 DE9_Plug, J5 OSTTC060162, J6 XT60-M, J7 OSTTC060162, J8 DE9_Plug, J9 Conn_02x04_Odd_Even, Q1 MMBTA06, Q10 BC817, Q2 MMBTA06, Q3 MMBTA06, Q4 IRFS4227, Q5 MMBTA06, Q6 MMBTA06, Q7 MMBTA06, Q8 IRFS4227, Q9 FDS4559, SW1 SW_Push, SW2 SW_Push, SW3 SW_Push, SW4 SW_Push, SW5 SW_Push, SW6 rst, SW7 SW_Push, U1 UC3843, U10 ESP32-DEVKIT-V1, U12 L7805, U13 L7805, U14 L7809, U2 BTS7960B, U3 BTS7960B, U4 LM358DT, U5 AMS1117-3.3, U7 BTS7960B, U8 BTS7960B, U9 LM358DT

Commit message: test
Parts:
- moved D61 94.0 mm to (126.3, 35.7)
- moved D60 94.0 mm to (121.9, 43.5)
- moved R126 94.0 mm to (108.0, 39.5)
- moved R127 94.0 mm to (108.0, 42.5)
- moved R50 94.0 mm to (143.5, 39.0)
- moved R56 94.0 mm to (140.5, 39.0)
- moved R95 94.0 mm to (93.5, 37.5)
- moved R96 94.0 mm to (93.5, 40.5)
- moved ZD29 94.0 mm to (98.3, 39.2)
- moved ZD30 94.0 mm to (98.3, 42.5)
Changed lines of the file:
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@@
 	(footprint "Diode_SMD:D_SOD-123"
 		(layer "F.Cu")
-		(at 175.35 -11.5)
+		(at 98.35 42.5)
 		(descr "SOD-123")
 		(tags "SOD-123")
@@
 	(footprint "Resistor_SMD:R_0805_2012Metric_Pad1.20x1.40mm_HandSolder"
 		(layer "F.Cu")
-		(at 185 -14.45)
+		(at 108 39.55)
 		(descr "Resistor SMD 0805 (2012 Metric), square (rectangular) end terminal, IPC-7351 nominal with elongated pad for handsoldering. (Body size source: IPC-SM-782 page 72, https://www.pcb-3d.com/wordpress/wp-content/uploads/ipc-sm-782a_amendment_1_and_2.pdf), generated with kicad-footprint-generator")
 		(tags "resistor handsolder")
@@
 	(footprint "Resistor_SMD:R_0805_2012Metric_Pad1.20x1.40mm_HandSolder"
 		(layer "F.Cu")
-		(at 170.5 -16.45)
+		(at 93.5 37.55)
 		(descr "Resistor SMD 0805 (2012 Metric), square (rectangular) end terminal, IPC-7351 nominal with elongated pad for handsoldering. (Body size source: IPC-SM-782 page 72, https://www.pcb-3d.com/wordpress/wp-content/uploads/ipc-sm-782a_amendment_1_and_2.pdf), generated with kicad-footprint-generator")
 		(tags "resistor handsolder")
@@
 	(footprint "Diode_SMD:D_0603_1608Metric_Pad1.05x0.95mm_HandSolder"
 		(layer "F.Cu")
-		(at 203.27 -18.27)
+		(at 126.27 35.73)
 		(descr "Diode SMD 0603 (1608 Metric), square (rectangular) end terminal, IPC-7351 nominal, (Body size source: http://www.tortai-tech.com/upload/download/2011102023233369053.pdf), generated with kicad-footprint-generator")
 		(tags "diode handsolder")
@@
 	(footprint "Diode_SMD:D_SOD-123"
 		(layer "F.Cu")
-		(at 175.35 -14.84)
+		(at 98.35 39.16)
 		(descr "SOD-123")
 		(tags "SOD-123")
@@
 	(footprint "Resistor_SMD:R_0805_2012Metric_Pad1.20x1.40mm_HandSolder"
 		(layer "F.Cu")
-		(at 185 -11.5)
+		(at 108 42.5)
 		(descr "Resistor SMD 0805 (2012 Metric), square (rectangular) end terminal, IPC-7351 nominal with elongated pad for handsoldering. (Body size source: IPC-SM-782 page 72, https://www.pcb-3d.com/wordpress/wp-content/uploads/ipc-sm-782a_amendment_1_and_2.pdf), generated with kicad-footprint-generator")
 		(tags "resistor handsolder")
@@
 	(footprint "Resistor_SMD:R_0805_2012Metric_Pad1.20x1.40mm_HandSolder"
 		(layer "F.Cu")
-		(at 170.5 -13.5)
+		(at 93.5 40.5)
 		(descr "Resistor SMD 0805 (2012 Metric), square (rectangular) end terminal, IPC-7351 nominal with elongated pad for handsoldering. (Body size source: IPC-SM-782 page 72, https://www.pcb-3d.com/wordpress/wp-content/uploads/ipc-sm-782a_amendment_1_and_2.pdf), generated with kicad-footprint-generator")
 		(tags "resistor handsolder")
@@
 	(footprint "Diode_SMD:D_0603_1608Metric_Pad1.05x0.95mm_HandSolder"
 		(layer "F.Cu")
-		(at 198.875 -10.5)
+		(at 121.875 43.5)
 		(descr "Diode SMD 0603 (1608 Metric), square (rectangular) end terminal, IPC-7351 nominal, (Body size source: http://www.tortai-tech.com/upload/download/2011102023233369053.pdf), generated with kicad-footprint-generator")
 		(tags "diode handsolder")
@@
 	(footprint "Resistor_SMD:R_0805_2012Metric_Pad1.20x1.40mm_HandSolder"
 		(layer "F.Cu")
-		(at 220.5 -15 -90)
+		(at 143.5 39 -90)
 		(descr "Resistor SMD 0805 (2012 Metric), square (rectangular) end terminal, IPC-7351 nominal with elongated pad for handsoldering. (Body size source: IPC-SM-782 page 72, https://www.pcb-3d.com/wordpress/wp-content/uploads/ipc-sm-782a_amendment_1_and_2.pdf), generated with kicad-footprint-generator")
 		(tags "resistor handsolder")
@@
 	(footprint "Resistor_SMD:R_0805_2012Metric_Pad1.20x1.40mm_HandSolder"
 		(layer "F.Cu")
-		(at 217.5 -15 -90)
+		(at 140.5 39 -90)
 		(descr "Resistor SMD 0805 (2012 Metric), square (rectangular) end terminal, IPC-7351 nominal with elongated pad for handsoldering. (Body size source: IPC-SM-782 page 72, https://www.pcb-3d.com/wordpress/wp-content/uploads/ipc-sm-782a_amendment_1_and_2.pdf), generated with kicad-footprint-generator")
 		(tags "resistor handsolder")

Commit message: Signed-off-by: ahmedsiddyq <morganalpop@gmail.com>
Parts:
- added D6: 1N4004-T_NRND, Diode_SMD:D_0603_1608Metric_Pad1.05x0.95mm_HandSolder, F.Cu at (489.0, -133.9)
- IC1: moved to F.Cu
- moved C86 612.2 mm to (466.5, 37.0), turned to -90 degrees
- moved C84 612.1 mm to (466.5, 33.5), turned to 90 degrees
- moved D27 608.1 mm to (462.5, 33.2), turned to -90 degrees
- moved D28 605.2 mm to (459.7, 33.8), turned to -90 degrees
- moved U12 604.5 mm to (473.9, 35.0), turned to 0 degrees
- moved R104 597.9 mm to (466.5, 41.5), turned to -90 degrees
- moved SW6 596.7 mm to (405.5, -85.0)
- moved ZD11 588.9 mm to (462.0, 39.8), turned to 90 degrees
- moved R106 580.4 mm to (466.0, 29.0), turned to 90 degrees
- moved C10 559.1 mm to (538.8, -85.1)
- moved C15 559.1 mm to (463.2, -81.1)
- moved C22 559.1 mm to (486.1, -112.1)
- moved C90 559.1 mm to (441.9, -110.6)
- moved D1 559.1 mm to (452.3, -81.5)
- moved D66 559.1 mm to (462.7, -170.0)
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Connections:
- D61 pad 1: unconnected-(D61-K-Pad1) -> Net-(D61-K)
- J2 pad 2: 3.3V -> Net-(D6-A)
- R95 pad 2: INH1 -> Net-(D61-K)
Routing:
- net GND: track 77.3 -> 69.7 mm
- net Mcler: track 0.00 -> 7.60 mm
