File: circuts/SBC/SBC.kicad_pcb (KiCad board)
At the start: 2 copper layers, 372 parts, among them IC1 PIC16F15243-I_SS, J1 640456-3, J10 DE9_Plug, J11 buzzer, J12 Screw_Terminal_01x04, J13 12v Power, J14 5v Power, J15 Barrel_Jack_MountingPin, J2 B5B-XH-A_LF__SN_, J3 Power, J4 DE9_Plug, J5 OSTTC060162, J6 XT60-M, J7 OSTTC060162, J8 DE9_Plug, J9 Conn_02x04_Odd_Even, Q1 MMBTA06, Q10 BC817, Q2 MMBTA06, Q3 MMBTA06, Q4 IRFS4227, Q5 MMBTA06, Q6 MMBTA06, Q7 MMBTA06, Q8 IRFS4227, Q9 FDS4559, SW1 SW_Push, SW2 SW_Push, SW3 SW_Push, SW4 SW_Push, SW5 SW_Push, SW6 rst, SW7 SW_Push, U1 UC3843, U10 ESP32-DEVKIT-V1, U12 L7805, U13 L7805, U14 L7809, U2 BTS7960B, U3 BTS7960B, U4 LM358DT, U5 AMS1117-3.3, U7 BTS7960B, U8 BTS7960B, U9 LM358DT

Commit message: now
Parts:
- moved D25 709.1 mm to (445.8, -157.5), turned to 180 degrees
- moved ZD9 694.8 mm to (448.8, -165.5), turned to 180 degrees
- moved R42 680.1 mm to (438.0, -170.0), turned to 90 degrees
- moved R100 675.2 mm to (438.0, -175.5), turned to -90 degrees
- moved C31 635.7 mm to (445.5, -169.0)
- moved C33 634.3 mm to (444.5, -165.0), turned to -90 degrees
- moved C82 632.5 mm to (456.5, -160.5), turned to -90 degrees
- moved R99 620.1 mm to (450.0, -157.5), turned to 90 degrees
- moved ZD6 609.1 mm to (453.0, -160.8), turned to 90 degrees
- moved ZD8 601.6 mm to (434.5, -175.2), turned to 90 degrees
- moved D67 532.9 mm to (434.5, -170.1), turned to -90 degrees
- moved U14 476.3 mm to (449.5, -161.5), turned to 180 degrees
- moved J2 3.28 mm to (491.5, -145.0)
Connections:
- C82 pad 2: Net-(D25-A) -> 9v+

Commit message: almost ready
Parts:
- removed D21, D22, D23, D27, D28: 1N4004-T_NRND, Diode_SMD:D_MiniMELF
- removed F6: 1A, Capacitor_SMD:C_0603_1608Metric_Pad1.08x0.95mm_HandSolder
- removed J12: Screw_Terminal_01x04, TerminalBlock:TerminalBlock_MaiXu_MX126-5.0-04P_1x04_P5.00mm
- removed Q9: FDS4559, Package_SO:SOIC-8_3.9x4.9mm_P1.27mm
- removed R44, R45, R81, R82, R83: 10k, Resistor_SMD:R_0805_2012Metric_Pad1.20x1.40mm_HandSolder
- removed ZD32: 3.3v, Diode_SMD:D_SOD-123
- added C94: C, Capacitor_SMD:C_0805_2012Metric_Pad1.18x1.45mm_HandSolder, B.Cu at (253.2, 118.8)
- added D2: 1N4004-T_NRND, Diode_SMD:D_0603_1608Metric_Pad1.05x0.95mm_HandSolder, F.Cu at (163.2, 46.9)
- added Q11: AO3400A, Package_TO_SOT_SMD:SOT-23_Handsoldering, B.Cu at (245.4, 120.2)
- added ZD10: BZV55B4V7, Diode_SMD:D_MiniMELF, F.Cu at (343.0, 124.4)
- added ZD35: BZV55B4V7, Diode_SMD:D_MiniMELF, F.Cu at (343.0, 127.8)
- added ZD36: BZV55B4V7, Diode_SMD:D_MiniMELF, B.Cu at (222.2, 122.5)
- C1, C10, C15, C31, C33, C69, C70, C71, C72, C75, C76, C77, C79, C8, C80, C82, C90, D10, D11, D16, D17, D18, D25, D45, D6, D66, D67, D68, F5, F7, IC1, Q10, R1, R10, R100, R107, R108, R11, R114, R16, R17, R19, R23, R26, R27, R4, R42, R60, R61, R62, R63, R64, R66, R67, R68, R70, R71, R72, R73, R74, R80, R9, R99, U1, ZD1, ZD2, ZD3, ZD33, ZD34, ZD4, ZD6, ZD8, ZD9: moved to B.Cu
- C11, C18, C4, C45, C46, C47: footprint Capacitor_SMD:C_0805_2012Metric_Pad1.18x1.45mm_HandSolder -> Capacitor_SMD:C_0201_0603Metric_Pad0.64x0.40mm_HandSolder
- C12: footprint Capacitor_THT:CP_Radial_D8.0mm_P5.00mm -> Capacitor_THT:CP_Radial_D4.0mm_P1.50mm
- C2, C78: footprint Capacitor_SMD:C_0805_2012Metric_Pad1.18x1.45mm_HandSolder -> Capacitor_SMD:C_0201_0603Metric_Pad0.64x0.40mm_HandSolder; moved to B.Cu
- C22: value 2uf -> 1nf; footprint Capacitor_THT:CP_Radial_D8.0mm_P5.00mm -> Capacitor_SMD:C_0201_0603Metric_Pad0.64x0.40mm_HandSolder; moved to B.Cu
- C26, C36, C87: footprint Resistor_SMD:R_0805_2012Metric_Pad1.20x1.40mm_HandSolder -> Capacitor_SMD:C_0201_0603Metric_Pad0.64x0.40mm_HandSolder
- C41, C42, C43, C44: footprint Resistor_SMD:R_0805_2012Metric_Pad1.20x1.40mm_HandSolder -> Capacitor_SMD:C_0201_0603Metric_Pad0.64x0.40mm_HandSolder; moved to B.Cu
- D19: value 20v zener -> SMAJ6.5A; moved to B.Cu
- D20: value 5.6v zener -> 1N4004-T_NRND; moved to B.Cu
- J13: value 12v Power -> Conn_01x04_Pin; footprint 282837-2:TE_282837-2 -> Connector_PinSocket_2.54mm:PinSocket_1x04_P2.54mm_Vertical
- ZD31: value 3.3v -> BZV55B4V7; footprint Diode_SMD:D_SOD-123 -> Diode_SMD:D_MiniMELF; moved to B.Cu
- moved D30 613.0 mm to (361.0, -49.6)
- moved D31 613.0 mm to (361.0, -46.2)
- moved D32 605.5 mm to (353.2, -46.0)
- moved D29 604.8 mm to (353.0, -49.8)
- moved D39 589.9 mm to (219.0, -378.8)
- moved D40 587.1 mm to (212.8, -378.7)
- moved D37 583.6 mm to (219.2, -374.8)
- moved D38 580.5 mm to (212.8, -374.8)
- moved C16 567.8 mm to (359.2, -296.8)
- moved C17 567.8 mm to (422.3, -289.2)
- moved C18 567.8 mm to (407.8, -295.8)
- moved C19 567.8 mm to (379.0, -338.8)
- moved C20 567.8 mm to (334.8, -321.2)
- moved C23 567.8 mm to (371.0, -336.8)
- moved C24 567.8 mm to (368.5, -328.2)
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Connections:
- C77 pad 1: HV -> buzzing_vcc
- D19 pad 1: HV -> buzzing_vcc
- D19 pad 2: GND -> buzzing_gnd
- D20 pad 1: 5v+ -> buzzing_vcc
- D20 pad 2: GND -> HV
- F5 pad 1: HV -> buzzing_vcc
- J13 pad 1: Net-(J13-Pin_1) -> GND
- J13 pad 2: GND -> detect
- J15 pad 1: Net-(J13-Pin_1) -> HV
- R114 pad 1: HV -> buzzing_vcc
- R117 pad 2: Net-(J12-Pin_1) -> Net-(J13-Pin_4)
- R72 pad 1: HV -> buzzing_vcc
- R73 pad 1: HV -> buzzing_vcc
- R79 pad 1: SDL -> SCL
- U10 pad 14: SDL -> SCL
- ZD31 pad 1: SCL -> SDA
Routing:
- net Mcler: track 7.60 -> 0.00 mm
- net GND: track 69.7 -> 62.1 mm

Commit message: bom has been deplated
Parts:
- removed C55, C56: 100uf, Capacitor_SMD:CP_Elec_4x4.5
- removed C58, C59: 470uf, Capacitor_SMD:CP_Elec_4x4.5
- removed C61, C62: 1000uf, Capacitor_SMD:CP_Elec_4x4.5
- removed D9: 1N4004-T_NRND, Diode_SMD:D_MiniMELF
- removed R78, R79: 10k, Resistor_SMD:R_0805_2012Metric_Pad1.20x1.40mm_HandSolder
- added C100: 2uf, Resistor_SMD:R_0805_2012Metric_Pad1.20x1.40mm_HandSolder, B.Cu at (201.2, 64.0)
- added C101: 100nf, Capacitor_SMD:C_0805_2012Metric_Pad1.18x1.45mm_HandSolder, B.Cu at (206.0, 65.5)
- added C102: 2uf, Resistor_SMD:R_0805_2012Metric_Pad1.20x1.40mm_HandSolder, B.Cu at (231.5, 93.8)
- added C103: 2uf, Resistor_SMD:R_0805_2012Metric_Pad1.20x1.40mm_HandSolder, B.Cu at (201.5, 95.5)
- added C104: 100nf, Capacitor_SMD:C_0805_2012Metric_Pad1.18x1.45mm_HandSolder, B.Cu at (226.7, 94.0)
- added C105: 100nf, Capacitor_SMD:C_0805_2012Metric_Pad1.18x1.45mm_HandSolder, B.Cu at (206.2, 94.0)
- added C95: 2uf, Capacitor_SMD:C_0805_2012Metric_Pad1.18x1.45mm_HandSolder, B.Cu at (164.2, 147.5)
- added C96: 470uf, Capacitor_THT:CP_Radial_D8.0mm_P5.00mm, F.Cu at (189.1, 98.2)
- added C97: 470uf, Capacitor_THT:CP_Radial_D8.0mm_P5.00mm, F.Cu at (239.2, 67.5)
- added C98: 100nf, Capacitor_SMD:C_0805_2012Metric_Pad1.18x1.45mm_HandSolder, B.Cu at (231.5, 64.2)
- added C99: 2uf, Resistor_SMD:R_0805_2012Metric_Pad1.20x1.40mm_HandSolder, B.Cu at (226.2, 64.2)
- added D21: BZV55B3V3, Diode_SMD:D_MiniMELF, B.Cu at (252.5, 155.0)
- C17, C18, C20, C25, C29, C36, C38, C46, C48, C49, C50, C52, C53, C67, C85, C89, D24, D26, D29, D30, D31, D32, D37, D38, D39, D40, D57, F3, R101, R102, R113, R117, R65, R69, ZD17, ZD18: moved to B.Cu
- C24: value 470uf -> 100nf; footprint Capacitor_THT:CP_Radial_D8.0mm_P5.00mm -> Resistor_SMD:R_0805_2012Metric_Pad1.20x1.40mm_HandSolder; moved to B.Cu
- C31, C33, ZD9: moved to F.Cu
- C54: value 100uf -> 470uf; footprint Capacitor_SMD:CP_Elec_4x4.5 -> Capacitor_THT:CP_Radial_D8.0mm_P5.00mm
- C57: footprint Capacitor_SMD:CP_Elec_4x4.5 -> Capacitor_THT:CP_Radial_D8.0mm_P5.00mm
- C60: value 1000uf -> 470uf; footprint Capacitor_SMD:CP_Elec_4x4.5 -> Capacitor_THT:CP_Radial_D8.0mm_P5.00mm
- D8: value 20v zener -> SMAJ6.5A; moved to B.Cu
- moved C63 685.2 mm to (253.5, 155.0)
- moved C66 684.7 mm to (258.0, 151.5), turned to 180 degrees
- moved R75 679.8 mm to (261.2, 144.8), turned to 180 degrees
- moved D12 679.1 mm to (265.0, 144.8), turned to 180 degrees
- moved C51 665.0 mm to (235.2, 95.8), turned to -90 degrees
- moved R77 657.9 mm to (239.5, 135.2), turned to -90 degrees
- moved D13 650.9 mm to (237.0, 135.8), turned to 90 degrees
- moved C64 629.4 mm to (198.3, 147.8), turned to 180 degrees
- moved C54 619.7 mm to (253.5, 101.5), turned to -90 degrees
- moved C52 611.2 mm to (180.7, 126.2)
- moved C49 609.8 mm to (199.0, 154.8), turned to 90 degrees
- moved C67 609.3 mm to (182.7, 149.5)
- moved C45 608.1 mm to (198.5, 63.5), turned to 90 degrees
- moved C53 607.7 mm to (176.0, 149.5), turned to 180 degrees
- moved C68 607.0 mm to (182.0, 127.2)
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Connections:
- C24 pad 1: HV -> 3.3V
- C65 pad 1: 3.3V -> GND
- C65 pad 2: GND -> Net-(U11-3.3V)
Routing:
- net GND: track 62.1 -> 0.00 mm

Commit message: siddyq at fanaly
Parts:
- added C11: 1nf, Capacitor_SMD:C_0201_0603Metric_Pad0.64x0.40mm_HandSolder, F.Cu at (243.5, 80.0)
- added C13: 2uf, Capacitor_SMD:C_0805_2012Metric_Pad1.18x1.45mm_HandSolder, F.Cu at (236.8, 79.8)
- added C4: 1nf, Capacitor_SMD:C_0201_0603Metric_Pad0.64x0.40mm_HandSolder, F.Cu at (173.8, 78.3)
- added C5: 2uf, Capacitor_SMD:C_0805_2012Metric_Pad1.18x1.45mm_HandSolder, B.Cu at (169.5, 78.3)
- added C9: 100nf, Capacitor_SMD:C_0805_2012Metric_Pad1.18x1.45mm_HandSolder, B.Cu at (263.0, 78.8)
- C63, C84, C86, D2, R104, R106, U12, ZD11: moved to B.Cu
- R19: moved to F.Cu
- moved C63 67.2 mm to (186.2, 154.7), turned to 90 degrees
- moved R122 19.6 mm to (188.2, 47.2), turned to 180 degrees
- moved R112 19.3 mm to (177.2, 55.0), turned to -90 degrees
- moved ZD33 16.6 mm to (170.2, 153.8), turned to 90 degrees
- moved C3 13.3 mm to (195.5, 78.5)
- moved D2 9.62 mm to (173.0, 48.9)
- moved J1 9.28 mm to (185.8, 68.0), turned to 0 degrees
- moved R42 9.03 mm to (184.2, 40.2), turned to 90 degrees
- moved R104 8.63 mm to (164.0, 50.2)
- moved C86 7.60 mm to (163.8, 45.5), turned to -90 degrees
- moved R25 7.46 mm to (207.2, 44.8), turned to 90 degrees
- moved R19 7.35 mm to (242.2, 57.5), turned to 90 degrees
- moved C97 6.89 mm to (245.5, 64.6), turned to -90 degrees
- moved C24 6.45 mm to (169.0, 58.8)
- moved R100 6.33 mm to (179.0, 41.8), turned to -90 degrees
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Connections:
- C24 pad 1: 3.3V -> 3.3v
- C35 pad 1: 3.3V -> 3.3v
- C36 pad 1: 3.3V -> 3.3v
- C37 pad 1: 3.3V -> 3.3v
- C38 pad 2: 3.3V -> 3.3v
- C47 pad 1: 3.3V -> 3.3v
- C50 pad 1: 3.3V -> 3.3v
- C53 pad 1: 3.3V -> 3.3v
- C68 pad 1: 3.3V -> 3.3v
- D6 pad 1: 3.3V -> 3.3v
- IC1 pad 1: 3.3V -> 3.3v
- J10 pad 4: 3.3V -> 3.3v
- J4 pad 4: 3.3V -> 3.3v
- J8 pad 4: 3.3V -> 3.3v
- J9 pad 2: 3.3V -> 3.3v
- R101 pad 1: 3.3V -> 3.3v
- R105 pad 2: 3.3V -> 3.3v
- R107 pad 2: 3.3V -> 3.3v
- R113 pad 1: 3.3V -> 3.3v
- R64 pad 1: 3.3V -> 3.3v
- R65 pad 2: 3.3V -> 3.3v
- R66 pad 1: 3.3V -> Net-(R66-Pad1)
- R67 pad 1: 3.3V -> 3.3v
- R68 pad 1: 3.3V -> Net-(R66-Pad1)
- R69 pad 2: 3.3V -> 3.3v
- R70 pad 2: 3.3V -> 3.3v
- R71 pad 2: 3.3V -> 3.3v
- R76 pad 2: 3.3V -> 3.3v
- R80 pad 2: 3.3V -> 3.3v
- ZD5 pad 1: 3.3V -> 3.3v
Routing:
- net GND: track 0.00 -> 594.0 mm, vias 0 -> 10
- net 5v+: track 0.00 -> 103.5 mm, vias 0 -> 4
- net 3.3v: track 0.00 -> 100.3 mm, vias 0 -> 5
- net HV: track 0.00 -> 94.7 mm, vias 0 -> 2
- net M2_R: track 0.00 -> 72.9 mm, vias 0 -> 1
- net M2_L: track 0.00 -> 62.3 mm
- net M1_R: track 0.00 -> 59.6 mm
- net M1_L: track 0.00 -> 47.1 mm
- net Mcler: track 0.00 -> 39.5 mm
- net tst1: track 0.00 -> 36.9 mm, vias 0 -> 5
- net buzzing_vcc: track 0.00 -> 36.5 mm
- net tst2: track 0.00 -> 35.8 mm
- net INH2: track 0.00 -> 34.8 mm, vias 0 -> 2
- net buzzing_gnd: track 0.00 -> 28.0 mm
- net Net-(R22-Pad2): track 0.00 -> 27.4 mm
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Other:
- board outline added: 108.2 x 121.5 mm
- board text added: "1N4004-T_NRND"
- board text added: "C12"

Commit message: BEFOR R MOTER EDIT OP-AMP
Parts:
- moved R21 7.72 mm to (209.5, 96.8)
- moved C41 5.53 mm to (263.8, 67.0), turned to 180 degrees
- moved C50 4.54 mm to (175.2, 104.0), turned to 90 degrees
- moved C42 4.00 mm to (263.8, 70.8), turned to 180 degrees
- moved ZD18 2.00 mm to (170.7, 104.5)
- moved C88 1.54 mm to (176.8, 46.4)
- moved R92 1.52 mm to (198.5, 100.2)
- moved C29 1.41 mm to (177.8, 104.0)
- moved ZD20 1.25 mm to (250.2, 53.6)
- moved R30 1.03 mm to (201.2, 59.5)
- moved R38 0.90 mm to (248.8, 97.0), turned to 90 degrees
- moved R25 0.79 mm to (207.5, 45.5)
- moved D39 0.56 mm to (163.8, 89.8)
- moved D56 0.56 mm to (190.4, 60.2)
- moved ZD14 0.56 mm to (185.6, 55.0)
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Routing:
- net HV: track 94.7 -> 359.2 mm, vias 2 -> 9
- net GND: track 594.0 -> 856.4 mm, vias 10 -> 21
- net 5v+: track 103.5 -> 211.0 mm, vias 4 -> 5
- net error 2: track 0.00 -> 61.0 mm, vias 0 -> 2
- net M1_L: track 47.1 -> 97.2 mm, vias 0 -> 1
- net Net-(D41-K): track 15.2 -> 62.5 mm, vias 1 -> 2
- net M2_L: track 62.3 -> 98.9 mm, vias 0 -> 1
- net A1: track 0.00 -> 33.7 mm, vias 0 -> 2
- net M1_R: track 59.6 -> 90.1 mm
- net M2_S1: track 0.00 -> 28.4 mm, vias 0 -> 3
- net 3.3v: track 100.3 -> 125.3 mm, vias 5 -> 7
- net B1: track 0.00 -> 24.8 mm, vias 0 -> 2
- net M2_R: track 72.9 -> 92.2 mm
- net Net-(C44-Pad1): track 0.00 -> 18.8 mm
- net Net-(C21-Pad2): track 9.58 -> 27.6 mm, vias 0 -> 2
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
Commit message: siddyq has done almost done 7-25
Parts:
- removed C4 (x2): 1nf, Capacitor_SMD:C_0201_0603Metric_Pad0.64x0.40mm_HandSolder
- removed the C9 at (249.0, 80.0)
- removed J9: Conn_02x04_Odd_Even, Connector_PinHeader_2.54mm:PinHeader_2x04_P2.54mm_Vertical
- removed R108: 1k, Resistor_SMD:R_0805_2012Metric_Pad1.20x1.40mm_HandSolder
- removed R48: 0.3, Resistor_SMD:R_2512_6332Metric_Pad1.40x3.35mm_HandSolder
- added C55: 2uf, Capacitor_SMD:C_0805_2012Metric_Pad1.18x1.45mm_HandSolder, F.Cu at (259.8, 80.2)
- added C56: 2uf, Capacitor_SMD:C_0805_2012Metric_Pad1.18x1.45mm_HandSolder, F.Cu at (172.6, 78.8)
- added C58: 2uf, Capacitor_SMD:C_0805_2012Metric_Pad1.18x1.45mm_HandSolder, F.Cu at (174.7, 78.9)
- C1, C10, C2, C21, C28, C38, C39, C40, C7, C8, C82, C83, C84, C86, C89, C92, C93, C95, D2, D25, D3, D67, D68, D7, IC1, R1, R10, R102, R104, R106, R107, R11, R118, R17, R22, R24, R25, R28, R29, R31, R32, R33, R4, R42, R51, R52, R53, R54, R55, R57, R58, R59, R61, R62, R65, R80, R89, R9, R99, U1, U12, U4, U9, ZD1, ZD11, ZD2, ZD6, ZD8: moved to F.Cu
- C34, C35, C45, C47, C65, D15, D48, J1, J8, Q7, R119, R120, R47, ZD10, ZD19, ZD20, ZD21, ZD22, ZD27, ZD9: moved to B.Cu
- C46: value 1nf -> 2uf; footprint Capacitor_SMD:C_0201_0603Metric_Pad0.64x0.40mm_HandSolder -> Capacitor_SMD:C_0805_2012Metric_Pad1.18x1.45mm_HandSolder; moved to F.Cu
- moved R107 91.6 mm to (166.3, 41.1), turned to -90 degrees
- moved C46 90.9 mm to (237.4, 80.1), turned to 90 degrees
- moved C10 88.0 mm to (166.6, 45.8), turned to 90 degrees
- moved R100 87.5 mm to (266.3, 47.9), turned to 90 degrees
- moved ZD22 86.5 mm to (165.9, 63.8), turned to 180 degrees
- moved ZD8 85.9 mm to (266.3, 48.4), turned to -90 degrees
- moved D66 85.0 mm to (182.0, 91.9), turned to -90 degrees
- moved ZD2 84.1 mm to (171.0, 45.7), turned to 90 degrees
- moved ZD21 83.2 mm to (169.3, 58.6), turned to 180 degrees
- moved R106 81.6 mm to (252.2, 41.7)
- moved C84 80.5 mm to (248.6, 40.1), turned to 0 degrees
- moved C36 80.2 mm to (166.1, 41.1), turned to 90 degrees
- moved R42 80.0 mm to (263.5, 51.2), turned to 0 degrees
- moved C31 79.9 mm to (264.1, 47.4), turned to -90 degrees
- moved D2 79.0 mm to (251.9, 45.5), turned to -90 degrees
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Connections:
- C46 pad 1: 5v+ -> M1_R
- C46 pad 2: GND -> M1_L
- SW6 pad 1: Net-(R108-Pad1) -> Mcler
- U10 pad 10: SDA2 -> int_a
- U10 pad 12: care -> care0
- U10 pad 13: care -> care0
- U10 pad 23: int_a -> unconnected-(U10-D25-Pad23)
- U10 pad 24: FSYC -> unconnected-(U10-D26-Pad24)
- U10 pad 27: care -> careuu
- U10 pad 3: care -> carett
- U10 pad 4: care -> carei
- U10 pad 6: unconnected-(U10-RX2-Pad6) -> SCL2
- U10 pad 7: unconnected-(U10-TX2-Pad7) -> SDA2
- U10 pad 9: SDL2 -> FSYC
Routing:
- net GND: track 856.4 -> 1379.4 mm, vias 21 -> 32
- net 5v+: track 211.0 -> 644.8 mm, vias 5 -> 17
- net 3.3v: track 125.3 -> 462.8 mm, vias 7 -> 11
- net HV: track 359.2 -> 687.4 mm, vias 9 -> 17
- net SCL: track 10.1 -> 266.8 mm, vias 0 -> 4
- net Mcler: track 32.4 -> 259.8 mm, vias 0 -> 4
- net M1_current_sen: track 8.56 -> 179.6 mm, vias 0 -> 3
- net 9v+: track 40.0 -> 203.6 mm, vias 2 -> 6
- net SDA: track 16.0 -> 169.3 mm, vias 0 -> 3
- net CS: track 0.00 -> 137.5 mm, vias 0 -> 5
- net M1_S1: track 0.00 -> 135.9 mm, vias 0 -> 5
- net Motor1_OFF: track 0.00 -> 128.2 mm, vias 0 -> 1
- net PWM: track 9.45 -> 129.9 mm, vias 0 -> 6
- net PGD: track 22.7 -> 123.4 mm, vias 3 -> 6
- net B1: track 24.8 -> 122.5 mm, vias 2 -> 3
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Other:
- board size 108.2 x 121.5 mm -> 108.2 x 124.9 mm
