File: circuts/SBC/SBC.kicad_pcb (KiCad board)
At the start: 2 copper layers, 108.2 x 124.9 mm, 369 parts, among them IC1 PIC16F15243-I_SS, J1 640456-3, J10 DE9_Plug, J11 buzzer, J13 Conn_01x04_Pin, J14 5v Power, J15 Barrel_Jack_MountingPin, J2 B5B-XH-A_LF__SN_, J3 Power, J4 DE9_Plug, J5 OSTTC060162, J6 XT60-M, J7 OSTTC060162, J8 DE9_Plug, Q1 MMBTA06, Q10 BC817, Q11 AO3400A, Q2 MMBTA06, Q3 MMBTA06, Q4 IRFS4227, Q5 MMBTA06, Q6 MMBTA06, Q7 MMBTA06, Q8 IRFS4227, SW1 SW_Push, SW2 SW_Push, SW3 SW_Push, SW4 SW_Push, SW5 SW_Push, SW6 rst, SW7 SW_Push, U1 UC3843, U10 ESP32-DEVKIT-V1, U12 L7805, U13 L7805, U14 L7809, U2 BTS7960B, U3 BTS7960B, U4 LM358DT, U5 AMS1117-3.3, U7 BTS7960B, U8 BTS7960B, U9 LM358DT

Commit message: siddyq test plane
Parts:
- removed the C13 at (235.3, 80.1)
- removed the C5 at (176.8, 79.2)
- added REF**: MountingHole_3.2mm_M3, MountingHole:MountingHole_3.2mm_M3, F.Cu at (237.2, 80.2)
- added REF**: MountingHole_3.2mm_M3, MountingHole:MountingHole_3.2mm_M3, F.Cu at (191.4, 80.0)
- moved C46 21.9 mm to (259.3, 80.0)
- moved C3 19.2 mm to (176.6, 79.1)
- moved D35 4.46 mm to (197.1, 77.5)
- moved D36 4.46 mm to (194.8, 81.0)
- moved C55 1.51 mm to (261.3, 80.1)
- moved R66 1.20 mm to (168.3, 68.2)
- moved R63 1.05 mm to (170.7, 68.1)
- moved D40 0.76 mm to (171.3, 89.5)
- moved C96 0.70 mm to (186.4, 98.1)
- moved C91 0.43 mm to (186.5, 80.4)
- moved R116 0.30 mm to (181.1, 81.2)
- moved C12 0.15 mm to (256.1, 80.9)
Routing:
- net M1_R: track 132.6 -> 115.7 mm, vias 5 -> 4
- net M2_R: track 83.0 -> 75.7 mm, vias 10 -> 7
- net INH2: track 64.4 -> 70.4 mm
- net M1_L: track 97.0 -> 92.4 mm
- net CS: track 137.5 -> 141.1 mm
- net Motor2_OFF: track 54.8 -> 52.3 mm
- net Net-(D42-K): track 87.5 -> 89.8 mm
- net error 1: track 45.7 -> 43.4 mm
- net tst2: track 77.3 -> 79.6 mm
- net HV: track 687.4 -> 689.7 mm
- net M2_L: track 85.6 -> 83.4 mm, vias 6 -> 5
- net SCL: track 266.8 -> 268.7 mm
- net Net-(D52-K): track 6.02 -> 4.40 mm
- net voltge_sen: track 48.7 -> 47.2 mm
- net 3.3v: track 462.8 -> 464.3 mm
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Other:
- outline, holes or cut-outs redrawn

Commit message: siddyq done
Routing:
- net 5v+: track 644.7 -> 634.2 mm
- net PGD: track 123.4 -> 113.5 mm
- net Mcler: track 260.3 -> 252.4 mm
- net HV: track 689.7 -> 682.2 mm
- net SCL: track 268.7 -> 262.9 mm
- net error 2: track 114.0 -> 108.4 mm
- net M1_S1: track 135.9 -> 130.4 mm
- net 9v+: track 203.6 -> 198.8 mm
- net Net-(C93-Pad1): track 28.5 -> 24.4 mm
- net M1_R: track 115.7 -> 119.6 mm
- net SDA: track 169.3 -> 165.4 mm
- net PWM: track 131.2 -> 127.3 mm
- net Motor1_OFF: track 127.4 -> 123.6 mm
- net CS: track 141.1 -> 137.6 mm
- net GND: track 1380.1 -> 1376.8 mm
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- added copper zone on B.Cu, net GND
- added copper zone on F.Cu, net GND

Commit message: siddyq has done it
Parts:
- added G***: LOGO, SBC:robochellogo, F.Cu at (245.2, 119.3)
- added G***: LOGO, LOGO, F.Cu at (252.9, 116.8)
- added G***: LOGO, LOGO, F.Cu at (214.8, 139.1)
- added G***: LOGO, LOGO, B.Cu at (215.5, 138.1)
Routing:
- net 5v+: track 634.2 -> 610.8 mm, vias 17 -> 16
- net 3.3v: track 461.9 -> 463.4 mm
- net GND: track 1376.8 -> 1377.3 mm
