File: circuts/main/mian_circut/mian_circut.kicad_sch (KiCad schematic)
At the start: 75 parts, among them J1 12v Power, J2 5v Power, J3 buzzer, J4 DE9_Plug, J5 metal detect, J6 Conn_02x04_Odd_Even, J7 302-S101, Q1 FDS4559, Q3 BC817, U1 ESP32-DEVKIT-V1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

Commit message: local_grib
Parts:
- J4: value DE9_Plug -> motor_con
Connections:
- net HVblock is gone; now on net HV: C3.1, D1.1 (K), D15.1 (A1), D2.K, F1.1, J4.1, J4.6
- net 12v: no longer C12.1, C13.1, C14.1, C15.1, C16.1, C17.1, C18.1, C19.1, R9.2
- net HV: now also C12.1, C13.1, C14.1, C15.1, C16.1, C17.1, C18.1, C19.1, R9.2
Other:
- moved on the sheet: C1, C28, C29, C3, D1, D12, D15, D16, D2, D3, D4, D8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

Commit message: compact ic int
Parts:
- removed J7: 302-S101, digikey-footprints:PinHeader_2x5_P2.54mm_Drill1.2mm, symbol dk_Rectangular-Connectors-Headers-Male-Pins:302-S101
- added J8: grip_con, Connector_Dsub:DSUB-9_Male_Horizontal_P2.77x2.54mm_EdgePinOffset9.40mm, symbol Connector:DE9_Plug
- added R13, R14: 10k, Resistor_SMD:R_0805_2012Metric_Pad1.20x1.40mm_HandSolder, symbol Device:R
Connections:
- net 3.3V: now also J8.4, R13.2, R14.2
- net 5v+: now also J8.3
- net GND: now also J8.2, J8.7
- net HV: now also J8.1, J8.6
- net RST: now also J8.8
- net SCL: now also J8.5, R13.1
- net SDA: now also J8.9, R14.1
Other:
- moved on the sheet: J6, U2

Commit message: last_touches
Other:
- moved on the sheet: C28, C29, F4, U4, ZD1

Commit message: make the full
Parts:
- removed D12: LED, Capacitor_SMD:C_0603_1608Metric_Pad1.08x0.95mm_HandSolder, symbol Device:LED
- removed R11: 220, Capacitor_SMD:C_0805_2012Metric_Pad1.18x1.45mm_HandSolder, symbol Device:R
- removed U3: ESP32-DEVKITC-32D, ESP32-DEVKITC-32D:MODULE_ESP32-DEVKITC-32D, symbol ESP32-DEVKITC-32D:ESP32-DEVKITC-32D
Connections:
- net IRQ: now also U1.25 (D27)
- net buzz: now also U1.5 (D4)
- net detect: now also U1.8 (D5)
Other:
- moved on the sheet: C10, C11, C12, C13, C14, C15, C16, C17, C18, C19, C20, C21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

Commit message: 29-6 siddyq
Parts:
- removed U4: 78M05 SMD, digikey-footprints:TO-220-3, symbol dk_PMIC-Voltage-Regulators-Linear:LM7805CT_Obsolete
- added U3: AMS1117-5.0, Package_TO_SOT_SMD:SOT-223-3_TabPin2, symbol Regulator_Linear:AMS1117-5.0
- added U5: AMS1117-3.3, Package_TO_SOT_SMD:SOT-223-3_TabPin2, symbol Regulator_Linear:AMS1117-3.3
Connections:
- net GND: now also U3.1 (GND)
- net at C28.2, R7.1: now also U3.3 (VI)
- net at C29.2, F4.1: now also U3.2 (VO)
Changed lines of the file:
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@@
 	)
 	(symbol
-		(lib_id "dk_PMIC-Voltage-Regulators-Linear:LM7805CT_Obsolete")
-		(at 274.2914 29.9406 0)
-		(unit 1)
-		(exclude_from_sim no)
-		(in_bom yes)
-		(on_board yes)
-		(dnp no)
-		(fields_autoplaced yes)
-		(property "Reference" "U4"
-			(at 274.2914 21.9942 0)
-			(effects
-				(font
-					(size 1.524 1.524)
-				)
-			)
-		)
-		(property "Value" "78M05 SMD"
-			(at 274.2914 24.5342 0)
-			(effects
-				(font
-					(size 1.524 1.524)
-				)
-			)
-		)
-		(property "Footprint" "digikey-footprints:TO-220-3"
-			(at 279.3714 24.8606 0)
-			(effects
-				(font
-					(size 1.524 1.524)
-				)
-				(justify left)
-				(hide yes)
-			)
-		)
-		(property "Datasheet" "https://media.digikey.com/pdf/Data%20Sheets/ON%20Semiconductor%20PDFs/MC7800(A,AE),NCV7800.pdf"
-			(at 279.3714 22.3206 0)
-			(effects
-				(font
-					(size 1.524 1.524)
-				)
-				(justify left)
-				(hide yes)
-			)
-		)
-		(property "Description" "IC REG LINEAR 5V 1A TO220AB"
-			(at 274.2914 29.9406 0)
-			(effects
-				(font
-					(size 1.27 1.27)
-				)
-				(hide yes)
-			)
-		)
-		(property "Digi-Key_PN" "LM7805CT-ND"
-			(at 279.3714 19.7806 0)
-			(effects
-				(font
-					(size 1.524 1.524)
-				)
-				(justify left)
-				(hide yes)
-			)
-		)
-		(property "MPN" "LM7805CT"
-			(at 279.3714 17.2406 0)
-			(effects
-				(font
-					(size 1.524 1.524)
-				)
-				(justify left)
-				(hide yes)
-			)
-		)
-		(property "Category" "Integrated Circuits (ICs)"
-			(at 279.3714 14.7006 0)
-			(effects
-				(font
-					(size 1.524 1.524)
-				)
-				(justify left)
-				(hide yes)
-			)
-		)
-		(property "Family" "PMIC - Voltage Regulators - Linear"
-			(at 279.3714 12.1606 0)
-			(effects
-				(font
-					(size 1.524 1.524)
-				)
-				(justify left)
-				(hide yes)
-			)
-		)
-		(property "DK_Datasheet_Link" "https://media.digikey.com/pdf/Data%20Sheets/ON%20Semiconductor%20PDFs/MC7800(A,AE),NCV7800.pdf"
-			(at 279.3714 9.6206 0)
-			(effects
-				(font
-					(size 1.524 1.524)
-				)
-				(justify left)
-				(hide yes)
-			)
-		)
-		(property "DK_Detail_Page" "/product-detail/en/on-semiconductor/LM7805CT/LM7805CT-ND/458698"
-			(at 279.3714 7.0806 0)
-			(effects
-				(font
-					(size 1.524 1.524)
-				)
-				(justify left)
-				(hide yes)
-			)
-		)
-		(property "Description_1" "IC REG LINEAR 5V 1A TO220AB"
-			(at 279.3714 4.5406 0)
-			(effects
-				(font
-					(size 1.524 1.524)
-				)
-				(justify left)
-				(hide yes)
-			)
-		)
-		(property "Manufacturer" "ON Semiconductor"
-			(at 279.3714 2.0006 0)
-			(effects
-				(font
-					(size 1.524 1.524)
-				)
-				(justify left)
-				(hide yes)
-			)
-		)
-		(property "Status" "Obsolete NonStock"
-			(at 279.3714 -0.5394 0)
-			(effects
-				(font
-					(size 1.524 1.524)
-				)
-				(justify left)
-				(hide yes)
-			)
-		)
-		(pin "2"
-		)
-		(pin "1"
-		)
-		(pin "3"
-		)
-		(instances
-			(project "mian_circut"
-				(path "/7d28df94-841d-403f-9b3f-5aa03bec09c7"
-					(reference "U4")
-					(unit 1)
-				)
-			)
-		)
-	)
-	(symbol
 		(lib_id "Diode:BZV55B3V3")
 		(at 83.2714 69.8548 270)
@@
 	)
 	(symbol
+		(lib_id "Regulator_Linear:AMS1117-5.0")
+		(at 274.2914 29.9406 0)
+		(unit 1)
+		(exclude_from_sim no)
+		(in_bom yes)
+		(on_board yes)
+		(dnp no)
+		(fields_autoplaced yes)
+		(property "Reference" "U3"
+			(at 274.2914 22.8658 0)
+			(effects
+				(font
+					(size 1.27 1.27)
+				)
+			)
+		)
+		(property "Value" "AMS1117-5.0"
+			(at 274.2914 25.4058 0)
+			(effects
+				(font
+					(size 1.27 1.27)
+				)
+			)
+		)
+		(property "Footprint" "Package_TO_SOT_SMD:SOT-223-3_TabPin2"
+			(at 274.2914 24.8606 0)
+			(effects
+				(font
+					(size 1.27 1.27)
+				)
+				(hide yes)
+			)
+		)
+		(property "Datasheet" "http://www.advanced-monolithic.com/pdf/ds1117.pdf"
+			(at 276.8314 36.2906 0)
+			(effects
+				(font
+					(size 1.27 1.27)
+				)
+				(hide yes)
+			)
+		)
+		(property "Description" "1A Low Dropout regulator, positive, 5.0V fixed output, SOT-223"
+			(at 274.2914 29.9406 0)
+			(effects
+				(font
+					(size 1.27 1.27)
+				)
+				(hide yes)
+			)
+		)
+		(pin "3"
+		)
+		(pin "1"
+		)
+		(pin "2"
+		)
+		(instances
+			(project ""
+				(path "/7d28df94-841d-403f-9b3f-5aa03bec09c7"
+					(reference "U3")
+					(unit 1)
+				)
+			)
+		)
+	)
+	(symbol
 		(lib_id "Connector:Screw_Terminal_01x02")
 		(at 389.268 64.0247 0)
@@
 					(unit 1)
 				)
+			)
+		)
+	)
+	(symbol
+		(lib_id "Regulator_Linear:AMS1117-3.3")
+		(at 317.815 61.8513 0)
+		(unit 1)
+		(exclude_from_sim no)
+		(in_bom yes)
+		(on_board yes)
+		(dnp no)
+		(fields_autoplaced yes)
+		(property "Reference" "U5"
+			(at 317.815 54.61 0)
+			(effects
+				(font
+					(size 1.27 1.27)
+				)
+			)
+		)
+		(property "Value" "AMS1117-3.3"
+			(at 317.815 57.15 0)
+			(effects
+				(font
+					(size 1.27 1.27)
+				)
+			)
+		)
+		(property "Footprint" "Package_TO_SOT_SMD:SOT-223-3_TabPin2"
+			(at 317.815 56.7713 0)
+			(effects
+				(font
+					(size 1.27 1.27)
+				)
+				(hide yes)
+			)
+		)
+		(property "Datasheet" "http://www.advanced-monolithic.com/pdf/ds1117.pdf"
+			(at 320.355 68.2013 0)
+			(effects
+				(font
+					(size 1.27 1.27)
+				)
+				(hide yes)
+			)
+		)
+		(property "Description" "1A Low Dropout regulator, positive, 3.3V fixed output, SOT-223"
+			(at 317.815 61.8513 0)
+			(effects
+				(font
+					(size 1.27 1.27)
+				)
+				(hide yes)
+			)
+		)
+		(pin "3"
+		)
+		(pin "1"
+		)
+		(pin "2"
+		)
+		(instances
+			(project ""
+				(path "/7d28df94-841d-403f-9b3f-5aa03bec09c7"
+					(reference "U5")
+					(unit 1)
+				)
