File: SBC.kicad_pcb (KiCad board)
At the start: 2 copper layers, 108.2 x 124.9 mm, 389 parts, among them IC1 PIC16F15243-I_SS, J1 640456-3, J10 DE9_Plug, J11 buzzer, J13 Conn_01x04_Pin, J14 5v Power, J15 Barrel_Jack_MountingPin, J2 B5B-XH-A_LF__SN_, J3 Power, J4 DE9_Plug, J5 OSTTC060162, J6 XT60-M, J7 OSTTC060162, J8 DE9_Plug, Q1 MMBTA06, Q10 BC817, Q11 AO3400A, Q2 MMBTA06, Q3 MMBTA06, Q4 IRFS4227, Q5 MMBTA06, Q6 MMBTA06, Q7 MMBTA06, Q8 IRFS4227, SW1 SW_Push, SW2 SW_Push, SW3 SW_Push, SW4 SW_Push, SW5 SW_Push, SW6 rst, SW7 SW_Push, U1 UC3843, U10 ESP32-DEVKIT-V1, U12 L7805, U13 L7805, U14 L7809, U2 BTS7960B, U3 BTS7960B, U4 LM358DT, U5 AMS1117-3.3, U7 BTS7960B, U8 BTS7960B, U9 LM358DT

Commit message: siddyq has finsh siddyq is done oh this feeling
Parts:
- removed ? (x3): , 
- removed the G*** at (181.6, 120.8)
- removed the G*** at (247.7, 113.5)
- removed the G*** at (214.5, 151.9)
- removed the G*** at (188.7, 141.3)
- removed the G*** at (243.2, 116.0)
- removed the G*** at (183.5, 138.2)
- removed the G*** at (194.0, 144.6)
- removed the G*** at (214.6, 117.7)
- removed the G*** at (210.1, 141.5)
- removed the G*** at (243.2, 129.6)
- removed the G*** at (245.4, 125.3)
- removed the G*** at (223.8, 158.9)
- removed the G*** at (217.2, 143.0)
- removed the G*** at (248.8, 135.8)
- added G***: LOGO, LOGO, F.Cu at (214.8, 139.1)
- moved G*** 1.04 mm to (215.5, 138.1)
Routing:
- net GND: track 1410.9 -> 1377.3 mm, vias 86 -> 32
- net HV: track 700.9 -> 682.1 mm, vias 22 -> 17
- net M1_L: track 106.3 -> 91.8 mm, vias 6 -> 4
- net M2_R: track 82.2 -> 74.3 mm
- net 5v+: track 618.4 -> 610.8 mm, vias 19 -> 16
- net M2_L: track 88.8 -> 83.0 mm, vias 12 -> 5
- net M1_R: track 124.0 -> 119.8 mm, vias 8 -> 4
- net SW2: track 16.8 -> 12.8 mm, vias 1 -> 0
- net SW1: track 16.5 -> 12.7 mm, vias 1 -> 0
- net SW3: track 12.4 -> 8.70 mm, vias 1 -> 0
- net SDA: track 168.6 -> 165.2 mm, vias 4 -> 3
- net SW4: track 12.3 -> 8.94 mm, vias 1 -> 0
- net 3.3v: track 466.4 -> 463.4 mm
- net Mcler: track 254.5 -> 252.4 mm, vias 5 -> 4
- net Net-(C43-Pad1): track 14.5 -> 12.6 mm, vias 1 -> 0
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